File: lopro/pcb/pcb.kicad_pcb (KiCad board)
At the start: 2 copper layers, 101 parts, among them J1 Conn_01x08_Female, J2 Conn_01x08_Female, J3 Conn_01x08_Female, J4 PCB_Lopro_Conn

Commit message: M .gitignore M  lopro/drawborderk.py M  lopro/pcb/pcb.kicad_pcb M  lopro/pcb/pcb.kicad_sch M  lopro/place_fp.py
Parts:
- added R1: R_Small, Resistor_SMD:R_0603_1608Metric_Pad0.98x0.95mm_HandSolder, F.Cu at (233.5, -17.9)
- added R10: R_Small, Resistor_SMD:R_0603_1608Metric_Pad0.98x0.95mm_HandSolder, F.Cu at (237.9, -20.4)
- added R11: R_Small, Resistor_SMD:R_0603_1608Metric_Pad0.98x0.95mm_HandSolder, F.Cu at (229.2, -25.4)
- added R12: R_Small, Resistor_SMD:R_0603_1608Metric_Pad0.98x0.95mm_HandSolder, F.Cu at (246.6, -22.9)
- added R13: R_Small, Resistor_SMD:R_0603_1608Metric_Pad0.98x0.95mm_HandSolder, F.Cu at (246.6, -20.4)
- added R14: R_Small, Resistor_SMD:R_0603_1608Metric_Pad0.98x0.95mm_HandSolder, F.Cu at (242.2, -25.4)
- added R15: R_Small, Resistor_SMD:R_0603_1608Metric_Pad0.98x0.95mm_HandSolder, F.Cu at (233.5, -25.4)
- added R16: R_Small, Resistor_SMD:R_0603_1608Metric_Pad0.98x0.95mm_HandSolder, F.Cu at (237.9, -22.9)
- added R17: R_Small, Resistor_SMD:R_0603_1608Metric_Pad0.98x0.95mm_HandSolder, F.Cu at (237.9, -17.9)
- added R18: R_Small, Resistor_SMD:R_0603_1608Metric_Pad0.98x0.95mm_HandSolder, F.Cu at (237.9, -27.9)
- added R19: R_Small, Resistor_SMD:R_0603_1608Metric_Pad0.98x0.95mm_HandSolder, F.Cu at (229.2, -17.9)
- added R2: R_Small, Resistor_SMD:R_0603_1608Metric_Pad0.98x0.95mm_HandSolder, F.Cu at (246.6, -27.9)
- added R20: R_Small, Resistor_SMD:R_0603_1608Metric_Pad0.98x0.95mm_HandSolder, F.Cu at (229.2, -22.9)
- added R21: R_Small, Resistor_SMD:R_0603_1608Metric_Pad0.98x0.95mm_HandSolder, F.Cu at (233.5, -22.9)
- added R22: R_Small, Resistor_SMD:R_0603_1608Metric_Pad0.98x0.95mm_HandSolder, F.Cu at (246.6, -25.4)
- added R23: R_Small, Resistor_SMD:R_0603_1608Metric_Pad0.98x0.95mm_HandSolder, F.Cu at (233.5, -27.9)
- added R24: R_Small, Resistor_SMD:R_0603_1608Metric_Pad0.98x0.95mm_HandSolder, F.Cu at (242.2, -22.9)
- added R3: R_Small, Resistor_SMD:R_0603_1608Metric_Pad0.98x0.95mm_HandSolder, F.Cu at (242.2, -27.9)
- added R4: R_Small, Resistor_SMD:R_0603_1608Metric_Pad0.98x0.95mm_HandSolder, F.Cu at (242.2, -17.9)
- added R5: R_Small, Resistor_SMD:R_0603_1608Metric_Pad0.98x0.95mm_HandSolder, F.Cu at (229.2, -20.4)
- added R6: R_Small, Resistor_SMD:R_0603_1608Metric_Pad0.98x0.95mm_HandSolder, F.Cu at (233.5, -20.4)
- added R7: R_Small, Resistor_SMD:R_0603_1608Metric_Pad0.98x0.95mm_HandSolder, F.Cu at (242.2, -20.4)
- added R8: R_Small, Resistor_SMD:R_0603_1608Metric_Pad0.98x0.95mm_HandSolder, F.Cu at (229.2, -27.9)
- added R9: R_Small, Resistor_SMD:R_0603_1608Metric_Pad0.98x0.95mm_HandSolder, F.Cu at (237.9, -25.4)
- J1: value Conn_01x08_Female -> PCB_Lopro_Conn; footprint Connector_PinHeader_2.54mm:PinHeader_1x08_P2.54mm_Vertical -> Connector:GB042-34S-H10
- J4: value PCB_Lopro_Conn -> Conn_01x08_Female; footprint Connector:GB042-34S-H10 -> Connector_PinHeader_2.54mm:PinHeader_1x08_P2.54mm_Vertical
- moved Hs8 199.5 mm to (209.0, 27.9)
- moved Hs9 198.3 mm to (268.4, 26.5)
- moved Hs7 96.7 mm to (152.0, 27.9)
- moved Hs16 72.9 mm to (157.8, 105.0)
- moved Hs18 72.0 mm to (285.0, 84.9)
- moved Hs17 66.5 mm to (228.0, 84.9)
- moved Hs10 60.1 mm to (90.2, 67.1)
- moved Hs6 57.0 mm to (95.0, 27.9)
- moved Hs11 42.5 mm to (185.2, 67.1)
- moved Hs15 27.2 mm to (117.8, 105.0)
- moved Hs5 26.9 mm to (35.6, 26.5)
- moved Hs13 23.8 mm to (0.00, 84.9)
- moved S58 9.50 mm to (275.5, 57.0)
- moved S70 9.50 mm to (237.5, 76.0)
- moved S71 9.50 mm to (256.5, 76.0)
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Connections:
- J1 pad 1: unconnected-(J1-Pad1) -> /COL1A
- J1 pad 2: unconnected-(J1-Pad2) -> /COL2A
- J1 pad 3: unconnected-(J1-Pad3) -> /COL3A
- J1 pad 4: unconnected-(J1-Pad4) -> /COL4A
- J1 pad 5: unconnected-(J1-Pad5) -> /COL5A
- J1 pad 6: unconnected-(J1-Pad6) -> /COL6A
- J1 pad 7: unconnected-(J1-Pad7) -> /COL7A
- J1 pad 8: unconnected-(J1-Pad8) -> /COL8A
- J4 pad 1: /COL1A -> unconnected-(J4-Pad1)
- J4 pad 2: /COL2A -> unconnected-(J4-Pad2)
- J4 pad 3: /COL3A -> unconnected-(J4-Pad3)
- J4 pad 4: /COL4A -> unconnected-(J4-Pad4)
- J4 pad 5: /COL5A -> unconnected-(J4-Pad5)
- J4 pad 6: /COL6A -> unconnected-(J4-Pad6)
- J4 pad 7: /COL7A -> unconnected-(J4-Pad7)
- J4 pad 8: /COL8A -> unconnected-(J4-Pad8)
Other:
- board outline added: 308.8 x 191.1 mm

Commit message: added tracks
M  Giri_Library.pretty/Keychron_Optical_Switch_1u.kicad_mod
D  lopro/drawborder.py
M  lopro/pcb/pcb.kicad_pcb
M  lopro/pcb/pcb.kicad_prl
M  lopro/place_fp.py
Parts:
- added Hs26: M2, giri:SMTSO_M2, F.Cu at (207.2, 119.0)
- moved Hs22 251.4 mm to (-10.8, 119.0)
- moved Hs21 239.2 mm to (-10.8, 173.0)
- moved J2 222.4 mm to (47.5, -10.0), turned to 90 degrees
- moved Hs19 180.1 mm to (68.2, 119.0)
- moved Hs20 175.0 mm to (68.2, 173.0)
- moved J4 162.9 mm to (237.5, -10.0), turned to 90 degrees
- moved J3 158.5 mm to (142.5, -10.0), turned to 90 degrees
- moved Hs24 57.1 mm to (286.2, 173.0)
- moved J1 50.7 mm to (3.75, 19.0), turned to 0 degrees
- moved Hs23 50.1 mm to (286.2, 119.0)
- moved Hs25 41.2 mm to (207.2, 173.0)
Routing:
- net +5V: track 0.00 -> 1327.7 mm
- net /ROW4: track 0.00 -> 231.5 mm
- net /ROW2: track 0.00 -> 222.0 mm
- net /ROW3: track 0.00 -> 219.6 mm
- net /ROW1: track 0.00 -> 217.2 mm
- net /ROW6: track 0.00 -> 147.7 mm
- net GND: track 0.00 -> 72.0 mm, vias 0 -> 72
- net /ROW5: track 0.00 -> 61.6 mm
- net /COL9A: track 0.00 -> 51.6 mm, vias 0 -> 3
- net /COL8A: track 0.00 -> 51.6 mm, vias 0 -> 3
- net /COL6A: track 0.00 -> 51.6 mm, vias 0 -> 3
- net /COL5A: track 0.00 -> 51.6 mm, vias 0 -> 3
- net /COL4A: track 0.00 -> 51.6 mm, vias 0 -> 3
- net /COL3A: track 0.00 -> 51.6 mm, vias 0 -> 3
- net /COL2A: track 0.00 -> 51.6 mm, vias 0 -> 3
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Other:
- board size 308.8 x 191.1 mm -> 314.5 x 191.1 mm

Commit message: add tracks
M  Giri_Library.kicad_sym
M  Giri_Library.pretty/Keychron_Optical_Switch_1u.kicad_mod
A  lopro/pcb/LED-Driver.kicad_sch
M  lopro/pcb/pcb.kicad_pcb
M  lopro/pcb/pcb.kicad_sch
M  lopro/place_fp.py
Parts:
- added C1: 10uF, Capacitor_SMD:C_1206_3216Metric, F.Cu at (158.5, 149.4)
- added C2: 10uF, Capacitor_SMD:C_1206_3216Metric, F.Cu at (164.8, 143.2)
- added C3: 100nF, Capacitor_SMD:C_0603_1608Metric, F.Cu at (184.0, 160.9)
- added C4: 100nF, Capacitor_SMD:C_0603_1608Metric, F.Cu at (188.4, 158.2)
- added D1: LED, LED_SMD:LED_0603_1608Metric_Pad1.05x0.95mm_HandSolder, F.Cu at (19.0, -4.80)
- added D10: LED, LED_SMD:LED_0603_1608Metric_Pad1.05x0.95mm_HandSolder, F.Cu at (190.0, -4.80)
- added D11: LED, LED_SMD:LED_0603_1608Metric_Pad1.05x0.95mm_HandSolder, F.Cu at (209.0, -4.80)
- added D12: LED, LED_SMD:LED_0603_1608Metric_Pad1.05x0.95mm_HandSolder, F.Cu at (228.0, -4.80)
- added D13: LED, LED_SMD:LED_0603_1608Metric_Pad1.05x0.95mm_HandSolder, F.Cu at (247.0, -4.80)
- added D14: LED, LED_SMD:LED_0603_1608Metric_Pad1.05x0.95mm_HandSolder, F.Cu at (266.0, -4.80)
- added D15: LED, LED_SMD:LED_0603_1608Metric_Pad1.05x0.95mm_HandSolder, F.Cu at (285.0, -4.80)
- added D16: LED, LED_SMD:LED_0603_1608Metric_Pad1.05x0.95mm_HandSolder, F.Cu at (23.8, 14.2)
- added D17: LED, LED_SMD:LED_0603_1608Metric_Pad1.05x0.95mm_HandSolder, F.Cu at (47.5, 14.2)
- added D18: LED, LED_SMD:LED_0603_1608Metric_Pad1.05x0.95mm_HandSolder, F.Cu at (66.5, 14.2)
- added D19: LED, LED_SMD:LED_0603_1608Metric_Pad1.05x0.95mm_HandSolder, F.Cu at (85.5, 14.2)
- added D2: LED, LED_SMD:LED_0603_1608Metric_Pad1.05x0.95mm_HandSolder, F.Cu at (38.0, -4.80)
- added D20: LED, LED_SMD:LED_0603_1608Metric_Pad1.05x0.95mm_HandSolder, F.Cu at (104.5, 14.2)
- added D21: LED, LED_SMD:LED_0603_1608Metric_Pad1.05x0.95mm_HandSolder, F.Cu at (123.5, 14.2)
- added D22: LED, LED_SMD:LED_0603_1608Metric_Pad1.05x0.95mm_HandSolder, F.Cu at (142.5, 14.2)
- added D23: LED, LED_SMD:LED_0603_1608Metric_Pad1.05x0.95mm_HandSolder, F.Cu at (161.5, 14.2)
- added D24: LED, LED_SMD:LED_0603_1608Metric_Pad1.05x0.95mm_HandSolder, F.Cu at (180.5, 14.2)
- added D25: LED, LED_SMD:LED_0603_1608Metric_Pad1.05x0.95mm_HandSolder, F.Cu at (199.5, 14.2)
- added D26: LED, LED_SMD:LED_0603_1608Metric_Pad1.05x0.95mm_HandSolder, F.Cu at (218.5, 14.2)
- added D27: LED, LED_SMD:LED_0603_1608Metric_Pad1.05x0.95mm_HandSolder, F.Cu at (237.5, 14.2)
- added D28: LED, LED_SMD:LED_0603_1608Metric_Pad1.05x0.95mm_HandSolder, F.Cu at (256.5, 14.2)
- added D29: LED, LED_SMD:LED_0603_1608Metric_Pad1.05x0.95mm_HandSolder, F.Cu at (280.2, 14.2)
- added D3: LED, LED_SMD:LED_0603_1608Metric_Pad1.05x0.95mm_HandSolder, F.Cu at (57.0, -4.80)
- added D30: LED, LED_SMD:LED_0603_1608Metric_Pad1.05x0.95mm_HandSolder, F.Cu at (11.9, 33.2)
- added D31: LED, LED_SMD:LED_0603_1608Metric_Pad1.05x0.95mm_HandSolder, F.Cu at (33.2, 33.2)
- added D32: LED, LED_SMD:LED_0603_1608Metric_Pad1.05x0.95mm_HandSolder, F.Cu at (52.2, 33.2)
- added D33: LED, LED_SMD:LED_0603_1608Metric_Pad1.05x0.95mm_HandSolder, F.Cu at (71.2, 33.2)
- added D34: LED, LED_SMD:LED_0603_1608Metric_Pad1.05x0.95mm_HandSolder, F.Cu at (90.2, 33.2)
- added D35: LED, LED_SMD:LED_0603_1608Metric_Pad1.05x0.95mm_HandSolder, F.Cu at (109.2, 33.2)
- added D36: LED, LED_SMD:LED_0603_1608Metric_Pad1.05x0.95mm_HandSolder, F.Cu at (128.2, 33.2)
- added D37: LED, LED_SMD:LED_0603_1608Metric_Pad1.05x0.95mm_HandSolder, F.Cu at (147.2, 33.2)
- added D38: LED, LED_SMD:LED_0603_1608Metric_Pad1.05x0.95mm_HandSolder, F.Cu at (166.2, 33.2)
- added D39: LED, LED_SMD:LED_0603_1608Metric_Pad1.05x0.95mm_HandSolder, F.Cu at (185.2, 33.2)
- added D4: LED, LED_SMD:LED_0603_1608Metric_Pad1.05x0.95mm_HandSolder, F.Cu at (76.0, -4.80)
- added D40: LED, LED_SMD:LED_0603_1608Metric_Pad1.05x0.95mm_HandSolder, F.Cu at (204.2, 33.2)
- added D41: LED, LED_SMD:LED_0603_1608Metric_Pad1.05x0.95mm_HandSolder, F.Cu at (223.2, 33.2)
- added D42: LED, LED_SMD:LED_0603_1608Metric_Pad1.05x0.95mm_HandSolder, F.Cu at (242.2, 33.2)
- added D43: LED, LED_SMD:LED_0603_1608Metric_Pad1.05x0.95mm_HandSolder, F.Cu at (261.2, 33.2)
- added D44: LED, LED_SMD:LED_0603_1608Metric_Pad1.05x0.95mm_HandSolder, F.Cu at (282.6, 33.2)
- added D45: LED, LED_SMD:LED_0603_1608Metric_Pad1.05x0.95mm_HandSolder, F.Cu at (9.50, 52.2)
- added D46: LED, LED_SMD:LED_0603_1608Metric_Pad1.05x0.95mm_HandSolder, F.Cu at (35.6, 52.2)
- added D47: LED, LED_SMD:LED_0603_1608Metric_Pad1.05x0.95mm_HandSolder, F.Cu at (61.8, 52.2)
- added D48: LED, LED_SMD:LED_0603_1608Metric_Pad1.05x0.95mm_HandSolder, F.Cu at (80.8, 52.2)
- added D49: LED, LED_SMD:LED_0603_1608Metric_Pad1.05x0.95mm_HandSolder, F.Cu at (99.8, 52.2)
- added D5: LED, LED_SMD:LED_0603_1608Metric_Pad1.05x0.95mm_HandSolder, F.Cu at (95.0, -4.80)
- added D50: LED, LED_SMD:LED_0603_1608Metric_Pad1.05x0.95mm_HandSolder, F.Cu at (118.8, 52.2)
- added D51: LED, LED_SMD:LED_0603_1608Metric_Pad1.05x0.95mm_HandSolder, F.Cu at (137.8, 52.2)
- added D52: LED, LED_SMD:LED_0603_1608Metric_Pad1.05x0.95mm_HandSolder, F.Cu at (156.8, 52.2)
- added D53: LED, LED_SMD:LED_0603_1608Metric_Pad1.05x0.95mm_HandSolder, F.Cu at (175.8, 52.2)
- added D54: LED, LED_SMD:LED_0603_1608Metric_Pad1.05x0.95mm_HandSolder, F.Cu at (194.8, 52.2)
- added D55: LED, LED_SMD:LED_0603_1608Metric_Pad1.05x0.95mm_HandSolder, F.Cu at (213.8, 52.2)
- added D56: LED, LED_SMD:LED_0603_1608Metric_Pad1.05x0.95mm_HandSolder, F.Cu at (232.8, 52.2)
- added D57: LED, LED_SMD:LED_0603_1608Metric_Pad1.05x0.95mm_HandSolder, F.Cu at (258.9, 52.2)
- added D58: LED, LED_SMD:LED_0603_1608Metric_Pad1.05x0.95mm_HandSolder, F.Cu at (285.0, 52.2)
- added D59: LED, LED_SMD:LED_0603_1608Metric_Pad1.05x0.95mm_HandSolder, F.Cu at (16.6, 71.2)
- added D6: LED, LED_SMD:LED_0603_1608Metric_Pad1.05x0.95mm_HandSolder, F.Cu at (114.0, -4.80)
- added D60: LED, LED_SMD:LED_0603_1608Metric_Pad1.05x0.95mm_HandSolder, F.Cu at (38.0, 71.2)
- added D61: LED, LED_SMD:LED_0603_1608Metric_Pad1.05x0.95mm_HandSolder, F.Cu at (57.0, 71.2)
- added D62: LED, LED_SMD:LED_0603_1608Metric_Pad1.05x0.95mm_HandSolder, F.Cu at (77.6, 72.2)
- added D63: LED, LED_SMD:LED_0603_1608Metric_Pad1.05x0.95mm_HandSolder, F.Cu at (97.7, 76.4)
- added D64: LED, LED_SMD:LED_0603_1608Metric_Pad1.05x0.95mm_HandSolder, F.Cu at (108.5, 90.9)
- added D65: LED, LED_SMD:LED_0603_1608Metric_Pad1.05x0.95mm_HandSolder, F.Cu at (137.8, 71.2)
- added D66: LED, LED_SMD:LED_0603_1608Metric_Pad1.05x0.95mm_HandSolder, F.Cu at (158.0, 94.1)
- added D67: LED, LED_SMD:LED_0603_1608Metric_Pad1.05x0.95mm_HandSolder, F.Cu at (177.8, 76.4)
- added D68: LED, LED_SMD:LED_0603_1608Metric_Pad1.05x0.95mm_HandSolder, F.Cu at (197.9, 72.2)
- added D69: LED, LED_SMD:LED_0603_1608Metric_Pad1.05x0.95mm_HandSolder, F.Cu at (218.5, 71.2)
- added D7: LED, LED_SMD:LED_0603_1608Metric_Pad1.05x0.95mm_HandSolder, F.Cu at (133.0, -4.80)
- added D70: LED, LED_SMD:LED_0603_1608Metric_Pad1.05x0.95mm_HandSolder, F.Cu at (237.5, 71.2)
- added D71: LED, LED_SMD:LED_0603_1608Metric_Pad1.05x0.95mm_HandSolder, F.Cu at (256.5, 71.2)
- added D72: LED, LED_SMD:LED_0603_1608Metric_Pad1.05x0.95mm_HandSolder, F.Cu at (275.5, 71.2)
- added D8: LED, LED_SMD:LED_0603_1608Metric_Pad1.05x0.95mm_HandSolder, F.Cu at (152.0, -4.80)
- added D9: LED, LED_SMD:LED_0603_1608Metric_Pad1.05x0.95mm_HandSolder, F.Cu at (171.0, -4.80)
- added R25: 20k, Resistor_SMD:R_0603_1608Metric, F.Cu at (184.0, 163.4)
- added R26: 20k, Resistor_SMD:R_0603_1608Metric, F.Cu at (192.8, 153.1)
- added R27: 20k, Resistor_SMD:R_0603_1608Metric, F.Cu at (188.4, 155.7)
- added R28: 20k, Resistor_SMD:R_0603_1608Metric, F.Cu at (198.5, 147.9)
- added R29: 20k, Resistor_SMD:R_0603_1608Metric, F.Cu at (179.6, 166.1)
- added R30: 20k, Resistor_SMD:R_0603_1608Metric, F.Cu at (199.1, 145.3)
- added U1: IS31FL3731-QF, Package_DFN_QFN:QFN-28-1EP_4x4mm_P0.4mm_EP2.3x2.3mm, F.Cu at (158.8, 144.6)
- J1: footprint Connector:GB042-34S-H10 -> Connector_Dsub:DSUB-37_Female_Horizontal_P2.77x2.84mm_EdgePinOffset4.94mm_Housed_MountingHolesOffset7.48mm
- moved R1 308.9 mm to (-73.8, 13.2)
- moved R10 308.9 mm to (-69.5, 10.7)
- moved R11 308.9 mm to (-78.2, 5.70)
- moved R12 308.9 mm to (-60.8, 8.21)
- moved R13 308.9 mm to (-60.8, 10.7)
- moved R14 308.9 mm to (-65.1, 5.70)
- moved R15 308.9 mm to (-73.8, 5.70)
- moved R16 308.9 mm to (-69.5, 8.21)
- moved R17 308.9 mm to (-69.5, 13.2)
- moved R18 308.9 mm to (-69.5, 3.19)
- moved R19 308.9 mm to (-78.2, 13.2)
- moved R2 308.9 mm to (-60.8, 3.19)
- moved R20 308.9 mm to (-78.2, 8.21)
- moved R21 308.9 mm to (-73.8, 8.21)
- moved R22 308.9 mm to (-60.8, 5.70)
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Routing:
- net CA4: track 0.00 -> 220.5 mm, vias 0 -> 5
- net CB1: track 0.00 -> 182.7 mm, vias 0 -> 5
- net CB4: track 0.00 -> 180.0 mm, vias 0 -> 5
- net CA3: track 0.00 -> 179.0 mm, vias 0 -> 4
- net CB3: track 0.00 -> 158.8 mm, vias 0 -> 4
- net CA2: track 0.00 -> 158.4 mm, vias 0 -> 4
- net CA1: track 0.00 -> 153.7 mm, vias 0 -> 4
- net CB2: track 0.00 -> 145.6 mm, vias 0 -> 5
- net CB5: track 0.00 -> 144.9 mm, vias 0 -> 5
- net CA5: track 0.00 -> 127.0 mm, vias 0 -> 5
- net CA6: track 0.00 -> 87.1 mm, vias 0 -> 6
- net CA8: track 0.00 -> 87.1 mm, vias 0 -> 6
- net CA9: track 0.00 -> 87.1 mm, vias 0 -> 6
- net CA7: track 0.00 -> 87.1 mm, vias 0 -> 6
- net CB6: track 0.00 -> 67.5 mm, vias 0 -> 6
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