File: lopro/pcb/pcb.kicad_sch (KiCad schematic)
At the start: 125 parts, among them J1 PCB_Lopro_Conn, J2 Conn_01x08_Female, J3 Conn_01x08_Female, J4 Conn_01x08_Female

Commit message: M .gitignore M  lopro/drawborderk.py M  lopro/pcb/pcb.kicad_pcb M  lopro/pcb/pcb.kicad_sch M  lopro/place_fp.py
Parts:
- added Hs18: M2, giri:SMTSO_M2, symbol giri:MountingHoleSMD
- renumbered Hs18 to Hs19, Hs19 to Hs20, Hs20 to Hs21, Hs21 to Hs22, Hs22 to Hs23, Hs23 to Hs24, Hs24 to Hs25, Hs25 to Hs26
Changed lines of the file:
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@@
   (symbol (lib_name "MountingHoleSMD_1") (lib_id "giri:MountingHoleSMD") (at 140.97 186.69 0) (unit 1)
     (in_bom yes) (on_board yes) (fields_autoplaced)
-    (property "Reference" "Hs18" (id 0) (at 143.51 185.8553 0)
+    (property "Reference" "Hs19" (id 0) (at 143.51 185.8553 0)
       (effects (font (size 1.27 1.27)) (justify left))
     )
@@
   (symbol (lib_name "MountingHoleSMD_1") (lib_id "giri:MountingHoleSMD") (at 160.02 186.69 0) (unit 1)
     (in_bom yes) (on_board yes) (fields_autoplaced)
-    (property "Reference" "Hs21" (id 0) (at 162.56 185.8553 0)
+    (property "Reference" "Hs22" (id 0) (at 162.56 185.8553 0)
       (effects (font (size 1.27 1.27)) (justify left))
     )
@@
   (symbol (lib_name "MountingHoleSMD_1") (lib_id "giri:MountingHoleSMD") (at 140.97 193.04 0) (unit 1)
     (in_bom yes) (on_board yes) (fields_autoplaced)
-    (property "Reference" "Hs22" (id 0) (at 143.51 192.2053 0)
+    (property "Reference" "Hs23" (id 0) (at 143.51 192.2053 0)
       (effects (font (size 1.27 1.27)) (justify left))
     )
@@
   (symbol (lib_name "MountingHoleSMD_1") (lib_id "giri:MountingHoleSMD") (at 160.02 193.04 0) (unit 1)
     (in_bom yes) (on_board yes) (fields_autoplaced)
-    (property "Reference" "Hs25" (id 0) (at 162.56 192.2053 0)
+    (property "Reference" "Hs26" (id 0) (at 162.56 192.2053 0)
       (effects (font (size 1.27 1.27)) (justify left))
     )
@@
   (symbol (lib_name "MountingHoleSMD_1") (lib_id "giri:MountingHoleSMD") (at 147.32 186.69 0) (unit 1)
     (in_bom yes) (on_board yes) (fields_autoplaced)
-    (property "Reference" "Hs19" (id 0) (at 149.86 185.8553 0)
+    (property "Reference" "Hs20" (id 0) (at 149.86 185.8553 0)
       (effects (font (size 1.27 1.27)) (justify left))
     )
@@
   (symbol (lib_name "MountingHoleSMD_1") (lib_id "giri:MountingHoleSMD") (at 153.67 193.04 0) (unit 1)
     (in_bom yes) (on_board yes) (fields_autoplaced)
-    (property "Reference" "Hs24" (id 0) (at 156.21 192.2053 0)
+    (property "Reference" "Hs25" (id 0) (at 156.21 192.2053 0)
       (effects (font (size 1.27 1.27)) (justify left))
     )
@@
     (pin "2")
   )
+  (symbol (lib_name "MountingHoleSMD_1") (lib_id "giri:MountingHoleSMD") (at 153.67 180.34 0) (unit 1)
+    (in_bom yes) (on_board yes) (fields_autoplaced)
+    (property "Reference" "Hs18" (id 0) (at 156.21 179.5053 0)
+      (effects (font (size 1.27 1.27)) (justify left))
+    )
+    (property "Value" "M2" (id 1) (at 156.21 182.0422 0)
+      (effects (font (size 1.27 1.27)) (justify left))
+    )
+    (property "Footprint" "giri:SMTSO_M2" (id 2) (at 153.67 180.34 0)
+      (effects (font (size 1.27 1.27)) hide)
+    )
+    (property "Datasheet" "~" (id 3) (at 153.67 180.34 0)
+      (effects (font (size 1.27 1.27)) hide)
+    )
+  )
   (symbol (lib_id "giri:OSw") (at 139.7 87.63 0) (unit 1)
     (in_bom yes) (on_board yes) (fields_autoplaced)
@@
   (symbol (lib_name "MountingHoleSMD_1") (lib_id "giri:MountingHoleSMD") (at 147.32 193.04 0) (unit 1)
     (in_bom yes) (on_board yes) (fields_autoplaced)
-    (property "Reference" "Hs23" (id 0) (at 149.86 192.2053 0)
+    (property "Reference" "Hs24" (id 0) (at 149.86 192.2053 0)
       (effects (font (size 1.27 1.27)) (justify left))
     )
@@
   (symbol (lib_name "MountingHoleSMD_1") (lib_id "giri:MountingHoleSMD") (at 153.67 186.69 0) (unit 1)
     (in_bom yes) (on_board yes) (fields_autoplaced)
-    (property "Reference" "Hs20" (id 0) (at 156.21 185.8553 0)
+    (property "Reference" "Hs21" (id 0) (at 156.21 185.8553 0)
       (effects (font (size 1.27 1.27)) (justify left))
     )
@@
       (reference "Hs17") (unit 1) (value "M2") (footprint "giri:SMTSO_M2")
     )
-    (path "/05f1735a-09dd-4080-94fd-8289ece55224"
+    (path "/cf27c8b0-03e3-4a38-874c-67ce991ac925"
       (reference "Hs18") (unit 1) (value "M2") (footprint "giri:SMTSO_M2")
     )
-    (path "/90526b54-8115-4651-9951-dea3a70d3eeb"
+    (path "/05f1735a-09dd-4080-94fd-8289ece55224"
       (reference "Hs19") (unit 1) (value "M2") (footprint "giri:SMTSO_M2")
     )
-    (path "/f6f1b343-d5d5-44d9-b160-7d2cc37caad3"
+    (path "/90526b54-8115-4651-9951-dea3a70d3eeb"
       (reference "Hs20") (unit 1) (value "M2") (footprint "giri:SMTSO_M2")
     )
-    (path "/3cb06765-d332-474e-8aee-88c0309c35ff"
+    (path "/f6f1b343-d5d5-44d9-b160-7d2cc37caad3"
       (reference "Hs21") (unit 1) (value "M2") (footprint "giri:SMTSO_M2")
     )
-    (path "/4621ce48-0ccd-43dd-bfc6-dc3c8b0a3c23"
+    (path "/3cb06765-d332-474e-8aee-88c0309c35ff"
       (reference "Hs22") (unit 1) (value "M2") (footprint "giri:SMTSO_M2")
     )
-    (path "/e2ebdd70-17ed-4afe-8674-9342ddab4254"
+    (path "/4621ce48-0ccd-43dd-bfc6-dc3c8b0a3c23"
       (reference "Hs23") (unit 1) (value "M2") (footprint "giri:SMTSO_M2")
     )
-    (path "/ac7a7bd4-0f91-4292-97eb-963a2361760c"
+    (path "/e2ebdd70-17ed-4afe-8674-9342ddab4254"
       (reference "Hs24") (unit 1) (value "M2") (footprint "giri:SMTSO_M2")
     )
-    (path "/638a5d8c-dfd0-4eeb-bac8-a6b2bb8852ea"
+    (path "/ac7a7bd4-0f91-4292-97eb-963a2361760c"
       (reference "Hs25") (unit 1) (value "M2") (footprint "giri:SMTSO_M2")
     )
+    (path "/638a5d8c-dfd0-4eeb-bac8-a6b2bb8852ea"
+      (reference "Hs26") (unit 1) (value "M2") (footprint "giri:SMTSO_M2")
+    )
     (path "/c6ce5191-7729-4f5b-9b94-cb2590b41d91"

Commit message: add tracks
M  Giri_Library.kicad_sym
M  Giri_Library.pretty/Keychron_Optical_Switch_1u.kicad_mod
A  lopro/pcb/LED-Driver.kicad_sch
M  lopro/pcb/pcb.kicad_pcb
M  lopro/pcb/pcb.kicad_sch
M  lopro/place_fp.py
Parts:
- added C1, C2: 10uF, Capacitor_SMD:C_1206_3216Metric, symbol Device:C_Small
- added C3, C4: 100nF, Capacitor_SMD:C_0603_1608Metric, symbol Device:C_Small
- added D1, D10, D11, D12, D13, D14, D15, D16, D17, D18, D19, D2, D20, D21, D22, D23, D24, D25, D26, D27, D28, D29, D3, D30, D31, D32, D33, D34, D35, D36, D37, D38, D39, D4, D40, D41, D42, D43, D44, D45, D46, D47, D48, D49, D5, D50, D51, D52, D53, D54, D55, D56, D57, D58, D59, D6, D60, D61, D62, D63, D64, D65, D66, D67, D68, D69, D7, D70, D71, D72, D8, D9: LED, LED_SMD:LED_0603_1608Metric_Pad1.05x0.95mm_HandSolder, symbol Device:LED
- added R25, R26, R27, R28, R29, R30: 20k, Resistor_SMD:R_0603_1608Metric, symbol Device:R_Small
- added U1: IS31FL3731-QF, Package_DFN_QFN:QFN-28-1EP_4x4mm_P0.4mm_EP2.3x2.3mm, symbol Driver_LED:IS31FL3731-QF
- J1: footprint Connector:GB042-34S-H10 -> Connector_Dsub:DSUB-37_Female_Horizontal_P2.77x2.84mm_EdgePinOffset4.94mm_Housed_MountingHolesOffset7.48mm
Connections:
- net +3V3: now also C1.2, C2.2, C3.2, R25.1, R26.1, R27.1, R28.1, U1.2 (VCC)
- net GND: now also C1.1, C2.1, C3.1, C4.1, R29.2, R30.2, U1.29 (GND), U1.5 (GND)
- new net AD: R30.1, U1.18 (AD)
- new net CA1: D1.1 (K), D16.2 (A), D2.1 (K), D3.1 (K), D30.2 (A), D4.1 (K), D45.2 (A), D5.1 (K), D59.2 (A), D6.1 (K), D7.1 (K), D8.1 (K), U1.21 (CA1)
- new net CA2: D1.2 (A), D16.1 (K), D17.1 (K), D18.1 (K), D19.1 (K), D20.1 (K), D21.1 (K), D22.1 (K), D23.1 (K), D31.2 (A), D46.2 (A), D60.2 (A), U1.22 (CA2)
- new net CA3: D17.2 (A), D2.2 (A), D30.1 (K), D31.1 (K), D32.1 (K), D33.1 (K), D34.1 (K), D35.1 (K), D36.1 (K), D37.1 (K), D47.2 (A), D61.2 (A), U1.23 (CA3)
- new net CA4: D18.2 (A), D3.2 (A), D32.2 (A), D45.1 (K), D46.1 (K), D47.1 (K), D48.1 (K), D49.1 (K), D50.1 (K), D51.1 (K), D52.1 (K), D62.2 (A), U1.24 (CA4)
- new net CA5: D19.2 (A), D33.2 (A), D4.2 (A), D48.2 (A), D59.1 (K), D60.1 (K), D61.1 (K), D62.1 (K), D63.1 (K), D64.1 (K), D65.1 (K), D66.1 (K), U1.25 (CA5)
- new net CA6: D20.2 (A), D34.2 (A), D49.2 (A), D5.2 (A), D63.2 (A), U1.26 (CA6)
- new net CA7: D21.2 (A), D35.2 (A), D50.2 (A), D6.2 (A), D64.2 (A), U1.27 (CA7)
- new net CA8: D22.2 (A), D36.2 (A), D51.2 (A), D65.2 (A), D7.2 (A), U1.28 (CA8)
- new net CA9: D23.2 (A), D37.2 (A), D52.2 (A), D66.2 (A), D8.2 (A), U1.1 (CA9)
- new net CB1: D10.1 (K), D11.1 (K), D12.1 (K), D13.1 (K), D14.1 (K), D15.1 (K), D24.2 (A), D38.2 (A), D53.2 (A), D67.2 (A), D9.1 (K), U1.7 (CB1)
- new net CB2: D24.1 (K), D25.1 (K), D26.1 (K), D27.1 (K), D28.1 (K), D29.1 (K), D39.2 (A), D54.2 (A), D68.2 (A), D9.2 (A), U1.8 (CB2)
- new net CB3: D10.2 (A), D25.2 (A), D38.1 (K), D39.1 (K), D40.1 (K), D41.1 (K), D42.1 (K), D43.1 (K), D44.1 (K), D55.2 (A), D69.2 (A), U1.9 (CB3)
- new net CB4: D11.2 (A), D26.2 (A), D40.2 (A), D53.1 (K), D54.1 (K), D55.1 (K), D56.1 (K), D57.1 (K), D58.1 (K), D70.2 (A), U1.10 (CB4)
- new net CB5: D12.2 (A), D27.2 (A), D41.2 (A), D56.2 (A), D67.1 (K), D68.1 (K), D69.1 (K), D70.1 (K), D71.1 (K), D72.1 (K), U1.11 (CB5)
- new net CB6: D13.2 (A), D28.2 (A), D42.2 (A), D57.2 (A), D71.2 (A), U1.12 (CB6)
- new net CB7: D14.2 (A), D29.2 (A), D43.2 (A), D58.2 (A), D72.2 (A), U1.13 (CB7)
- new net CB8: D15.2 (A), D44.2 (A), U1.14 (CB8)
- new net C_FLT: C4.2, U1.16 (C_FILT)
- new net R_EXT: R29.1, U1.6 (R_EXT)
- new net SCL: J1.35 (GPIO1), R26.2, U1.20 (SCL)
- new net SDA: J1.36 (GPIO2), R25.2, U1.19 (SDA)
- new net ~{INTB}: R27.2, U1.4 (~{INTB})
- new net ~{SDB}: R28.2, U1.3 (~{SDB})
- no-connect marks 24 -> 28
Other:
- note added: "Dummy Conn"
- note added: "Filter / VCC Cap"
- note added: "Holes"
- note added: "LED Driver"
- note added: "LEDs"
- note added: "MCU Conn"
- note added: "Pull up / down"
- note added: "Switch Matrix"
- moved on the sheet: Hs1, Hs10, Hs11, Hs12, Hs13, Hs14, Hs15, Hs16, Hs17, Hs18, Hs19, Hs2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
