File: lopro/6rows/pcb/pcb.kicad_sch (KiCad schematic)
At the start: 209 parts, among them J1 PCB_Lopro_Conn, J2 Conn_01x08_Female, J3 Conn_01x08_Female, J4 Conn_01x08_Female, U1 IS31FL3731-QF

Commit message: Added new keyboard
D  .DS_Store
A  giri-kicad-lib/.gitignore
R  Giri_Library.kicad_sym -> giri-kicad-lib/switches.kicad_sym
A  giri-kicad-lib/switches_lib.pretty/C_0402_1005Metric.kicad_mod
A  giri-kicad-lib/switches_lib.pretty/C_0603_1608Metric.kicad_mod
A  giri-kicad-lib/switches_lib.pretty/C_1206_3216Metric.kicad_mod
A  giri-kicad-lib/switches_lib.pretty/Keychron_Optical_Switch_1u.kicad_mod
R  Giri_Library.pretty/Keychron_Optical_Switch_1u.kicad_mod -> giri-kicad-lib/switches_lib.pretty/Keychron_Optical_Switch_R_1u.kicad_mod
A  giri-kicad-lib/switches_lib.pretty/LED_0603_1608Metric_Pad1.05x0.95mm_HandSolder.kicad_mod
A  giri-kicad-lib/switches_lib.pretty/MountingHole_1.7mm_M1.6_Pad.kicad_mod
A  giri-kicad-lib/switches_lib.pretty/MountingHole_2.2mm_M2_ISO7380_Pad.kicad_mod
A  giri-kicad-lib/switches_lib.pretty/Pad_Only_SMTSO_M2.kicad_mod
A  giri-kicad-lib/switches_lib.pretty/PinHeader_1x03_P2.54mm_Vertical.kicad_mod
A  giri-kicad-lib/switches_lib.pretty/R_0402_1005Metric.kicad_mod
A  giri-kicad-lib/switches_lib.pretty/R_0603_1608Metric_Pad0.98x0.95mm_HandSolder.kicad_mod
A  giri-kicad-lib/switches_lib.pretty/SMTSO_M1.6.kicad_mod
R  Giri_Library.pretty/SMTSO_M2.kicad_mod -> giri-kicad-lib/switches_lib.pretty/SMTSO_M2.kicad_mod
R  Giri_Library.pretty/Switch_Cutout_LoPro.kicad_mod -> giri-kicad-lib/switches_lib.pretty/Switch_Cutout_LoPro.kicad_mod
R  Giri_Library.pretty/Switch_Cutout_LoPro_2.25u_Faulty.kicad_mod -> giri-kicad-lib/switches_lib.pretty/Switch_Cutout_LoPro_2.25u_Faulty.kicad_mod
R  Giri_Library.pretty/Switch_Cutout_MX.kicad_mod -> giri-kicad-lib/switches_lib.pretty/Switch_Cutout_MX.kicad_mod
D  lopro/6banks/pcb/pcb.kicad_sch
R  lopro/6banks/drawborderk.py -> lopro/6rows/drawborderk.py
R  lopro/6banks/pcb/.gitignore -> lopro/6rows/pcb/.gitignore
R  lopro/6banks/pcb/LED-Driver.kicad_sch -> lopro/6rows/pcb/LED-Driver.kicad_sch
R  lopro/6banks/pcb/fp-lib-table -> lopro/6rows/pcb/fp-lib-table
R  lopro/6banks/pcb/pcb.kicad_pcb -> lopro/6rows/pcb/pcb.kicad_pcb
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
Parts:
- added C? (x2): 10uF, Capacitor_SMD:C_0603_1608Metric, symbol Device:C_Small
- added C? (x2): 100nF, Capacitor_SMD:C_0402_1005Metric, symbol rdzen:1_CAP
- added R? (x6): 20k, Resistor_SMD:R_0402_1005Metric, symbol Device:R_Small
- added R?: 0R, Resistor_SMD:R_0402_1005Metric_Pad0.72x0.64mm_HandSolder, symbol Device:R_Small
- added U?: IS31FL3731-QF, Package_DFN_QFN:QFN-28-1EP_4x4mm_P0.4mm_EP2.3x2.3mm, symbol Driver_LED:IS31FL3731-QF
Connections:
- net +3V3: now also C?.2, C?.2, C?.2, R?.1, R?.1, R?.1, R?.1, R?.1, U?.2 (VCC)
- net AD: now also R?.1, U?.18 (AD)
- net CA1: now also U?.21 (CA1)
- net CA2: now also U?.22 (CA2)
- net CA3: now also U?.23 (CA3)
- net CA4: now also U?.24 (CA4)
- net CA5: now also U?.25 (CA5)
- net CA6: now also U?.26 (CA6)
- net CA7: now also U?.27 (CA7)
- net CA8: now also U?.28 (CA8)
- net CA9: now also U?.1 (CA9)
- net CB1: now also U?.7 (CB1)
- net CB2: now also U?.8 (CB2)
- net CB3: now also U?.9 (CB3)
- net CB4: now also U?.10 (CB4)
- net CB5: now also U?.11 (CB5)
- net CB6: now also U?.12 (CB6)
- net CB7: now also U?.13 (CB7)
- net CB8: now also U?.14 (CB8)
- net C_FLT: now also C?.2, U?.16 (C_FILT)
- net GND: now also C?.1, C?.1, C?.1, C?.1, R?.2, R?.2, U?.29 (GND), U?.5 (GND)
- net R_EXT: now also R?.1, U?.6 (R_EXT)
- net SCL: now also R?.2, U?.20 (SCL)
- net SDA: now also R?.2, U?.19 (SDA)
- net ~{INTB}: now also R?.2, U?.4 (~{INTB})
- net ~{SDB}: now also R?.2, U?.3 (~{SDB})
- new net CB9: U?.15 (CB9)
- new net PP5000_VIN: R?.2
- no-connect marks 28 -> 29
