File: lopro/8rows/pcb/pcb.kicad_sch (KiCad schematic)
At the start: 265 parts, among them J1 Conn_01x03, J2 Conn_01x03, J3 Conn_01x03

Commit message: Add images
M  lopro/8rows/drawborder8b.py
A  lopro/8rows/pcb/pcb-b.png
A  lopro/8rows/pcb/pcb-f.png
M  lopro/8rows/pcb/pcb.kicad_pcb
M  lopro/8rows/pcb/pcb.kicad_sch
Parts:
- renumbered R7 to R6, R8 to R7, R9 to R8, R6 to R9
Changed lines of the file:
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@@
   (symbol (lib_id "Device:R_Small") (at 110.49 33.02 90) (unit 1)
     (in_bom yes) (on_board yes)
-    (property "Reference" "R7" (id 0) (at 114.3 31.75 90))
+    (property "Reference" "R6" (id 0) (at 114.3 31.75 90))
     (property "Value" "R_Small" (id 1) (at 110.49 31.1205 90)
       (effects (font (size 1.27 1.27)) hide)
@@
   (symbol (lib_id "Device:R_Small") (at 143.51 33.02 90) (unit 1)
     (in_bom yes) (on_board yes)
-    (property "Reference" "R9" (id 0) (at 147.32 31.75 90))
+    (property "Reference" "R8" (id 0) (at 147.32 31.75 90))
     (property "Value" "R_Small" (id 1) (at 143.51 31.1205 90)
       (effects (font (size 1.27 1.27)) hide)
@@
   (symbol (lib_id "Device:R_Small") (at 127 33.02 90) (unit 1)
     (in_bom yes) (on_board yes)
-    (property "Reference" "R8" (id 0) (at 130.81 31.75 90))
+    (property "Reference" "R7" (id 0) (at 130.81 31.75 90))
     (property "Value" "R_Small" (id 1) (at 127 31.1205 90)
       (effects (font (size 1.27 1.27)) hide)
@@
   (symbol (lib_id "Device:R_Small") (at 160.02 33.02 90) (unit 1)
     (in_bom yes) (on_board yes)
-    (property "Reference" "R6" (id 0) (at 163.83 31.75 90))
+    (property "Reference" "R9" (id 0) (at 163.83 31.75 90))
     (property "Value" "R_Small" (id 1) (at 160.02 31.1205 90)
       (effects (font (size 1.27 1.27)) hide)
@@
       (reference "R5") (unit 1) (value "R_Small") (footprint "giri:R_0603_1608Metric_Pad0.98x0.95mm_HandSolder")
     )
-    (path "/a2eb7068-3655-4878-9609-210ec312df4f"
+    (path "/42ef8d69-8f2d-4172-8a20-2e1e6ecccbb7"
       (reference "R6") (unit 1) (value "R_Small") (footprint "giri:R_0603_1608Metric_Pad0.98x0.95mm_HandSolder")
     )
-    (path "/42ef8d69-8f2d-4172-8a20-2e1e6ecccbb7"
+    (path "/99523b99-c6fb-4e51-b856-0bceee8d75cf"
       (reference "R7") (unit 1) (value "R_Small") (footprint "giri:R_0603_1608Metric_Pad0.98x0.95mm_HandSolder")
     )
-    (path "/99523b99-c6fb-4e51-b856-0bceee8d75cf"
+    (path "/897913f2-9485-4368-ba0a-fa043d4c69bd"
       (reference "R8") (unit 1) (value "R_Small") (footprint "giri:R_0603_1608Metric_Pad0.98x0.95mm_HandSolder")
     )
-    (path "/897913f2-9485-4368-ba0a-fa043d4c69bd"
+    (path "/a2eb7068-3655-4878-9609-210ec312df4f"
       (reference "R9") (unit 1) (value "R_Small") (footprint "giri:R_0603_1608Metric_Pad0.98x0.95mm_HandSolder")
     )
