File: lopro/8rows/pcb/pcb.kicad_pcb (KiCad board)
At the start: 2 copper layers, 309.5 x 188.8 mm, 265 parts, among them J1 Conn_01x03, J2 Conn_01x03, J3 Conn_01x03

Commit message: Add images
M  lopro/8rows/drawborder8b.py
A  lopro/8rows/pcb/pcb-b.png
A  lopro/8rows/pcb/pcb-f.png
M  lopro/8rows/pcb/pcb.kicad_pcb
M  lopro/8rows/pcb/pcb.kicad_sch
Parts:
- moved Hs19 1.41 mm to (67.2, 120.0)
- moved Hs20 1.41 mm to (67.2, 172.0)
- moved Hs21 1.41 mm to (-7.75, 172.0)
- moved Hs22 1.41 mm to (-7.75, 120.0)
- moved Hs23 1.41 mm to (283.2, 120.0)
- moved Hs24 1.41 mm to (283.2, 172.0)
- moved Hs25 1.41 mm to (208.2, 172.0)
- moved Hs26 1.41 mm to (208.2, 120.0)
Changed lines of the file:
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@@
   )
   (footprint "giri:SMTSO_M2" (layer "F.Cu")
-    (at 68.25 119.025)
+    (at 67.25 120.025)
     (descr "Mounting Hole 2.2mm, M2")
     (tags "mounting hole 2.2mm m2")
@@
   )
   (footprint "giri:SMTSO_M2" (layer "F.Cu")
-    (at 68.25 173.025)
+    (at 67.25 172.025)
     (descr "Mounting Hole 2.2mm, M2")
     (tags "mounting hole 2.2mm m2")
@@
   )
   (footprint "giri:SMTSO_M2" (layer "F.Cu")
-    (at 207.25 119.025)
+    (at 208.25 120.025)
     (descr "Mounting Hole 2.2mm, M2")
     (tags "mounting hole 2.2mm m2")
@@
   )
   (footprint "giri:SMTSO_M2" (layer "F.Cu")
-    (at 207.25 173.025)
+    (at 208.25 172.025)
     (descr "Mounting Hole 2.2mm, M2")
     (tags "mounting hole 2.2mm m2")
@@
   )
   (footprint "giri:SMTSO_M2" (layer "F.Cu")
-    (at 284.25 119.025)
+    (at 283.25 120.025)
     (descr "Mounting Hole 2.2mm, M2")
     (tags "mounting hole 2.2mm m2")
@@
   )
   (footprint "giri:SMTSO_M2" (layer "F.Cu")
-    (at -8.75 119.025)
+    (at -7.75 120.025)
     (descr "Mounting Hole 2.2mm, M2")
     (tags "mounting hole 2.2mm m2")
@@
   )
   (footprint "giri:SMTSO_M2" (layer "F.Cu")
-    (at -8.75 173.025)
+    (at -7.75 172.025)
     (descr "Mounting Hole 2.2mm, M2")
     (tags "mounting hole 2.2mm m2")
@@
   )
   (footprint "giri:SMTSO_M2" (layer "F.Cu")
-    (at 284.25 173.025)
+    (at 283.25 172.025)
     (descr "Mounting Hole 2.2mm, M2")
     (tags "mounting hole 2.2mm m2")
