File: lopro/8rows/pcb/pcb.kicad_pcb (KiCad board)
At the start: 2 copper layers, 309.5 x 188.8 mm, 265 parts, among them J1 Conn_01x03, J2 Conn_01x03, J3 Conn_01x03

Commit message: add tracks
M  giri-kicad-lib/switches.kicad_sym
A  giri-kicad-lib/switches_lib.pretty/JLC_Order_Num.kicad_mod
A  lopro/8rows/border8r.py
M  lopro/8rows/pcb/pcb.kicad_pcb
M  lopro/8rows/pcb/pcb.kicad_prl
M  lopro/8rows/pcb/pcb.kicad_pro
M  lopro/8rows/pcb/pcb.kicad_sch
A  lopro/8rows/pickle8r.py
A  lopro/8rows/place8r.py
R  lopro/8rows/drawborder8b.py -> lopro/bak/8rows-v0/drawborder8b.py
A  lopro/bak/8rows-v0/pcb/.gitignore
A  lopro/bak/8rows-v0/pcb/LED-Driver.kicad_sch
A  lopro/bak/8rows-v0/pcb/fp-lib-table
A  lopro/bak/8rows-v0/pcb/jlcpcb/gerbers/pcb-B_Cu.gbl
A  lopro/bak/8rows-v0/pcb/jlcpcb/gerbers/pcb-B_Mask.gbs
A  lopro/bak/8rows-v0/pcb/jlcpcb/gerbers/pcb-B_Paste.gbp
A  lopro/bak/8rows-v0/pcb/jlcpcb/gerbers/pcb-B_Silkscreen.gbo
A  lopro/bak/8rows-v0/pcb/jlcpcb/gerbers/pcb-Edge_Cuts.gm1
A  lopro/bak/8rows-v0/pcb/jlcpcb/gerbers/pcb-F_Cu.gtl
A  lopro/bak/8rows-v0/pcb/jlcpcb/gerbers/pcb-F_Mask.gts
A  lopro/bak/8rows-v0/pcb/jlcpcb/gerbers/pcb-F_Paste.gtp
A  lopro/bak/8rows-v0/pcb/jlcpcb/gerbers/pcb-F_Silkscreen.gto
A  lopro/bak/8rows-v0/pcb/jlcpcb/gerbers/pcb-NPTH-drl_map.gbr
A  lopro/bak/8rows-v0/pcb/jlcpcb/gerbers/pcb-NPTH.drl
A  lopro/bak/8rows-v0/pcb/jlcpcb/gerbers/pcb-PTH-drl_map.gbr
A  lopro/bak/8rows-v0/pcb/jlcpcb/gerbers/pcb-PTH.drl
A  lopro/bak/8rows-v0/pcb/pcb-b.png
A  lopro/bak/8rows-v0/pcb/pcb-f.png
A  lopro/bak/8rows-v0/pcb/pcb.kicad_pcb
A  lopro/bak/8rows-v0/pcb/pcb.kicad_prl
A  lopro/bak/8rows-v0/pcb/pcb.kicad_pro
A  lopro/bak/8rows-v0/pcb/pcb.kicad_sch
A  lopro/bak/8rows-v0/pcb/sym-lib-table
R  lopro/8rows/placefp8b.py -> lopro/bak/8rows-v0/placefp8b.py
A  lopro/bak/8rows-v0/switch-plate/.gitignore
A  lopro/bak/8rows-v0/switch-plate/fp-lib-table
A  lopro/bak/8rows-v0/switch-plate/switch-plate.kicad_pcb
A  lopro/bak/8rows-v0/switch-plate/switch-plate.kicad_prl
A  lopro/bak/8rows-v0/switch-plate/switch-plate.kicad_pro
A  lopro/bak/8rows-v0/switch-plate/switch-plate.kicad_sch
A  lopro/bak/8rows-v0/switch-plate/sym-lib-table
A  lopro/bak/8rows-v0/wrist-s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
Parts:
- removed Hs26: M2, giri:SMTSO_M2
- removed MOD1: Conn_rp2040_v1_module_Outline, RP2040_Minimal:Module_Conn_Regular_Outline
- removed MOD2: LED_Driver_Module_Conn, RP2040_Minimal:LED_Driver_Mod_Conn
- removed R15, R16, R17, R18: R_Small, giri:R_0603_1608Metric_Pad0.98x0.95mm_HandSolder
- added C1: 10uF, RP2040_Minimal:C_1206_3216Metric, F.Cu at (158.9, 79.8)
- added C10: 100nF, RP2040_Minimal:C_0603_1608Metric_Pad1.08x0.95mm_HandSolder, F.Cu at (114.0, 80.0)
- added C11: 100nF, RP2040_Minimal:C_0603_1608Metric_Pad1.08x0.95mm_HandSolder, F.Cu at (119.5, 81.3)
- added C12: 100nF, RP2040_Minimal:C_0603_1608Metric_Pad1.08x0.95mm_HandSolder, F.Cu at (124.9, 73.2)
- added C13: 100nF, RP2040_Minimal:C_0603_1608Metric_Pad1.08x0.95mm_HandSolder, F.Cu at (122.7, 66.1)
- added C14: 2.2uF, RP2040_Minimal:C_0603_1608Metric_Pad1.08x0.95mm_HandSolder, F.Cu at (9.85, 13.0)
- added C15: 1uF, RP2040_Minimal:C_0603_1608Metric_Pad1.08x0.95mm_HandSolder, F.Cu at (109.5, 69.6)
- added C16: 1uF, RP2040_Minimal:C_0603_1608Metric_Pad1.08x0.95mm_HandSolder, F.Cu at (112.0, 68.7)
- added C17: 10uF, RP2040_Minimal:C_0603_1608Metric_Pad1.08x0.95mm_HandSolder, F.Cu at (105.8, 66.7)
- added C18: 2.2uF, RP2040_Minimal:C_0603_1608Metric_Pad1.08x0.95mm_HandSolder, F.Cu at (7.70, 25.4)
- added C19: 1uF, RP2040_Minimal:C_0603_1608Metric_Pad1.08x0.95mm_HandSolder, F.Cu at (13.4, 23.3)
- added C2: 10uF, RP2040_Minimal:C_0603_1608Metric_Pad1.08x0.95mm_HandSolder, F.Cu at (162.6, 79.6)
- added C20: 100nF, RP2040_Minimal:C_0603_1608Metric_Pad1.08x0.95mm_HandSolder, F.Cu at (105.8, 78.0)
- added C21: 2.2uF, RP2040_Minimal:C_0603_1608Metric_Pad1.08x0.95mm_HandSolder, F.Cu at (105.8, 79.6)
- added C22: 15pF, RP2040_Minimal:C_0603_1608Metric_Pad1.08x0.95mm_HandSolder, F.Cu at (127.6, 80.0)
- added C23: 15pF, RP2040_Minimal:C_0603_1608Metric_Pad1.08x0.95mm_HandSolder, F.Cu at (127.6, 76.6)
- added C3: 100nF, RP2040_Minimal:C_0603_1608Metric_Pad1.08x0.95mm_HandSolder, F.Cu at (161.0, 79.6)
- added C4: 100nF, RP2040_Minimal:C_0603_1608Metric_Pad1.08x0.95mm_HandSolder, F.Cu at (168.6, 70.0)
- added C5: 100nF, RP2040_Minimal:C_0603_1608Metric_Pad1.08x0.95mm_HandSolder, F.Cu at (109.0, 76.0)
- added C6: 100nF, RP2040_Minimal:C_0603_1608Metric_Pad1.08x0.95mm_HandSolder, F.Cu at (125.8, 71.6)
- added C7: 100nF, RP2040_Minimal:C_0603_1608Metric_Pad1.08x0.95mm_HandSolder, F.Cu at (109.0, 74.5)
- added C8: 100nF, RP2040_Minimal:C_0603_1608Metric_Pad1.08x0.95mm_HandSolder, F.Cu at (111.0, 66.2)
- added C9: 100nF, RP2040_Minimal:C_0603_1608Metric_Pad1.08x0.95mm_HandSolder, F.Cu at (114.2, 67.1)
- added J4: Conn_01x03, giri:PinHeader_1x03_P2.54mm_Vertical, F.Cu at (45.0, -8.40)
- added JLC1: JLC_Order_Num, giri:JLC_Order_Num, F.Cu at (245.7, 119.9)
- added Q1: Q_NMOS_DGS, RP2040_Minimal:Diodes_U_DFN1212_3_Handsolder, F.Cu at (179.2, 3.20)
- added Q2: Q_NMOS_DGS, RP2040_Minimal:Diodes_U_DFN1212_3_Handsolder, F.Cu at (188.7, 22.2)
- added Q3: Q_NMOS_DGS, RP2040_Minimal:Diodes_U_DFN1212_3_Handsolder, F.Cu at (174.4, 41.2)
- added Q4: Q_NMOS_DGS, RP2040_Minimal:Diodes_U_DFN1212_3_Handsolder, F.Cu at (183.9, 60.2)
- added Q5: Q_NMOS_DGS, RP2040_Minimal:Diodes_U_DFN1212_3_Handsolder, F.Cu at (60.5, 79.2)
- added Q6: Q_NMOS_DGS, RP2040_Minimal:Diodes_U_DFN1212_3_Handsolder, F.Cu at (231.4, 79.2)
- added Q7: Q_NMOS_DGS, RP2040_Minimal:Diodes_U_DFN1212_3_Handsolder, F.Cu at (193.4, 41.2)
- added Q8: Q_NMOS_DGS, RP2040_Minimal:Diodes_U_DFN1212_3_Handsolder, F.Cu at (198.2, 3.20)
- added Rgr1: 160R, Resistor_SMD:R_0603_1608Metric_Pad0.98x0.95mm_HandSolder, F.Cu at (179.2, 6.20)
- added Rgr2: 160R, Resistor_SMD:R_0603_1608Metric_Pad0.98x0.95mm_HandSolder, F.Cu at (188.7, 25.2)
- added Rgr3: 160R, Resistor_SMD:R_0603_1608Metric_Pad0.98x0.95mm_HandSolder, F.Cu at (174.4, 44.2)
- added Rgr4: 160R, Resistor_SMD:R_0603_1608Metric_Pad0.98x0.95mm_HandSolder, F.Cu at (183.9, 63.2)
- added Rgr5: 160R, Resistor_SMD:R_0603_1608Metric_Pad0.98x0.95mm_HandSolder, F.Cu at (60.5, 82.2)
- added Rgr6: 160R, Resistor_SMD:R_0603_1608Metric_Pad0.98x0.95mm_HandSolder, F.Cu at (231.4, 82.2)
- added Rgr7: 160R, Resistor_SMD:R_0603_1608Metric_Pad0.98x0.95mm_HandSolder, F.Cu at (193.4, 44.2)
- added Rgr8: 160R, Resistor_SMD:R_0603_1608Metric_Pad0.98x0.95mm_HandSolder, F.Cu at (198.2, 6.20)
- added Rpt1: Rpt, giri:R_0603_1608Metric_Pad0.98x0.95mm_HandSolder, F.Cu at (15.8, 21.2)
- added Rpt10: Rpt, giri:R_0603_1608Metric_Pad0.98x0.95mm_HandSolder, F.Cu at (182.0, 2.20)
- added Rpt11: Rpt, giri:R_0603_1608Metric_Pad0.98x0.95mm_HandSolder, F.Cu at (201.0, 2.20)
- added Rpt12: Rpt, giri:R_0603_1608Metric_Pad0.98x0.95mm_HandSolder, F.Cu at (220.0, 2.20)
- added Rpt13: Rpt, giri:R_0603_1608Metric_Pad0.98x0.95mm_HandSolder, F.Cu at (239.0, 2.20)
- added Rpt14: Rpt, giri:R_0603_1608Metric_Pad0.98x0.95mm_HandSolder, F.Cu at (258.0, 2.20)
- added Rpt15: Rpt, giri:R_0603_1608Metric_Pad0.98x0.95mm_HandSolder, F.Cu at (277.0, 2.20)
- added Rpt16: Rpt, giri:R_0603_1608Metric_Pad0.98x0.95mm_HandSolder, F.Cu at (229.5, 21.2)
- added Rpt17: Rpt, giri:R_0603_1608Metric_Pad0.98x0.95mm_HandSolder, F.Cu at (210.5, 21.2)
- added Rpt18: Rpt, giri:R_0603_1608Metric_Pad0.98x0.95mm_HandSolder, F.Cu at (191.5, 21.2)
- added Rpt2: Rpt, giri:R_0603_1608Metric_Pad0.98x0.95mm_HandSolder, F.Cu at (39.5, 21.2)
- added Rpt3: Rpt, giri:R_0603_1608Metric_Pad0.98x0.95mm_HandSolder, F.Cu at (58.5, 21.2)
- added Rpt4: Rpt, giri:R_0603_1608Metric_Pad0.98x0.95mm_HandSolder, F.Cu at (77.5, 21.2)
- added Rpt5: Rpt, giri:R_0603_1608Metric_Pad0.98x0.95mm_HandSolder, F.Cu at (96.5, 21.2)
- added Rpt6: Rpt, giri:R_0603_1608Metric_Pad0.98x0.95mm_HandSolder, F.Cu at (115.5, 21.2)
- added Rpt7: Rpt, giri:R_0603_1608Metric_Pad0.98x0.95mm_HandSolder, F.Cu at (134.5, 21.2)
- added Rpt8: Rpt, giri:R_0603_1608Metric_Pad0.98x0.95mm_HandSolder, F.Cu at (153.5, 21.2)
- added Rpt9: Rpt, giri:R_0603_1608Metric_Pad0.98x0.95mm_HandSolder, F.Cu at (172.5, 21.2)
- added SW1: SW_DIP_x01_XKB_TS_2030, RP2040_Minimal:SW_CK_KXT3, F.Cu at (151.8, 73.8)
- added SW2: SW_DIP_x01_XKB_TS_2030, RP2040_Minimal:SW_CK_KXT3, F.Cu at (148.8, 73.8)
- added U1: IS31FL3731-QF, RP2040_Minimal:QFN-28-1EP_4x4mm_P0.4mm_EP2.3x2.3mm-Handsolder, F.Cu at (164.3, 74.5)
- added U2: NCP114ASN330T1G, Package_SO:TSOP-5_1.65x3.05mm_P0.95mm, F.Cu at (10.7, 25.2)
- added U3: RP2040, RP2040_Minimal:RP2040-QFN-56-Handsolder, F.Cu at (117.8, 73.4)
- added U4: Memory_Flash_W25Q64_XSON, RP2040_Minimal:8-USON-Handsolder, F.Cu at (109.3, 80.5)
- added X1: 12.000MHz, RP2040_Minimal:Crystal_SMD_2520-4Pin_2.5x2.0mm-Handsolder, F.Cu at (124.8, 77.9)
- Hs18: value M1.6 -> M2; footprint giri:SMTSO_M1.6 -> giri:SMTSO_M2
- J1: value Conn_01x03 -> U262-161N-4BVC11; footprint giri:PinHeader_1x03_P2.54mm_Vertical -> Connector_USB:USB_C_Receptacle_XKB_U262-16XN-4BVC11
- J3: moved to F.Cu
- R1, R2, R3: value R_Small -> 4.7k; footprint giri:R_0603_1608Metric_Pad0.98x0.95mm_HandSolder -> RP2040_Minimal:R_0603_1608Metric_Pad0.98x0.95mm_HandSolder
- R10, R7: value R_Small -> 27R; footprint giri:R_0603_1608Metric_Pad0.98x0.95mm_HandSolder -> RP2040_Minimal:R_0603_1608Metric_Pad0.98x0.95mm_HandSolder
- R11, R12: value R_Small -> 10k; footprint giri:R_0603_1608Metric_Pad0.98x0.95mm_HandSolder -> RP2040_Minimal:R_0603_1608Metric_Pad0.98x0.95mm_HandSolder
- R13, R14: value R_Small -> 1k; footprint giri:R_0603_1608Metric_Pad0.98x0.95mm_HandSolder -> RP2040_Minimal:R_0603_1608Metric_Pad0.98x0.95mm_HandSolder
- R4, R5, R6: value R_Small -> 20k; footprint giri:R_0603_1608Metric_Pad0.98x0.95mm_HandSolder -> RP2040_Minimal:R_0603_1608Metric_Pad0.98x0.95mm_HandSolder
- R8, R9: value R_Small -> 5.1k; footprint giri:R_0603_1608Metric_Pad0.98x0.95mm_HandSolder -> RP2040_Minimal:R_0603_1608Metric_Pad0.98x0.95mm_HandSolder
- moved Hs22 291.0 mm to (283.2, 120.0)
- moved Hs18 228.1 mm to (67.2, 120.0)
- moved R1 162.9 mm to (164.1, 69.3)
- moved R9 149.3 mm to (10.9, 15.9), turned to 0 degrees
- moved R2 140.5 mm to (162.6, 69.3)
- moved R14 132.8 mm to (125.1, 74.7), turned to 0 degrees
- moved R8 130.0 mm to (10.9, 18.9), turned to 0 degrees
- moved R3 128.0 mm to (165.7, 80.5), turned to 90 degrees
- moved R4 108.5 mm to (164.1, 79.9), turned to 90 degrees
- moved R5 94.9 mm to (168.3, 80.1)
- moved Hs15 91.3 mm to (232.8, 46.9)
- moved R13 90.9 mm to (148.4, 69.9)
- moved Hs17 81.0 mm to (291.8, 80.1)
- moved Hs20 75.0 mm to (-7.75, 172.0)
- moved Hs24 75.0 mm to (208.2, 172.0)
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Connections:
- D59 pad 1: CA5 -> CB7
- D59 pad 2: CA1 -> CB1
- D60 pad 1: CA5 -> CB7
- D60 pad 2: CA2 -> CB2
- D61 pad 1: CA5 -> CB7
- D61 pad 2: CA3 -> CB3
- D62 pad 1: CA5 -> CB7
- D62 pad 2: CA4 -> CB4
- D63 pad 1: CA5 -> CB6
- D63 pad 2: CA6 -> CB4
- D64 pad 1: CA5 -> CB6
- D64 pad 2: CA7 -> CB3
- D65 pad 1: CA5 -> CB6
- D65 pad 2: CA8 -> CB2
- D66 pad 1: CA5 -> CB6
- D66 pad 2: CA9 -> CB1
- R1 pad 1: /COL1A -> +3V3
- R1 pad 2: +3V3 -> SDA
- R10 pad 1: /COL1B -> Net-(R10-Pad1)
- R10 pad 2: +3V3 -> /USB_D-
- R11 pad 1: /COL2B -> +3V3
- R11 pad 2: +3V3 -> /RUN
- R12 pad 1: /COL3B -> +3V3
- R12 pad 2: +3V3 -> /QSPI_SS
- R13 pad 1: /COL4B -> /QSPI_SS
- R13 pad 2: +3V3 -> /~{USB_BOOT}
- R14 pad 1: /COL5B -> /XOUT
- R14 pad 2: +3V3 -> Net-(C22-Pad1)
- R2 pad 1: /COL2A -> +3V3
- R2 pad 2: +3V3 -> SCL
- R3 pad 1: /COL3A -> +3V3
- R3 pad 2: +3V3 -> /~{INTB}
- R4 pad 1: /COL4A -> +3V3
- R4 pad 2: +3V3 -> /~{SDB}
- R5 pad 1: /COL5A -> /R_EXT
- R5 pad 2: +3V3 -> GND
- R6 pad 1: /COL6A -> /AD
- R6 pad 2: +3V3 -> GND
- R7 pad 1: /COL7A -> Net-(R7-Pad1)
- R7 pad 2: +3V3 -> /USB_D+
- R8 pad 1: /COL8A -> Net-(J1-PadB5)
- R8 pad 2: +3V3 -> GND
- R9 pad 1: /COL9A -> Net-(J1-PadA5)
- R9 pad 2: +3V3 -> GND
Routing:
- net /COL8B: track 416.3 -> 245.1 mm, vias 9 -> 11
- net /USB_D+: track 0.00 -> 162.9 mm, vias 0 -> 2
- net /USB_D-: track 0.00 -> 160.8 mm
- net CB2: track 299.4 -> 453.9 mm, vias 7 -> 12
- net /INPUT1: track 148.2 -> 0.00 mm
- net /COL5B: track 474.3 -> 327.8 mm, vias 9 -> 7
- net /INPUT2: track 146.4 -> 0.00 mm
- net /ROW8: track 313.2 -> 167.2 mm, vias 3 -> 2
- net /INPUT3: track 144.7 -> 0.00 mm
- net CB3: track 315.3 -> 459.9 mm, vias 7 -> 12
- net /INPUT4: track 143.0 -> 0.00 mm
- net /P8: track 0.00 -> 142.3 mm, vias 0 -> 4
- net CB1: track 325.1 -> 467.4 mm, vias 6 -> 8
- net /INPUT8: track 142.0 -> 0.00 mm
- net /INPUT7: track 141.5 -> 0.00 mm
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Other:
- outline, holes or cut-outs redrawn

Commit message: enlarge center hole of keychron switch footprint
M  giri-kicad-lib/switches.kicad_sym
M  giri-kicad-lib/switches_lib.pretty/Keychron_Optical_Switch_1u.kicad_mod
M  giri-kicad-lib/switches_lib.pretty/Keychron_Optical_Switch_R_1u.kicad_mod
A  giri-kicad-lib/switches_lib.pretty/USB_C_Receptacle_Outline_XKB_U262-16XN-4BVC11.kicad_mod
M  lopro/8rows/border8r.py
D  lopro/8rows/pcb/jlcpcb/gerbers/pcb-B_Cu.gbl
D  lopro/8rows/pcb/jlcpcb/gerbers/pcb-F_Cu.gtl
D  lopro/8rows/pcb/jlcpcb/gerbers/pcb-F_Paste.gtp
D  lopro/8rows/pcb/jlcpcb/gerbers/pcb-F_Silkscreen.gto
D  lopro/8rows/pcb/jlcpcb/gerbers/pcb-NPTH-drl_map.gbr
D  lopro/8rows/pcb/jlcpcb/gerbers/pcb-PTH-drl_map.gbr
D  lopro/8rows/pcb/jlcpcb/gerbers/pcb-PTH.drl
A  lopro/8rows/pcb/jlcpcb/gerbers1p2/pcb-B_Cu.gbl
R  lopro/8rows/pcb/jlcpcb/gerbers/pcb-B_Mask.gbs -> lopro/8rows/pcb/jlcpcb/gerbers1p2/pcb-B_Mask.gbs
R  lopro/8rows/pcb/jlcpcb/gerbers/pcb-B_Paste.gbp -> lopro/8rows/pcb/jlcpcb/gerbers1p2/pcb-B_Paste.gbp
R  lopro/8rows/pcb/jlcpcb/gerbers/pcb-B_Silkscreen.gbo -> lopro/8rows/pcb/jlcpcb/gerbers1p2/pcb-B_Silkscreen.gbo
R  lopro/8rows/pcb/jlcpcb/gerbers/pcb-Edge_Cuts.gm1 -> lopro/8rows/pcb/jlcpcb/gerbers1p2/pcb-Edge_Cuts.gm1
A  lopro/8rows/pcb/jlcpcb/gerbers1p2/pcb-F_Cu.gtl
R  lopro/8rows/pcb/jlcpcb/gerbers/pcb-F_Mask.gts -> lopro/8rows/pcb/jlcpcb/gerbers1p2/pcb-F_Mask.gts
A  lopro/8rows/pcb/jlcpcb/gerbers1p2/pcb-F_Paste.gtp
A  lopro/8rows/pcb/jlcpcb/gerbers1p2/pcb-F_Silkscreen.gto
A  lopro/8rows/pcb/jlcpcb/gerbers1p2/pcb-NPTH-drl_map.gbr
R  lopro/8rows/pcb/jlcpcb/gerbers/pcb-NPTH.drl -> lopro/8rows/pcb/jlcpcb/gerbers1p2/pcb-NPTH.drl
A  lopro/8rows/pcb/jlcpcb/gerbers1p2/pcb-PTH-drl_map.gbr
A  lopro/8rows/pcb/jlcpcb/gerbers1p2/pcb-PTH.drl
A  lopro/8rows/pcb/pcb-b.jpg
D  lopro/8rows/pcb/pcb-b.png
D  lopro/8rows/pcb/pcb-f.png
A  lopro/8rows/pcb/pcb.jpg
M  lopro/8rows/pcb/pcb.kicad_pcb
M  lopro/8rows/pcb/pcb.kicad_prl
M  lopro/8rows/pcb/pcb.kicad_pro
M  lopro/8rows/pickle8r.py
M  lopro/8rows/place8r.py
A  lopro/8rows/switch-pl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
Parts:
- moved Ri66 16.6 mm to (164.9, 100.5)
- moved D66 9.54 mm to (166.3, 90.3), turned to -62 degrees
- turned S66 to -62 degrees
Routing:
- net +5V: track 1579.8 -> 1603.2 mm, vias 6 -> 10
- net CB2: track 453.9 -> 440.9 mm
- net /COL9B: track 231.9 -> 226.8 mm
- net /COL8B: track 245.1 -> 249.7 mm, vias 11 -> 13
- net /ROW5: track 196.2 -> 200.1 mm, vias 6 -> 7
- net Net-(Ri66-Pad2): track 6.94 -> 10.5 mm
- net CB1: track 467.4 -> 464.7 mm
- net GND: track 480.7 -> 482.8 mm, vias 99 -> 100
- net /P2: track 117.9 -> 117.0 mm
- net /COL7B: track 278.4 -> 279.1 mm
- net CB6: track 337.2 -> 336.9 mm, vias 15 -> 13
