File: lopro/bak/8rows-v0/pcb/pcb.kicad_sch (KiCad schematic)
At the start: 324 parts, among them J1 U262-161N-4BVC11, J2 Conn_01x03, J3 Conn_01x03, J4 Conn_01x03, Q1 Q_NMOS_DGS, Q2 Q_NMOS_DGS, Q3 Q_NMOS_DGS, Q4 Q_NMOS_DGS, Q5 Q_NMOS_DGS, Q6 Q_NMOS_DGS, Q7 Q_NMOS_DGS, Q8 Q_NMOS_DGS, SW1 SW_DIP_x01_XKB_TS_2030, SW2 SW_DIP_x01_XKB_TS_2030, U1 IS31FL3731-QF, U2 NCP114ASN330T1G, U3 RP2040, U4 Memory_Flash_W25Q64_XSON, X1 12.000MHz

Commit message: add tracks
M  giri-kicad-lib/switches.kicad_sym
A  giri-kicad-lib/switches_lib.pretty/JLC_Order_Num.kicad_mod
A  lopro/8rows/border8r.py
M  lopro/8rows/pcb/pcb.kicad_pcb
M  lopro/8rows/pcb/pcb.kicad_prl
M  lopro/8rows/pcb/pcb.kicad_pro
M  lopro/8rows/pcb/pcb.kicad_sch
A  lopro/8rows/pickle8r.py
A  lopro/8rows/place8r.py
R  lopro/8rows/drawborder8b.py -> lopro/bak/8rows-v0/drawborder8b.py
A  lopro/bak/8rows-v0/pcb/.gitignore
A  lopro/bak/8rows-v0/pcb/LED-Driver.kicad_sch
A  lopro/bak/8rows-v0/pcb/fp-lib-table
A  lopro/bak/8rows-v0/pcb/jlcpcb/gerbers/pcb-B_Cu.gbl
A  lopro/bak/8rows-v0/pcb/jlcpcb/gerbers/pcb-B_Mask.gbs
A  lopro/bak/8rows-v0/pcb/jlcpcb/gerbers/pcb-B_Paste.gbp
A  lopro/bak/8rows-v0/pcb/jlcpcb/gerbers/pcb-B_Silkscreen.gbo
A  lopro/bak/8rows-v0/pcb/jlcpcb/gerbers/pcb-Edge_Cuts.gm1
A  lopro/bak/8rows-v0/pcb/jlcpcb/gerbers/pcb-F_Cu.gtl
A  lopro/bak/8rows-v0/pcb/jlcpcb/gerbers/pcb-F_Mask.gts
A  lopro/bak/8rows-v0/pcb/jlcpcb/gerbers/pcb-F_Paste.gtp
A  lopro/bak/8rows-v0/pcb/jlcpcb/gerbers/pcb-F_Silkscreen.gto
A  lopro/bak/8rows-v0/pcb/jlcpcb/gerbers/pcb-NPTH-drl_map.gbr
A  lopro/bak/8rows-v0/pcb/jlcpcb/gerbers/pcb-NPTH.drl
A  lopro/bak/8rows-v0/pcb/jlcpcb/gerbers/pcb-PTH-drl_map.gbr
A  lopro/bak/8rows-v0/pcb/jlcpcb/gerbers/pcb-PTH.drl
A  lopro/bak/8rows-v0/pcb/pcb-b.png
A  lopro/bak/8rows-v0/pcb/pcb-f.png
A  lopro/bak/8rows-v0/pcb/pcb.kicad_pcb
A  lopro/bak/8rows-v0/pcb/pcb.kicad_prl
A  lopro/bak/8rows-v0/pcb/pcb.kicad_pro
A  lopro/bak/8rows-v0/pcb/pcb.kicad_sch
A  lopro/bak/8rows-v0/pcb/sym-lib-table
R  lopro/8rows/placefp8b.py -> lopro/bak/8rows-v0/placefp8b.py
A  lopro/bak/8rows-v0/switch-plate/.gitignore
A  lopro/bak/8rows-v0/switch-plate/fp-lib-table
A  lopro/bak/8rows-v0/switch-plate/switch-plate.kicad_pcb
A  lopro/bak/8rows-v0/switch-plate/switch-plate.kicad_prl
A  lopro/bak/8rows-v0/switch-plate/switch-plate.kicad_pro
A  lopro/bak/8rows-v0/switch-plate/switch-plate.kicad_sch
A  lopro/bak/8rows-v0/switch-plate/sym-lib-table
A  lopro/bak/8rows-v0/wrist-s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
Parts:
- removed C1: 10uF, RP2040_Minimal:C_1206_3216Metric, symbol Device:C_Small
- removed C10, C11, C12, C13, C20, C3, C4, C5, C6, C7, C8, C9: 100nF, RP2040_Minimal:C_0603_1608Metric_Pad1.08x0.95mm_HandSolder, symbol Device:C_Small
- removed C14, C18, C21: 2.2uF, RP2040_Minimal:C_0603_1608Metric_Pad1.08x0.95mm_HandSolder, symbol Device:C_Small
- removed C15, C16, C19: 1uF, RP2040_Minimal:C_0603_1608Metric_Pad1.08x0.95mm_HandSolder, symbol Device:C_Small
- removed C17, C2: 10uF, RP2040_Minimal:C_0603_1608Metric_Pad1.08x0.95mm_HandSolder, symbol Device:C_Small
- removed C22, C23: 15pF, RP2040_Minimal:C_0603_1608Metric_Pad1.08x0.95mm_HandSolder, symbol Device:C_Small
- removed J1: U262-161N-4BVC11, Connector_USB:USB_C_Receptacle_XKB_U262-16XN-4BVC11, symbol RP2040_Minimal:USB_TYPE_C_Receptacle_16P
- removed JLC1: JLC_Order_Num, giri:JLC_Order_Num, symbol giri:JLC_Order_Num
- removed Q1, Q2, Q3, Q4, Q5, Q6, Q7, Q8: Q_NMOS_DGS, RP2040_Minimal:Diodes_U_DFN1212_3_Handsolder, symbol Device:Q_NMOS_DGS
- removed R10, R7: 27R, RP2040_Minimal:R_0603_1608Metric_Pad0.98x0.95mm_HandSolder, symbol Device:R
- removed R11, R12: 10k, RP2040_Minimal:R_0603_1608Metric_Pad0.98x0.95mm_HandSolder, symbol Device:R
- removed R13, R14: 1k, RP2040_Minimal:R_0603_1608Metric_Pad0.98x0.95mm_HandSolder, symbol Device:R
- removed R8, R9: 5.1k, RP2040_Minimal:R_0603_1608Metric_Pad0.98x0.95mm_HandSolder, symbol Device:R
- removed Rgr1, Rgr2, Rgr3, Rgr4, Rgr5, Rgr6, Rgr7, Rgr8: 160R, Resistor_SMD:R_0603_1608Metric_Pad0.98x0.95mm_HandSolder, symbol giri:Rgr
- removed Rpt1, Rpt10, Rpt11, Rpt12, Rpt13, Rpt14, Rpt15, Rpt16, Rpt17, Rpt18, Rpt2, Rpt3, Rpt4, Rpt5, Rpt6, Rpt7, Rpt8, Rpt9: Rpt, giri:R_0603_1608Metric_Pad0.98x0.95mm_HandSolder, symbol giri:Rpt
- removed SW1, SW2: SW_DIP_x01_XKB_TS_2030, RP2040_Minimal:SW_CK_KXT3, symbol RP2040_Minimal:SW_DIP_x01_XKB_TS_2030
- removed U1: IS31FL3731-QF, RP2040_Minimal:QFN-28-1EP_4x4mm_P0.4mm_EP2.3x2.3mm-Handsolder, symbol Driver_LED:IS31FL3731-QF
- removed U2: NCP114ASN330T1G, Package_SO:TSOP-5_1.65x3.05mm_P0.95mm, symbol RP2040_Minimal:Regulator_LDO_ONS_NCP114_TSOP5
- removed U3: RP2040, RP2040_Minimal:RP2040-QFN-56-Handsolder, symbol RP2040_Minimal:RP2040
- removed U4: Memory_Flash_W25Q64_XSON, RP2040_Minimal:8-USON-Handsolder, symbol RP2040_Minimal:Memory_Flash_W25Q64_XSON
- removed X1: 12.000MHz, RP2040_Minimal:Crystal_SMD_2520-4Pin_2.5x2.0mm-Handsolder, symbol RP2040_Minimal:Crystal_P4
- added Hs18: M1.6, giri:SMTSO_M1.6, symbol giri:MountingHoleSMD
- added MOD1: Conn_rp2040_v1_module_Outline, RP2040_Minimal:Module_Conn_Regular_Outline, symbol RP2040_Minimal:Conn_rp2040_v1_module_Outline
- added MOD2: LED_Driver_Module_Conn, RP2040_Minimal:LED_Driver_Mod_Conn, symbol RP2040_Minimal:LED_Driver_Module_Conn
- added R10, R11, R12, R13, R14, R15, R16, R17, R18, R7, R8, R9: R_Small, giri:R_0603_1608Metric_Pad0.98x0.95mm_HandSolder, symbol Device:R_Small
- R1, R2, R3: value 4.7k -> R_Small; footprint RP2040_Minimal:R_0603_1608Metric_Pad0.98x0.95mm_HandSolder -> giri:R_0603_1608Metric_Pad0.98x0.95mm_HandSolder; LCSC C105871 -> (none); Manufacturer Yageo -> (none); Tolerance 1% -> (none); Type Thick Film -> (none)
- R4, R5, R6: value 20k -> R_Small; footprint RP2040_Minimal:R_0603_1608Metric_Pad0.98x0.95mm_HandSolder -> giri:R_0603_1608Metric_Pad0.98x0.95mm_HandSolder; JLC 20k -> (none); LCSC C144783 -> (none); Manufacturer Yageo -> (none); Tolerance 1% -> (none); Type Thick Film -> (none)
- renumbered Hs18 to Hs19, Hs19 to Hs20, Hs20 to Hs21, Hs21 to Hs22, Hs22 to Hs23, Hs23 to Hs24, Hs24 to Hs25, Hs25 to Hs26, J2 to J1, J3 to J2, J4 to J3
Connections:
- net AD is gone; now on net COL6A: R6.1
- net R_EXT is gone; now on net COL5A: R5.1
- net ~{INTB} is gone; now on net +3V3: R3.2
- net ~{SDB} is gone; now on net +3V3: R4.2
- net +3V3: now also R1.2, R2.2, R5.2, R6.2, MOD1.3 (+3.3V), MOD2.19 (VDD), R10.2, R11.2, R12.2, R13.2, R14.2, R15.2, R16.2, R17.2, R18.2, R7.2, R8.2, R9.2; no longer R1.1, R2.1, R3.1, R4.1
- net +5V: now also MOD1.1 (+5V)
- net CA1: now also D59.2 (A), MOD2.9 (A1)
- net CA2: now also D60.2 (A), MOD2.8 (A2)
- net CA3: now also D61.2 (A), MOD2.7 (A3)
- net CA4: now also D62.2 (A), MOD2.6 (A4)
- net CA5: now also D59.1 (K), D60.1 (K), D61.1 (K), D62.1 (K), D63.1 (K), D64.1 (K), D65.1 (K), D66.1 (K), MOD2.5 (A5)
- net CA6: now also D63.2 (A), MOD2.4 (A6)
- net CA7: now also D64.2 (A), MOD2.3 (A7)
- net CA8: now also D65.2 (A), MOD2.2 (A8)
- net CA9: now also D66.2 (A), MOD2.1 (A9)
- net CB1: now also MOD2.18 (B1); no longer D59.2 (A), D66.2 (A)
- net CB2: now also MOD2.17 (B2); no longer D60.2 (A), D65.2 (A)
- net CB3: now also MOD2.16 (B3); no longer D61.2 (A), D64.2 (A)
- net CB4: now also MOD2.15 (B4); no longer D62.2 (A), D63.2 (A)
- net CB5: now also MOD2.14 (B5)
- net CB6: now also MOD2.13 (B6); no longer D63.1 (K), D64.1 (K), D65.1 (K), D66.1 (K)
- net CB7: now also MOD2.12 (B7); no longer D59.1 (K), D60.1 (K), D61.1 (K), D62.1 (K)
- net CB8: now also MOD2.11 (B8)
- net COL1A: now also R1.1, MOD1.17 (GPIO13)
- net COL1B: now also MOD1.6 (GPIO2), R10.1
- net COL2A: now also R2.1, MOD1.18 (GPIO14)
- net COL2B: now also MOD1.7 (GPIO3), R11.1
- net COL3A: now also R3.1, MOD1.19 (GPIO15)
- net COL3B: now also MOD1.8 (GPIO4), R12.1
- net COL4A: now also R4.1, MOD1.20 (GPIO16)
- net COL4B: now also MOD1.9 (GPIO5), R13.1
- net COL5A: now also MOD1.21 (GPIO17)
- net COL5B: now also MOD1.10 (GPIO6), R14.1
- net COL6A: now also MOD1.22 (GPIO18)
- net COL6B: now also MOD1.11 (GPIO7), R15.1
- net COL7A: now also MOD1.23 (GPIO19), R7.1
- net COL7B: now also MOD1.12 (GPIO8), R16.1
- net COL8A: now also MOD1.24 (GPIO20), R8.1
- net COL8B: now also MOD1.13 (GPIO9), R17.1
- net COL9A: now also MOD1.25 (GPIO21), R9.1
- net COL9B: now also MOD1.16 (GPIO12), R18.1
- net GND: now also MOD1.2 (GND), MOD1.34 (GND), MOD2.20 (GND), MOD2.39 (GND); no longer R5.2, R6.2
- net ROW1: now also MOD2.23 (R1)
- net ROW2: now also MOD2.24 (R2)
- net ROW3: now also MOD2.25 (R3)
- net ROW4: now also MOD2.27 (R5)
- net ROW5: now also MOD2.26 (R4)
- net ROW6: now also MOD2.28 (R6)
- net ROW7: now also MOD2.29 (R7)
- net ROW8: now also MOD2.30 (R8)
- net SCL: now also MOD1.15 (GPIO11), MOD2.22 (SCL); no longer R2.2
- net SDA: now also MOD1.14 (GPIO10), MOD2.21 (SDA); no longer R1.2
- new net INPUT1: MOD1.28 (GPIO24), MOD2.38 (GPIO1)
- new net INPUT2: MOD1.29 (GPIO25), MOD2.37 (GPIO2)
- new net INPUT3: MOD1.30 (GPIO26_ADC0), MOD2.36 (GPIO3)
- new net INPUT4: MOD1.31 (GPIO27_ADC1), MOD2.35 (GPIO4)
- new net INPUT5: MOD1.5 (GPIO1), MOD2.34 (GPIO5)
- new net INPUT6: MOD1.4 (GPIO0), MOD2.33 (GPIO6)
- new net INPUT7: MOD1.33 (GPIO29_ADC3), MOD2.32 (GPIO7)
- new net INPUT8: MOD1.32 (GPIO28_ADC2), MOD2.31 (GPIO8)
- no-connect marks 16 -> 10
Other:
- note added: "MCU Conn"
- note removed: "3.3V/300mA LDO"
- note removed: "4-64Mbit Flash, Quad SPI, 100-133MHz, XIP (eXecute In Place), 3.3V: USON 2x3x.6 mm Winbond: W25Q16JVUXIQ (2MB, 133 MHz) GigaDevice: GD25Q40CEIGR (512kB, 120MHz) GigaDevice: GD25Q80CEIGR (1MB, 120 MHz) GigaDevice: GD25Q80EEIGR (1MB, 133MHz) ISSI: IS25LP080D-JULE (1MB, 133 MHz) WSON-8 5x6mm: Winbond W25Q128JV 16MB C190862 XSON-8 4x4mm: Winbond W25Q64JV 8MB C2940195"
- note removed: "BOM:"
- note removed: "Boot"
- note removed: "Crystal"
- note removed: "Crystal 12MHz, 2520 SMD package: JYJE: 2TJ412000NYGBC JGHC: S22120001210120 Yangxing Tech: X252012MMB4SI-24 Seiko Epson: Q24FA20H0068700 ECS: ECS-120-12-36-AGN-TR3"
- note removed: "Filter / VCC Cap"
- note removed: "LDO 3.3V/300mA, TSOP5 package: On Semi NCP114ASN330T1G Richtek RT9078-33GJ5"
- note removed: "LED Driver"
- note removed: "MOSFET Power Switch"
- note removed: "Make sure these two R's are close to RP2040"
- note removed: "Make sure this C is close to pin 44 of RP2040"
- note removed: "Make sure this C is close to pin 45 of RP2040"
- note removed: "NCP114: Input Capacitor Selection (CIN) It is recommended to connect at least a 1uF Ceramic X5R or X7R capacitor as close as possible to the IN pin of the device. Output Decoupling (COUT) The NCP114 requires an output capacitor connected as close as possible to the output pin of the regulator. The recommended capacitor value is 1uF and X7R or X5R dielectric due to its low capacitance variations o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"
- note removed: "Power"
- note removed: "Pull up / down"
- note removed: "QSPI Flash"
- note removed: "RP2040"
- note removed: "Reset"
- note removed: "Tactile switch: Alps: SKSF, SKSGACE010, side SKSCPBE010 Panasonic: EVPAL7A1AB24, EVPAF7B70, side mount EVPAVAA1A, EVPAEGE2A, EVPAEBB2A Omron: B3U-1000P, side B3U-3000P"
- note removed: "USB TYPE C"
- moved on the sheet: D59, D60, D61, D62, D63, D64, D65, D66, D67, D68, D69, D70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
