File: lopro/8rows/switch-plate/switch-plate.kicad_pcb (KiCad board)
At the start: 2 copper layers, 17.7 x 17.7 mm, 89 parts

Commit message: add wrist support
M  giri-kicad-lib/switches.kicad_sym
A  giri-kicad-lib/switches_lib.pretty/MountingHole_1.7mm_M1.6_NoPad.kicad_mod
M  giri-kicad-lib/switches_lib.pretty/Pad_Only_SMTSO_M2.kicad_mod
A  giri-kicad-lib/switches_lib.pretty/SMTSO_M2_Hole_Only.kicad_mod
M  giri-kicad-lib/switches_lib.pretty/Switch_Cutout_LoPro.kicad_mod
A  giri-kicad-lib/switches_lib.pretty/Switch_Cutout_LoPro_R.kicad_mod
A  giri-kicad-lib/switches_lib.pretty/Switch_Cutout_LoPro_Wide.kicad_mod
M  lopro/8rows/drawborder8b.py
A  lopro/8rows/pcb/jlcpcb/gerbers/pcb-B_Cu.gbl
A  lopro/8rows/pcb/jlcpcb/gerbers/pcb-B_Mask.gbs
A  lopro/8rows/pcb/jlcpcb/gerbers/pcb-B_Paste.gbp
A  lopro/8rows/pcb/jlcpcb/gerbers/pcb-B_Silkscreen.gbo
A  lopro/8rows/pcb/jlcpcb/gerbers/pcb-Edge_Cuts.gm1
A  lopro/8rows/pcb/jlcpcb/gerbers/pcb-F_Cu.gtl
A  lopro/8rows/pcb/jlcpcb/gerbers/pcb-F_Mask.gts
A  lopro/8rows/pcb/jlcpcb/gerbers/pcb-F_Paste.gtp
A  lopro/8rows/pcb/jlcpcb/gerbers/pcb-F_Silkscreen.gto
A  lopro/8rows/pcb/jlcpcb/gerbers/pcb-NPTH-drl_map.gbr
A  lopro/8rows/pcb/jlcpcb/gerbers/pcb-NPTH.drl
A  lopro/8rows/pcb/jlcpcb/gerbers/pcb-PTH-drl_map.gbr
A  lopro/8rows/pcb/jlcpcb/gerbers/pcb-PTH.drl
M  lopro/8rows/pcb/pcb.kicad_pcb
M  lopro/8rows/placefp8b.py
M  lopro/8rows/switch-plate/fp-lib-table
M  lopro/8rows/switch-plate/switch-plate.kicad_pcb
M  lopro/8rows/switch-plate/switch-plate.kicad_prl
M  lopro/8rows/switch-plate/switch-plate.kicad_sch
M  lopro/8rows/switch-plate/sym-lib-table
A  lopro/8rows/wrist-support/fp-lib-table
A  lopro/8rows/wrist-support/sym-lib-table
A  lopro/8rows/wrist-support/wrist-support.kicad_pcb
A  lopro/8rows/wrist-support/wrist-support.kicad_prl
A  lopro/8rows/wrist-support/wrist-support.kicad_pro
A  lopro/8rows/wrist-support/wrist-support.kicad_sch
A  lopro/8rows/wrist-washer/fp-lib-table
A  lopro/8rows/wrist-washer/sym-lib-table
A  lopro/8rows/wrist-washer/wrist-washer.kicad_pcb
A  lopro/8rows/wrist-washer/wrist-washer.kicad_prl
A  lopro/8rows/wrist-washer/wrist-washer.kicad_pro
A  lop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
Parts:
- removed H_S1, H_S10, H_S11, H_S12, H_S13, H_S14, H_S15, H_S16, H_S17, H_S2, H_S3, H_S4, H_S5, H_S6, H_S7, H_S8, H_S9: MountingHoleSMD, Giri_Library:SMTSO_M2
- added Hs1: MountingHoleSMD, Giri_Library:MountingHole_1.7mm_M1.6_Pad, F.Cu at (28.5, -7.10)
- added Hs10: MountingHoleSMD, Giri_Library:MountingHole_1.7mm_M1.6_Pad, F.Cu at (47.5, 48.1)
- added Hs11: MountingHoleSMD, Giri_Library:MountingHole_1.7mm_M1.6_Pad, F.Cu at (185.2, 67.1)
- added Hs12: MountingHoleSMD, Giri_Library:MountingHole_1.7mm_M1.6_Pad, F.Cu at (291.8, 47.5)
- added Hs13: MountingHoleSMD, Giri_Library:MountingHole_1.7mm_M1.6_Pad, F.Cu at (1.80, 83.1)
- added Hs14: MountingHoleSMD, Giri_Library:MountingHole_1.7mm_M1.6_Pad, F.Cu at (81.9, 85.0)
- added Hs15: MountingHoleSMD, Giri_Library:MountingHole_1.7mm_M1.6_Pad, F.Cu at (149.2, 83.7)
- added Hs16: MountingHoleSMD, Giri_Library:MountingHole_1.7mm_M1.6_Pad, F.Cu at (232.8, 46.9)
- added Hs17: MountingHoleSMD, Giri_Library:MountingHole_1.7mm_M1.6_Pad, F.Cu at (210.9, 83.1)
- added Hs18: MountingHoleSMD, Giri_Library:MountingHole_1.7mm_M1.6_Pad, F.Cu at (291.8, 80.1)
- added Hs2: MountingHoleSMD, Giri_Library:MountingHole_1.7mm_M1.6_Pad, F.Cu at (104.5, -7.10)
- added Hs3: MountingHoleSMD, Giri_Library:MountingHole_1.7mm_M1.6_Pad, F.Cu at (199.5, -7.10)
- added Hs4: MountingHoleSMD, Giri_Library:MountingHole_1.7mm_M1.6_Pad, F.Cu at (275.5, -7.10)
- added Hs5: MountingHoleSMD, Giri_Library:MountingHole_1.7mm_M1.6_Pad, F.Cu at (35.6, 27.9)
- added Hs6: MountingHoleSMD, Giri_Library:MountingHole_1.7mm_M1.6_Pad, F.Cu at (95.0, 27.9)
- added Hs7: MountingHoleSMD, Giri_Library:MountingHole_1.7mm_M1.6_Pad, F.Cu at (137.8, 46.9)
- added Hs8: MountingHoleSMD, Giri_Library:MountingHole_1.7mm_M1.6_Pad, F.Cu at (171.0, 27.9)
- added Hs9: MountingHoleSMD, Giri_Library:MountingHole_1.7mm_M1.6_Pad, F.Cu at (268.4, 27.9)
- moved S70 4.75 mm to (242.2, 76.0)
- moved S71 4.75 mm to (261.2, 76.0)
- moved S72 4.75 mm to (280.2, 76.0)
- moved S69 2.38 mm to (223.2, 76.0)
- moved S64 0.40 mm to (113.4, 92.5), turned to 62 degrees
- moved S66 0.40 mm to (162.1, 92.5), turned to 118 degrees
- moved S63 0.30 mm to (94.0, 81.2)
- moved S67 0.20 mm to (179.1, 81.2)
Other:
- board size 17.7 x 17.7 mm -> 302.6 x 118.1 mm

Commit message: enlarge center hole of keychron switch footprint
M  giri-kicad-lib/switches.kicad_sym
M  giri-kicad-lib/switches_lib.pretty/Keychron_Optical_Switch_1u.kicad_mod
M  giri-kicad-lib/switches_lib.pretty/Keychron_Optical_Switch_R_1u.kicad_mod
A  giri-kicad-lib/switches_lib.pretty/USB_C_Receptacle_Outline_XKB_U262-16XN-4BVC11.kicad_mod
M  lopro/8rows/border8r.py
D  lopro/8rows/pcb/jlcpcb/gerbers/pcb-B_Cu.gbl
D  lopro/8rows/pcb/jlcpcb/gerbers/pcb-F_Cu.gtl
D  lopro/8rows/pcb/jlcpcb/gerbers/pcb-F_Paste.gtp
D  lopro/8rows/pcb/jlcpcb/gerbers/pcb-F_Silkscreen.gto
D  lopro/8rows/pcb/jlcpcb/gerbers/pcb-NPTH-drl_map.gbr
D  lopro/8rows/pcb/jlcpcb/gerbers/pcb-PTH-drl_map.gbr
D  lopro/8rows/pcb/jlcpcb/gerbers/pcb-PTH.drl
A  lopro/8rows/pcb/jlcpcb/gerbers1p2/pcb-B_Cu.gbl
R  lopro/8rows/pcb/jlcpcb/gerbers/pcb-B_Mask.gbs -> lopro/8rows/pcb/jlcpcb/gerbers1p2/pcb-B_Mask.gbs
R  lopro/8rows/pcb/jlcpcb/gerbers/pcb-B_Paste.gbp -> lopro/8rows/pcb/jlcpcb/gerbers1p2/pcb-B_Paste.gbp
R  lopro/8rows/pcb/jlcpcb/gerbers/pcb-B_Silkscreen.gbo -> lopro/8rows/pcb/jlcpcb/gerbers1p2/pcb-B_Silkscreen.gbo
R  lopro/8rows/pcb/jlcpcb/gerbers/pcb-Edge_Cuts.gm1 -> lopro/8rows/pcb/jlcpcb/gerbers1p2/pcb-Edge_Cuts.gm1
A  lopro/8rows/pcb/jlcpcb/gerbers1p2/pcb-F_Cu.gtl
R  lopro/8rows/pcb/jlcpcb/gerbers/pcb-F_Mask.gts -> lopro/8rows/pcb/jlcpcb/gerbers1p2/pcb-F_Mask.gts
A  lopro/8rows/pcb/jlcpcb/gerbers1p2/pcb-F_Paste.gtp
A  lopro/8rows/pcb/jlcpcb/gerbers1p2/pcb-F_Silkscreen.gto
A  lopro/8rows/pcb/jlcpcb/gerbers1p2/pcb-NPTH-drl_map.gbr
R  lopro/8rows/pcb/jlcpcb/gerbers/pcb-NPTH.drl -> lopro/8rows/pcb/jlcpcb/gerbers1p2/pcb-NPTH.drl
A  lopro/8rows/pcb/jlcpcb/gerbers1p2/pcb-PTH-drl_map.gbr
A  lopro/8rows/pcb/jlcpcb/gerbers1p2/pcb-PTH.drl
A  lopro/8rows/pcb/pcb-b.jpg
D  lopro/8rows/pcb/pcb-b.png
D  lopro/8rows/pcb/pcb-f.png
A  lopro/8rows/pcb/pcb.jpg
M  lopro/8rows/pcb/pcb.kicad_pcb
M  lopro/8rows/pcb/pcb.kicad_prl
M  lopro/8rows/pcb/pcb.kicad_pro
M  lopro/8rows/pickle8r.py
M  lopro/8rows/place8r.py
A  lopro/8rows/switch-pl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
Parts:
- removed Hs18: MountingHoleSMD, Giri_Library:MountingHole_1.7mm_M1.6_Pad
- added J1: USB_C_Dummy, Giri_Library:USB_C_Receptacle_Outline_XKB_U262-16XN-4BVC11, F.Cu at (3.70, 17.4)
- Hs1, Hs10, Hs11, Hs12, Hs13, Hs14, Hs15, Hs16, Hs17, Hs2, Hs3, Hs4, Hs5, Hs6, Hs7, Hs8, Hs9: value MountingHoleSMD -> M1.6; footprint Giri_Library:MountingHole_1.7mm_M1.6_Pad -> Giri_Library:MountingHole_1.7mm_M1.6_NoPad
- moved Hs15 91.3 mm to (232.8, 46.9)
- moved Hs17 81.0 mm to (291.8, 80.1)
- moved Hs16 42.3 mm to (210.9, 83.1)
- moved Hs13 0.54 mm to (2.34, 83.1)
Other:
- board size 302.6 x 118.1 mm -> 296.1 x 118.1 mm
