File: mx/prototype/pcb/pcb.kicad_sch (KiCad schematic)
At the start: 45 parts, among them J1 Conn_01x06_Socket, J2 Conn_01x03_Socket, J3 Conn_01x05_Socket, J4 Conn_01x03_Socket, J5 Conn_01x03_Socket, Q1 MMBT3904, Q2 MMBT3904, Q3 MMBT3904

Commit message: M  giri-kicad-lib/switches.kicad_sym A  giri-kicad-lib/switches_lib.pretty/Gateron_1u.kicad_mod A  giri-kicad-lib/switches_lib.pretty/LED_0603_1608Metric.kicad_mod A  giri-kicad-lib/switches_lib.pretty/LargePad_M2.kicad_mod A  giri-kicad-lib/switches_lib.pretty/MINEW-MS88SF3-Daughter-Board.kicad_mod A  giri-kicad-lib/switches_lib.pretty/MINEW-MS88SF3.kicad_mod A  giri-kicad-lib/switches_lib.pretty/MountingHole_2.2mm_M2_LargePad.kicad_mod A  giri-kicad-lib/switches_lib.pretty/PGA2040_PTH_NO_SLOT.kicad_mod A  giri-kicad-lib/switches_lib.pretty/PGA2040_PTH_WITH_SLOT.kicad_mod A  giri-kicad-lib/switches_lib.pretty/PGA2040_SMT_WITH_SLOT.kicad_mod A  giri-kicad-lib/switches_lib.pretty/R_0603_1608Metric.kicad_mod M  lopro/6rows/pcb/pcb.kicad_prl M  lopro/6rows/pcb/pcb.kicad_pro A  lopro/8rows/.gitignore M  lopro/8rows/pcb/pcb.kicad_pro A  lopro/8rows/pcb/~pcb.kicad_sch.lck R  mx/simple/pcb/.gitignore -> mx/prototype/pcb/.gitignore R  mx/simple/pcb/fp-lib-table -> mx/prototype/pcb/fp-lib-table R  mx/simple/pcb/pcb.kicad_pcb -> mx/prototype/pcb/pcb.kicad_pcb R  mx/simple/pcb/pcb.kicad_prl -> mx/prototype/pcb/pcb.kicad_prl R  mx/simple/pcb/pcb.kicad_pro -> mx/prototype/pcb/pcb.kicad_pro R  mx/simple/pcb/pcb.kicad_sch -> mx/prototype/pcb/pcb.kicad_sch R  mx/simple/pcb/sym-lib-table -> mx/prototype/pcb/sym-lib-table A  mx/rev3/.gitignore A  mx/rev3/border.py A  mx/rev3/pcb/.gitignore A  mx/rev3/pcb/LED-Driver.kicad_sch A  mx/rev3/pcb/fp-lib-table A  mx/rev3/pcb/pcb-b.jpg A  mx/rev3/pcb/pcb.jpg A  mx/rev3/pcb/pcb.kicad_pcb A  mx/rev3/pcb/pcb.kicad_prl A  mx/rev3/pcb/pcb.kicad_pro A  mx/rev3/pcb/pcb.kicad_sch A  mx/rev3/pcb/sym-lib-table A  mx/rev3/pickle.py A  mx/rev3/place.py A  mx/rev3/switch-plate/.gitignore A  mx/rev3/switch-plate/fp-lib-table A  mx/rev3/switch-plate/jlcpcb/gerbers/switch-plate-B_Cu.gbl A  mx/rev3/switch-plate/jlcpcb/gerbers/switch-plate-B_Mask.gbs A  mx/rev3/switch-plate/jlcpcb/gerbers/switch-plate-B_Paste.gbp A  mx/rev3/switch-plate/jlcpcb/gerbers/switch-p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
Parts:
- N1, N2, N5: value NMOS-BSH105 -> NMOS-BSH105-or-BSS138LT1
- N3, N4: value NMOS-BSH105 -> NMOS-BSH105-Or-BSS138LT1
Other:
- note added: "SMD welding: 1) put some paste on pad, use solder to smear it on the pad, 2) add very small amout of paste, smaller or none for IC chips, 3) place component and hot air solder"
Changed lines of the file:
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@@
     (stroke (width 0) (type default))
+  )
+  (text "SMD welding: \n1) put some paste on pad, use solder to smear it on the pad, \n2) add very small amout of paste, smaller or none for IC chips, \n3) place component and hot air solder"
+    (at 175.26 43.18 0)
+    (effects (font (size 1.27 1.27)) (justify left bottom))
   )
   (label "ROW4" (at 140.97 109.22 180) (fields_autoplaced)
@@
       (effects (font (size 1.27 1.27)) (justify left))
     )
-    (property "Value" "NMOS-BSH105" (at 154.94 123.825 0)
+    (property "Value" "NMOS-BSH105-or-BSS138LT1" (at 154.94 123.825 0)
       (effects (font (size 1.27 1.27)) (justify left))
     )
@@
       (effects (font (size 1.27 1.27)) (justify left))
     )
-    (property "Value" "NMOS-BSH105" (at 154.94 32.385 0)
+    (property "Value" "NMOS-BSH105-or-BSS138LT1" (at 154.94 32.385 0)
       (effects (font (size 1.27 1.27)) (justify left))
     )
@@
       (effects (font (size 1.27 1.27)) (justify left))
     )
-    (property "Value" "NMOS-BSH105" (at 154.94 55.245 0)
+    (property "Value" "NMOS-BSH105-or-BSS138LT1" (at 154.94 55.245 0)
       (effects (font (size 1.27 1.27)) (justify left))
     )
@@
       (effects (font (size 1.27 1.27)) (justify left))
     )
-    (property "Value" "NMOS-BSH105" (at 154.94 78.105 0)
+    (property "Value" "NMOS-BSH105-Or-BSS138LT1" (at 154.94 78.105 0)
       (effects (font (size 1.27 1.27)) (justify left))
     )
@@
       (effects (font (size 1.27 1.27)) (justify left))
     )
-    (property "Value" "NMOS-BSH105" (at 154.94 100.965 0)
-      (effects (font (size 1.27 1.27)) (justify left))
-    )
+    (property "Value" "NMOS-BSH105-Or-BSS138LT1" (at 154.94 100.965 0)
+      (effects (font (size 1.27 1.27)) (justify left))
+    )
