File: mx/rev3/pcb/pcb.kicad_pcb (KiCad board)
At the start: 2 copper layers, 309.5 x 190.8 mm, 277 parts, among them J1 Conn_01x03, J2 Conn_01x03, J3 Conn_01x03, J4 Conn_01x03, J5 Conn_01x03, J6 Conn_01x03, J7 Conn_01x03, J8 Conn_01x03, Q1 MMBT3904, Q10 MMBT3904, Q11 MMBT3904, Q12 MMBT3904, Q13 MMBT3904, Q14 MMBT3904, Q15 MMBT3904, Q2 MMBT3904, Q3 MMBT3904, Q4 MMBT3904, Q5 MMBT3904, Q6 MMBT3904, Q7 MMBT3904, Q8 MMBT3904, Q9 MMBT3904, SW1 SW_DIP_x01_XKB_TS_2030, SW2 SW_DIP_x01_XKB_TS_2030, U1 IS31FL3731-QF

Commit message: M  .gitignore M  giri-kicad-lib/switches.kicad_sym A  giri-kicad-lib/switches_lib.pretty/RP2040_Stamp.kicad_mod A  giri-kicad-lib/switches_lib.pretty/SW_B3U-3000P.kicad_mod M  lopro/8rows/pcb/pcb.kicad_sch A  mx/rev3/.border.py.swp A  mx/rev3/.build.py.swp A  mx/rev3/build.py M  mx/rev3/pcb/pcb.kicad_pcb M  mx/rev3/pcb/pcb.kicad_prl M  mx/rev3/pcb/pcb.kicad_sch D  mx/rev3/place.py A  mx/rev3/test.py D  rp2040backpack/pcb/jlcpcb/gerbers1p2/pcb-B_Cu.gbl D  rp2040backpack/pcb/jlcpcb/gerbers1p2/pcb-B_Mask.gbs D  rp2040backpack/pcb/jlcpcb/gerbers1p2/pcb-B_Paste.gbp D  rp2040backpack/pcb/jlcpcb/gerbers1p2/pcb-B_Silkscreen.gbo D  rp2040backpack/pcb/jlcpcb/gerbers1p2/pcb-Edge_Cuts.gm1 D  rp2040backpack/pcb/jlcpcb/gerbers1p2/pcb-F_Cu.gtl D  rp2040backpack/pcb/jlcpcb/gerbers1p2/pcb-F_Mask.gts D  rp2040backpack/pcb/jlcpcb/gerbers1p2/pcb-F_Paste.gtp D  rp2040backpack/pcb/jlcpcb/gerbers1p2/pcb-F_Silkscreen.gto D  rp2040backpack/pcb/jlcpcb/gerbers1p2/pcb-NPTH-drl_map.gbr D  rp2040backpack/pcb/jlcpcb/gerbers1p2/pcb-NPTH.drl D  rp2040backpack/pcb/jlcpcb/gerbers1p2/pcb-PTH-drl_map.gbr D  rp2040backpack/pcb/jlcpcb/gerbers1p2/pcb-PTH.drl R  rp2040backpack/pickle.py -> rp2040stamp/pickle.py R  rp2040backpack/pcb/.gitignore -> rp2040stamp/rev1/pcb/.gitignore R  rp2040backpack/pcb/LED-Driver.kicad_sch -> rp2040stamp/rev1/pcb/LED-Driver.kicad_sch R  rp2040backpack/pcb/fp-lib-table -> rp2040stamp/rev1/pcb/fp-lib-table R  rp2040backpack/pcb/pcb-b.jpg -> rp2040stamp/rev1/pcb/pcb-b.jpg R  rp2040backpack/pcb/pcb.jpg -> rp2040stamp/rev1/pcb/pcb.jpg R  rp2040backpack/pcb/pcb.kicad_pcb -> rp2040stamp/rev1/pcb/pcb.kicad_pcb R  rp2040backpack/pcb/pcb.kicad_prl -> rp2040stamp/rev1/pcb/pcb.kicad_prl R  rp2040backpack/pcb/pcb.kicad_pro -> rp2040stamp/rev1/pcb/pcb.kicad_pro R  rp2040backpack/pcb/pcb.kicad_sch -> rp2040stamp/rev1/pcb/pcb.kicad_sch R  rp2040backpack/pcb/sym-lib-table -> rp2040stamp/rev1/pcb/sym-lib-table A  rp2040stamp/rev2/pcb/.gitignore A  rp2040stamp/rev2/pcb/LED-Driver.kicad_sch A  r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
Parts:
- moved R6 118.2 mm to (157.6, 66.9), turned to 90 degrees
- moved C4 112.9 mm to (160.9, 69.4)
- moved R5 108.9 mm to (162.5, 77.4), turned to -90 degrees
- moved R2 107.7 mm to (154.3, 67.0), turned to -90 degrees
- moved C1 107.4 mm to (154.2, 78.1), turned to 90 degrees
- moved U1 106.3 mm to (155.6, 72.2), turned to 90 degrees
- moved R1 106.2 mm to (156.0, 66.9), turned to -90 degrees
- moved R4 105.2 mm to (159.4, 77.4), turned to 90 degrees
- moved R3 103.8 mm to (161.0, 77.4), turned to 90 degrees
- moved C3 102.3 mm to (157.8, 77.4), turned to -90 degrees
- moved C2 99.3 mm to (156.2, 77.4), turned to -90 degrees
- moved R7 74.4 mm to (146.0, 112.8)
- moved R9 62.1 mm to (140.2, 113.7)
- moved C5 60.0 mm to (122.7, 112.3)
- moved R8 60.0 mm to (131.4, 109.8)
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Connections:
- C1 pad 2: +3V3 -> +5V
- C2 pad 1: +3V3 -> +5V
- C3 pad 1: +3V3 -> +5V
- Jrp1 pad H5: unconnected-(Jrp1-GPIO15-PadH5) -> /~{SDB}
Routing:
- net CB7: track 62.7 -> 432.8 mm, vias 0 -> 7
- net CB3: track 117.9 -> 424.6 mm, vias 0 -> 10
- net CB2: track 172.4 -> 410.1 mm, vias 0 -> 11
- net CB4: track 137.2 -> 373.1 mm, vias 0 -> 10
- net CB6: track 114.8 -> 339.5 mm, vias 0 -> 7
- net CA2: track 117.9 -> 317.6 mm, vias 0 -> 6
- net CB8: track 0.00 -> 199.0 mm, vias 0 -> 4
- net CA5: track 0.00 -> 164.3 mm, vias 0 -> 5
- net CA3: track 139.9 -> 287.8 mm, vias 0 -> 6
- net CA6: track 0.00 -> 146.6 mm, vias 0 -> 5
- net CA7: track 0.00 -> 126.4 mm, vias 0 -> 5
- net CB1: track 138.9 -> 263.4 mm, vias 2 -> 8
- net CB5: track 103.2 -> 223.1 mm, vias 0 -> 7
- net CA1: track 214.2 -> 328.9 mm, vias 5 -> 7
- net CA8: track 0.00 -> 110.4 mm, vias 0 -> 5
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
Commit message: M mx/rev3/border.py M  mx/rev3/pcb/pcb.kicad_pcb M  mx/rev3/pcb/pcb.kicad_prl M  mx/rev3/pcb/pcb.kicad_sch RM mx/rev3/build.py -> mx/rev3/place.py
Parts:
- moved Rgr1 190.8 mm to (62.5, -8.76)
- moved N1 187.4 mm to (66.5, -6.86), turned to -90 degrees
- moved N2 158.3 mm to (75.9, 13.3), turned to -90 degrees
- moved Rgr2 153.0 mm to (76.0, 9.99)
- moved Rgr3 127.6 mm to (60.4, 46.8)
- moved N4 123.9 mm to (71.3, 61.3), turned to 90 degrees
- moved N5 123.9 mm to (61.7, 80.4), turned to 90 degrees
- moved Rgr4 122.0 mm to (69.5, 65.5)
- moved Rgr5 121.0 mm to (61.6, 83.5)
- moved N3 121.0 mm to (61.8, 42.9), turned to 90 degrees
- moved D58 9.50 mm to (275.5, 51.9)
- moved Ri20 9.50 mm to (283.7, 57.0)
- moved S58 9.50 mm to (275.5, 57.0)
- moved D45 7.12 mm to (16.6, 51.9)
- moved S45 7.12 mm to (16.6, 57.0)
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Routing:
- net CB1: track 263.4 -> 456.6 mm, vias 8 -> 10
- net CA2: track 317.6 -> 203.3 mm, vias 6 -> 5
- net CA3: track 287.8 -> 266.9 mm, vias 6 -> 5
- net Net-(Q4-B): track 104.6 -> 85.5 mm
- net CA1: track 328.9 -> 310.7 mm
- net Net-(Q13-B): track 111.5 -> 129.2 mm, vias 4 -> 5
- net CB4: track 373.1 -> 363.7 mm
- net CA4: track 248.9 -> 241.8 mm
- net Net-(S58-IR_A): track 23.1 -> 16.2 mm, vias 2 -> 0
- net /R4_SINK: track 232.8 -> 226.8 mm
- net Net-(Q2-B): track 100.4 -> 105.9 mm
- net +3V3: track 1513.5 -> 1508.2 mm, vias 25 -> 21
- net /R3_SINK: track 236.0 -> 241.2 mm
- net Net-(N1-G): track 0.00 -> 4.65 mm
- net /R5_SINK: track 221.8 -> 226.4 mm
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
Commit message: M giri-kicad-lib/switches.kicad_sym  M giri-kicad-lib/switches_lib.pretty/PGA2040_SMT_WITH_SLOT.kicad_mod M  mx/rev3/border.py M  mx/rev3/pcb/pcb.kicad_pcb M  mx/rev3/pcb/pcb.kicad_prl M  mx/rev3/pcb/pcb.kicad_sch M  mx/rev3/place.py ?? giri-kicad-lib/switches_lib.pretty/ALS-PT19.kicad_mod ?? giri-kicad-lib/switches_lib.pretty/Debug_PinHeader_1x06_P2.00mm_Vertical.kicad_mod ?? giri-kicad-lib/switches_lib.pretty/PGA2040_SMT_NO_SLOT.kicad_mod ?? giri-kicad-lib/switches_lib.pretty/PinHeader_1x02_P2.54mm_Vertical.kicad_mod ?? giri-kicad-lib/switches_lib.pretty/TEMT6000-sensor.kicad_mod ?? giri-kicad-lib/switches_lib.pretty/mouse-bite-2mm-slot.kicad_mod
Parts:
- removed J2, J3, J4, J5, J6, J7, J8: Conn_01x03, giri:PinHeader_1x03_P2.54mm_Vertical
- added R10: 10k, RP2040_Minimal:R_0603_1608Metric_Pad0.98x0.95mm_HandSolder, F.Cu at (-9.72, -6.02)
- added Sens1: ~, giri:ALS-PT19, F.Cu at (-13.0, -6.81)
- H1, H2, H3, H4, H5, H6, H7, H8: footprint giri:MountingHole_2.2mm_M2_ISO7380_Pad -> giri:SMTSO_M2
- J1: value Conn_01x03 -> Conn_01x06_Socket; footprint giri:PinHeader_1x03_P2.54mm_Vertical -> giri:Debug_PinHeader_1x06_P2.00mm_Vertical
- Jrp1: footprint giri:PGA2040_SMT_WITH_SLOT -> giri:PGA2040_SMT_NO_SLOT
- moved R9 183.1 mm to (-2.43, -1.07)
- moved SW2 178.0 mm to (-12.8, 50.2), turned to 90 degrees
- moved SW1 176.0 mm to (-12.8, 56.7), turned to 90 degrees
- moved R7 167.9 mm to (-9.93, 50.5), turned to 90 degrees
- moved R8 167.6 mm to (-1.71, 7.95), turned to -90 degrees
- moved C5 164.5 mm to (-3.50, 6.69), turned to 90 degrees
- moved J1 163.3 mm to (-12.5, 63.2)
- moved Rgr3 11.5 mm to (70.0, 52.9), turned to -90 degrees
- moved N3 9.96 mm to (61.5, 33.0), turned to -90 degrees
- moved Hs1 9.50 mm to (0.00, -7.00)
- moved Hs2 4.75 mm to (-9.50, 42.8)
- moved Jusb1 2.02 mm to (-9.77, 1.44)
- moved H2 0.73 mm to (-7.25, 171.5)
- moved H3 0.73 mm to (66.8, 171.5)
- moved H6 0.73 mm to (208.8, 171.5)
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Connections:
- J1 pad 1: unconnected-(J1-Pin_1-Pad1) -> SWCLK
- J1 pad 2: unconnected-(J1-Pin_2-Pad2) -> GND
- J1 pad 3: unconnected-(J1-Pin_3-Pad3) -> SWDIO
- Jrp1 pad B1: /COL1 -> unconnected-(Jrp1-GPIO0-PadB1)
- Jrp1 pad B5: unconnected-(Jrp1-SWCLK-PadB5) -> SWCLK
- Jrp1 pad B6: unconnected-(Jrp1-SWDIO-PadB6) -> SWDIO
- Jrp1 pad B8: unconnected-(Jrp1-GPIO29/ADC3-PadB8) -> SENSOR
- Jrp1 pad C1: /COL2 -> unconnected-(Jrp1-GPIO1-PadC1)
- Jrp1 pad C2: /COL3 -> unconnected-(Jrp1-GPIO2-PadC2)
- Jrp1 pad C7: unconnected-(Jrp1-GPIO28/ADC2-PadC7) -> /ROW1
- Jrp1 pad C8: unconnected-(Jrp1-GPIO27/ADC1-PadC8) -> /COL1
- Jrp1 pad D1: /COL4 -> unconnected-(Jrp1-GPIO3-PadD1)
- Jrp1 pad D2: /COL5 -> unconnected-(Jrp1-GPIO4-PadD2)
- Jrp1 pad D7: unconnected-(Jrp1-GPIO26/ADC0-PadD7) -> /COL2
- Jrp1 pad D8: unconnected-(Jrp1-GPIO25-PadD8) -> /COL3
- Jrp1 pad E1: /COL6 -> unconnected-(Jrp1-GPIO5-PadE1)
- Jrp1 pad E2: /COL7 -> SDA
- Jrp1 pad E7: unconnected-(Jrp1-GPIO24-PadE7) -> /COL4
- Jrp1 pad E8: unconnected-(Jrp1-GPIO23-PadE8) -> /COL5
- Jrp1 pad F1: /COL8 -> SCL
- Jrp1 pad F2: /COL9 -> /~{SDB}
- Jrp1 pad F7: /ROW5 -> /COL6
- Jrp1 pad F8: /ROW4 -> /COL7
- Jrp1 pad G1: /COL10 -> /ROW5
- Jrp1 pad G3: /COL13 -> /COL15
- Jrp1 pad G4: /COL15 -> /COL13
- Jrp1 pad G5: SDA -> /COL11
- Jrp1 pad G6: /ROW1 -> /COL9
- Jrp1 pad G8: /ROW3 -> /COL8
- Jrp1 pad H2: /COL11 -> /ROW4
- Jrp1 pad H3: /COL12 -> /ROW3
- Jrp1 pad H5: /~{SDB} -> /COL12
- Jrp1 pad H6: SCL -> /COL10
Routing:
- net /COL15: track 2.20 -> 332.2 mm, vias 0 -> 2
- net /COL14: track 2.20 -> 309.9 mm, vias 0 -> 2
- net /COL13: track 2.20 -> 292.4 mm, vias 0 -> 2
- net /COL12: track 2.20 -> 268.2 mm, vias 0 -> 2
- net /COL11: track 2.20 -> 251.6 mm, vias 0 -> 2
- net /COL10: track 2.20 -> 228.0 mm, vias 0 -> 2
- net /COL9: track 2.20 -> 209.9 mm, vias 0 -> 2
- net /COL8: track 2.20 -> 146.6 mm
- net /COL7: track 2.20 -> 126.6 mm
- net /ROW5: track 0.00 -> 116.2 mm, vias 0 -> 2
- net /COL6: track 2.20 -> 110.1 mm
- net /ROW4: track 0.00 -> 98.8 mm
- net /ROW3: track 0.00 -> 89.2 mm
- net /COL5: track 2.20 -> 87.5 mm
- net /ROW2: track 0.00 -> 82.4 mm
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
Commit message: M giri-kicad-lib/switches.kicad_sym  M giri-kicad-lib/switches_lib.pretty/Gateron_1u.kicad_mod  M giri-kicad-lib/switches_lib.pretty/Gateron_Sw_1u.kicad_mod  M giri-kicad-lib/switches_lib.pretty/PGA2040_SMT_WITH_SLOT.kicad_mod  M giri-kicad-lib/switches_lib.pretty/SW_B3U-3000P.kicad_mod M  mx/rev3/border.py M  mx/rev3/pcb/fp-lib-table M  mx/rev3/pcb/pcb.kicad_pcb M  mx/rev3/pcb/pcb.kicad_prl M  mx/rev3/pcb/pcb.kicad_pro M  mx/rev3/pcb/pcb.kicad_sch M  mx/rev3/place.py M  mx/rev3/switch-plate/switch-plate.kicad_pcb M  mx/rev3/switch-plate/switch-plate.kicad_prl M  mx/rev3/switch-plate/switch-plate.kicad_pro M  mx/rev3/switch-plate/switch-plate.kicad_sch M  mx/rev3/wrist-washer/wrist-washer.kicad_pcb M  mx/rev3/wrist-washer/wrist-washer.kicad_prl M  mx/rev3/wrist-washer/wrist-washer.kicad_pro M  mx/rev3/wrist-washer/wrist-washer.kicad_sch ?? giri-kicad-lib/switches_lib.pretty/ALS-PT19.kicad_mod ?? giri-kicad-lib/switches_lib.pretty/Debug_PinHeader_1x06_P2.00mm_Vertical.kicad_mod ?? giri-kicad-lib/switches_lib.pretty/Debug_PinHeader_1x06_P2.54mm_Vertical.kicad_mod ?? giri-kicad-lib/switches_lib.pretty/Gateron_1.25.kicad_mod ?? giri-kicad-lib/switches_lib.pretty/Gateron_1.25u_v2.kicad_mod ?? giri-kicad-lib/switches_lib.pretty/Gateron_1u_v2.kicad_mod ?? giri-kicad-lib/switches_lib.pretty/Gateron_2.25u.kicad_mod ?? giri-kicad-lib/switches_lib.pretty/Gateron_2u.kicad_mod ?? giri-kicad-lib/switches_lib.pretty/Gateron_2u_v2.kicad_mod ?? giri-kicad-lib/switches_lib.pretty/MountingHole_2.2mm_M2_NoPad.kicad_mod ?? giri-kicad-lib/switches_lib.pretty/PGA2040_SMT_NO_SLOT.kicad_mod ?? giri-kicad-lib/switches_lib.pretty/PinHeader_1x02_P2.54mm_Vertical.kicad_mod ?? giri-kicad-lib/switches_lib.pretty/Switch_Cutout_MX_2.25u.kicad_mod ?? giri-kicad-lib/switches_lib.pretty/Switch_Cutout_MX_2u.kicad_mod ?? giri-kicad-lib/switches_lib.pretty/TEMT6000-sensor.kicad_mod ?? giri-kicad-lib/switches_lib.pretty/mouse-bite-2mm-slot.kicad_mod ?? "resources/1x2 stabilizer.png" ?? resources/Keymodule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
Parts:
- added Ba1: Conn_01x02_Socket, giri:PinHeader_1x02_P2.54mm_Vertical, F.Cu at (-5.37, 131.7)
- added F1: 500ma, Fuse:Fuse_0603_1608Metric, F.Cu at (6.05, -0.39)
- added JP1: SolderJumper_2_Bridged, Jumper:SolderJumper-2_P1.3mm_Bridged2Bar_RoundedPad1.0x1.5mm, F.Cu at (2.58, -0.67)
- added JP2: SolderJumper_2_Open, Jumper:SolderJumper-2_P1.3mm_Open_TrianglePad1.0x1.5mm, F.Cu at (-12.2, 8.22)
- added JP3: SolderJumper_2_Open, Jumper:SolderJumper-2_P1.3mm_Open_TrianglePad1.0x1.5mm, F.Cu at (-6.13, 72.8)
- added JP4: SolderJumper_2_Open, Jumper:SolderJumper-2_P1.3mm_Open_TrianglePad1.0x1.5mm, F.Cu at (-2.44, 48.2)
- added Sens2: ~, giri:TEMT6000-sensor, F.Cu at (-11.0, -8.98)
- J1: footprint giri:Debug_PinHeader_1x06_P2.00mm_Vertical -> giri:Debug_PinHeader_1x06_P2.54mm_Vertical
- S1, S10, S11, S12, S13, S14, S15, S16, S17, S18, S19, S2, S20, S21, S22, S23, S24, S25, S26, S27, S28, S29, S3, S30, S31, S32, S33, S34, S35, S36, S37, S38, S39, S4, S40, S41, S42, S43, S44, S45, S46, S47, S48, S49, S5, S50, S51, S52, S53, S54, S55, S56, S57, S58, S59, S6, S60, S61, S62, S65, S67, S68, S69, S7, S70, S71, S72, S8, S9: footprint giri:Gateron_1u -> giri:Gateron_1u_v2
- S63: footprint giri:Gateron_1u -> giri:Gateron_1.25u_v2
- S64, S66: footprint giri:Gateron_1u -> giri:Gateron_2u_v2
- SW1, SW2: footprint RP2040_Minimal:SW_XKB_TS_2030 -> giri:SW_B3U-3000P
- moved SW1 11.0 mm to (-11.7, 45.8), turned to -90 degrees
- moved Hs2 4.75 mm to (-9.50, 38.0)
- moved J1 3.99 mm to (-12.2, 59.3)
- moved R7 3.30 mm to (-8.65, 53.6), turned to -90 degrees
- moved SW2 2.89 mm to (-11.7, 52.9), turned to -90 degrees
- moved Sens1 1.26 mm to (-13.2, -5.57), turned to -100 degrees
- moved R9 1.10 mm to (-1.55, -0.41)
Connections:
- C5 pad 2: +5V -> VBUS
- J1 pad 1: SWCLK -> GND
- J1 pad 2: GND -> SWCLK
- J1 pad 6: +5V -> VDDH
- Jrp1 pad A2: +5V -> VBUS
- Jrp1 pad B1: unconnected-(Jrp1-GPIO0-PadB1) -> Net-(JP2-A)
- Jrp1 pad C1: unconnected-(Jrp1-GPIO1-PadC1) -> Net-(JP3-A)
- Jusb1 pad A4: +5V -> VBUS
- Jusb1 pad A9: +5V -> VBUS
- Jusb1 pad B4: +5V -> VBUS
- Jusb1 pad B9: +5V -> VBUS
Routing:
- net GND: track 0.00 -> 360.9 mm, vias 0 -> 37
- net /~{SDB}: track 5.52 -> 226.7 mm, vias 0 -> 2
- net SDA: track 2.69 -> 217.9 mm, vias 0 -> 2
- net SCL: track 2.60 -> 212.0 mm, vias 0 -> 2
- net CA2: track 191.2 -> 334.9 mm, vias 5 -> 6
- net BATT: track 0.00 -> 87.3 mm, vias 0 -> 2
- net +3V3: track 1589.7 -> 1654.8 mm, vias 23 -> 28
- net Net-(JP3-A): track 0.00 -> 64.1 mm, vias 0 -> 2
- net /RUN: track 30.8 -> 84.3 mm, vias 2 -> 3
- net VBUS: track 0.00 -> 32.7 mm
- net Net-(Q4-B): track 81.7 -> 104.8 mm, vias 4 -> 5
- net CA3: track 271.4 -> 293.1 mm
- net +5V: track 805.4 -> 784.1 mm, vias 27 -> 26
- net CA1: track 311.6 -> 332.1 mm
- net Net-(Q8-B): track 155.6 -> 139.6 mm
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- added copper zone on B.Cu, net GND
- added copper zone on F.Cu, net GND
Other:
- board size 309.5 x 190.8 mm -> 309.8 x 191 mm
