File: mx/rev3/switch-plate/switch-plate.kicad_sch (KiCad schematic)
At the start: 90 parts, among them J1 USB_C_Dummy

Commit message: M giri-kicad-lib/switches.kicad_sym  M giri-kicad-lib/switches_lib.pretty/Gateron_1u.kicad_mod  M giri-kicad-lib/switches_lib.pretty/Gateron_Sw_1u.kicad_mod  M giri-kicad-lib/switches_lib.pretty/PGA2040_SMT_WITH_SLOT.kicad_mod  M giri-kicad-lib/switches_lib.pretty/SW_B3U-3000P.kicad_mod M  mx/rev3/border.py M  mx/rev3/pcb/fp-lib-table M  mx/rev3/pcb/pcb.kicad_pcb M  mx/rev3/pcb/pcb.kicad_prl M  mx/rev3/pcb/pcb.kicad_pro M  mx/rev3/pcb/pcb.kicad_sch M  mx/rev3/place.py M  mx/rev3/switch-plate/switch-plate.kicad_pcb M  mx/rev3/switch-plate/switch-plate.kicad_prl M  mx/rev3/switch-plate/switch-plate.kicad_pro M  mx/rev3/switch-plate/switch-plate.kicad_sch M  mx/rev3/wrist-washer/wrist-washer.kicad_pcb M  mx/rev3/wrist-washer/wrist-washer.kicad_prl M  mx/rev3/wrist-washer/wrist-washer.kicad_pro M  mx/rev3/wrist-washer/wrist-washer.kicad_sch ?? giri-kicad-lib/switches_lib.pretty/ALS-PT19.kicad_mod ?? giri-kicad-lib/switches_lib.pretty/Debug_PinHeader_1x06_P2.00mm_Vertical.kicad_mod ?? giri-kicad-lib/switches_lib.pretty/Debug_PinHeader_1x06_P2.54mm_Vertical.kicad_mod ?? giri-kicad-lib/switches_lib.pretty/Gateron_1.25.kicad_mod ?? giri-kicad-lib/switches_lib.pretty/Gateron_1.25u_v2.kicad_mod ?? giri-kicad-lib/switches_lib.pretty/Gateron_1u_v2.kicad_mod ?? giri-kicad-lib/switches_lib.pretty/Gateron_2.25u.kicad_mod ?? giri-kicad-lib/switches_lib.pretty/Gateron_2u.kicad_mod ?? giri-kicad-lib/switches_lib.pretty/Gateron_2u_v2.kicad_mod ?? giri-kicad-lib/switches_lib.pretty/MountingHole_2.2mm_M2_NoPad.kicad_mod ?? giri-kicad-lib/switches_lib.pretty/PGA2040_SMT_NO_SLOT.kicad_mod ?? giri-kicad-lib/switches_lib.pretty/PinHeader_1x02_P2.54mm_Vertical.kicad_mod ?? giri-kicad-lib/switches_lib.pretty/Switch_Cutout_MX_2.25u.kicad_mod ?? giri-kicad-lib/switches_lib.pretty/Switch_Cutout_MX_2u.kicad_mod ?? giri-kicad-lib/switches_lib.pretty/TEMT6000-sensor.kicad_mod ?? giri-kicad-lib/switches_lib.pretty/mouse-bite-2mm-slot.kicad_mod ?? "resources/1x2 stabilizer.png" ?? resources/Keymodule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
Parts:
- removed J1: USB_C_Dummy, Giri_Library:USB_C_Receptacle_Outline_XKB_U262-16XN-4BVC11, symbol Giri:USB_C_Dummy
- added Hs18: ~, Giri_Library:MountingHole_2.2mm_M2_NoPad, symbol Giri:MountingHoleSMD
- added JLC1: JLC_Order_Num, Giri_Library:JLC_Order_Num, symbol Giri:JLC_Order_Num
- Hs1, Hs10, Hs11, Hs12, Hs13, Hs14, Hs15, Hs16, Hs17, Hs2, Hs3, Hs4, Hs5, Hs6, Hs7, Hs8, Hs9: value M1.6 -> ~; footprint Giri_Library:MountingHole_1.7mm_M1.6_NoPad -> Giri_Library:MountingHole_2.2mm_M2_NoPad
- S1, S10, S11, S12, S13, S14, S15, S16, S17, S18, S19, S2, S20, S21, S22, S23, S24, S25, S26, S27, S28, S29, S3, S30, S31, S32, S33, S34, S35, S36, S37, S38, S39, S4, S40, S41, S42, S43, S44, S45, S46, S47, S48, S49, S5, S50, S51, S52, S53, S54, S55, S56, S57, S58, S59, S6, S60, S61, S62, S63, S64, S65, S66, S67, S68, S69, S7, S70, S71, S72, S8, S9: footprint Giri_Library:Switch_Cutout_LoPro -> Giri_Library:Switch_Cutout_MX
