File: mx/rev3/switch-plate/switch-plate.kicad_pcb (KiCad board)
At the start: 2 copper layers, 296.1 x 118.1 mm, 90 parts, among them J1 USB_C_Dummy

Commit message: M giri-kicad-lib/switches.kicad_sym  M giri-kicad-lib/switches_lib.pretty/Gateron_1u.kicad_mod  M giri-kicad-lib/switches_lib.pretty/Gateron_Sw_1u.kicad_mod  M giri-kicad-lib/switches_lib.pretty/PGA2040_SMT_WITH_SLOT.kicad_mod  M giri-kicad-lib/switches_lib.pretty/SW_B3U-3000P.kicad_mod M  mx/rev3/border.py M  mx/rev3/pcb/fp-lib-table M  mx/rev3/pcb/pcb.kicad_pcb M  mx/rev3/pcb/pcb.kicad_prl M  mx/rev3/pcb/pcb.kicad_pro M  mx/rev3/pcb/pcb.kicad_sch M  mx/rev3/place.py M  mx/rev3/switch-plate/switch-plate.kicad_pcb M  mx/rev3/switch-plate/switch-plate.kicad_prl M  mx/rev3/switch-plate/switch-plate.kicad_pro M  mx/rev3/switch-plate/switch-plate.kicad_sch M  mx/rev3/wrist-washer/wrist-washer.kicad_pcb M  mx/rev3/wrist-washer/wrist-washer.kicad_prl M  mx/rev3/wrist-washer/wrist-washer.kicad_pro M  mx/rev3/wrist-washer/wrist-washer.kicad_sch ?? giri-kicad-lib/switches_lib.pretty/ALS-PT19.kicad_mod ?? giri-kicad-lib/switches_lib.pretty/Debug_PinHeader_1x06_P2.00mm_Vertical.kicad_mod ?? giri-kicad-lib/switches_lib.pretty/Debug_PinHeader_1x06_P2.54mm_Vertical.kicad_mod ?? giri-kicad-lib/switches_lib.pretty/Gateron_1.25.kicad_mod ?? giri-kicad-lib/switches_lib.pretty/Gateron_1.25u_v2.kicad_mod ?? giri-kicad-lib/switches_lib.pretty/Gateron_1u_v2.kicad_mod ?? giri-kicad-lib/switches_lib.pretty/Gateron_2.25u.kicad_mod ?? giri-kicad-lib/switches_lib.pretty/Gateron_2u.kicad_mod ?? giri-kicad-lib/switches_lib.pretty/Gateron_2u_v2.kicad_mod ?? giri-kicad-lib/switches_lib.pretty/MountingHole_2.2mm_M2_NoPad.kicad_mod ?? giri-kicad-lib/switches_lib.pretty/PGA2040_SMT_NO_SLOT.kicad_mod ?? giri-kicad-lib/switches_lib.pretty/PinHeader_1x02_P2.54mm_Vertical.kicad_mod ?? giri-kicad-lib/switches_lib.pretty/Switch_Cutout_MX_2.25u.kicad_mod ?? giri-kicad-lib/switches_lib.pretty/Switch_Cutout_MX_2u.kicad_mod ?? giri-kicad-lib/switches_lib.pretty/TEMT6000-sensor.kicad_mod ?? giri-kicad-lib/switches_lib.pretty/mouse-bite-2mm-slot.kicad_mod ?? "resources/1x2 stabilizer.png" ?? resources/Keymodule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
Parts:
- removed J1: USB_C_Dummy, Giri_Library:USB_C_Receptacle_Outline_XKB_U262-16XN-4BVC11
- added Hs18: ~, Giri_Library:MountingHole_2.2mm_M2_NoPad, F.Cu at (169.1, 83.6)
- added JLC1: JLC_Order_Num, Giri_Library:JLC_Order_Num, F.Cu at (246.8, 28.2)
- Hs1, Hs10, Hs11, Hs12, Hs13, Hs14, Hs15, Hs16, Hs17, Hs2, Hs3, Hs4, Hs5, Hs6, Hs7, Hs8, Hs9: value M1.6 -> ~; footprint Giri_Library:MountingHole_1.7mm_M1.6_NoPad -> Giri_Library:MountingHole_2.2mm_M2_NoPad
- S1, S10, S11, S12, S13, S14, S15, S16, S17, S18, S19, S2, S20, S21, S22, S23, S24, S25, S26, S27, S28, S29, S3, S30, S31, S32, S33, S34, S35, S36, S37, S38, S39, S4, S40, S41, S42, S43, S44, S45, S46, S47, S48, S49, S5, S50, S51, S52, S53, S54, S55, S56, S57, S58, S59, S6, S60, S61, S62, S63, S64, S65, S66, S67, S68, S69, S7, S70, S71, S72, S8, S9: footprint Giri_Library:Switch_Cutout_LoPro -> Giri_Library:Switch_Cutout_MX
- moved Hs4 228.0 mm to (47.5, -8.90)
- moved Hs3 226.1 mm to (-9.50, 79.2)
- moved Hs17 188.4 mm to (103.5, 87.4)
- moved Hs9 173.4 mm to (95.0, 27.9)
- moved Hs12 154.0 mm to (137.8, 46.9)
- moved Hs7 148.6 mm to (275.5, -8.90)
- moved Hs14 142.6 mm to (223.2, 65.9)
- moved Hs8 135.4 mm to (35.6, 26.5)
- moved Hs10 125.1 mm to (171.0, 27.9)
- moved Hs2 122.6 mm to (-9.50, 38.0)
- moved Hs6 110.8 mm to (199.5, -8.90)
- moved Hs5 95.3 mm to (123.5, -8.90)
- moved Hs16 79.0 mm to (289.8, 79.0)
- moved Hs13 62.2 mm to (62.7, 68.0)
- moved Hs15 61.7 mm to (291.6, 28.5)
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Other:
- board size 296.1 x 118.1 mm -> 309.8 x 120.6 mm

Commit message: M giri-kicad-lib/switches.kicad_sym  M giri-kicad-lib/switches_lib.pretty/C_0603_1608Metric.kicad_mod  M giri-kicad-lib/switches_lib.pretty/Gateron_1u.kicad_mod  M giri-kicad-lib/switches_lib.pretty/Gateron_Sw_1u.kicad_mod  M giri-kicad-lib/switches_lib.pretty/PGA2040_SMT_WITH_SLOT.kicad_mod  M giri-kicad-lib/switches_lib.pretty/Pad_Only_SMTSO_M2.kicad_mod  M giri-kicad-lib/switches_lib.pretty/SW_B3U-3000P.kicad_mod  D giri-kicad-lib/switches_lib.pretty/WristExtension.kicad_mod A  mx/rev3/Wrist-Plate2/Wrist-Plate2.kicad_pcb A  mx/rev3/Wrist-Plate2/Wrist-Plate2.kicad_prl A  mx/rev3/Wrist-Plate2/Wrist-Plate2.kicad_pro A  mx/rev3/Wrist-Plate2/Wrist-Plate2.kicad_sch A  mx/rev3/Wrist-Plate2/fp-lib-table M  mx/rev3/border.py R  mx/rev3/pcb/LED-Driver.kicad_sch -> mx/rev3/pcb-rev1/pcb/LED-Driver.kicad_sch R  mx/rev3/pcb/fp-lib-table -> mx/rev3/pcb-rev1/pcb/fp-lib-table R  mx/rev3/pcb/pcb-b.jpg -> mx/rev3/pcb-rev1/pcb/pcb-b.jpg R  mx/rev3/pcb/pcb.jpg -> mx/rev3/pcb-rev1/pcb/pcb.jpg R  mx/rev3/pcb/pcb.kicad_pcb -> mx/rev3/pcb-rev1/pcb/pcb.kicad_pcb A  mx/rev3/pcb-rev1/pcb/pcb.kicad_prl R  mx/rev3/pcb/pcb.kicad_pro -> mx/rev3/pcb-rev1/pcb/pcb.kicad_pro R  mx/rev3/pcb/pcb.kicad_sch -> mx/rev3/pcb-rev1/pcb/pcb.kicad_sch R  mx/rev3/pcb/sym-lib-table -> mx/rev3/pcb-rev1/pcb/sym-lib-table A  mx/rev3/pcb-rev2/pcb/LED-Driver.kicad_sch A  mx/rev3/pcb-rev2/pcb/fp-lib-table A  mx/rev3/pcb-rev2/pcb/pcb-b.jpg A  mx/rev3/pcb-rev2/pcb/pcb.jpg A  mx/rev3/pcb-rev2/pcb/pcb.kicad_pcb R  mx/rev3/pcb/pcb.kicad_prl -> mx/rev3/pcb-rev2/pcb/pcb.kicad_prl A  mx/rev3/pcb-rev2/pcb/pcb.kicad_pro A  mx/rev3/pcb-rev2/pcb/pcb.kicad_sch A  mx/rev3/pcb-rev2/pcb/sym-lib-table D  mx/rev3/pcb/.gitignore M  mx/rev3/place.py A  mx/rev3/switch-plate-wide/fp-lib-table A  mx/rev3/switch-plate-wide/switch-plate-wide.kicad_pcb A  mx/rev3/switch-plate-wide/switch-plate-wide.kicad_prl A  mx/rev3/switch-plate-wide/switch-plate-wide.kicad_pro A  mx/rev3/switch-plate-wide/switch-plate-wide.kicad_sch A  mx/rev3/switch-plat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
Parts:
- S64, S66: footprint Giri_Library:Switch_Cutout_MX -> Giri_Library:Switch_Cutout_MX_2u
- moved Hs18 3.00 mm to (168.2, 80.8)
- turned S64 to 69 degrees
- turned S66 to -70 degrees
Other:
- board size 309.8 x 120.6 mm -> 309.8 x 126.8 mm
