File: mx/rev3/wrist-washer/wrist-washer.kicad_sch (KiCad schematic)
At the start: 4 parts

Commit message: M giri-kicad-lib/switches.kicad_sym  M giri-kicad-lib/switches_lib.pretty/Gateron_1u.kicad_mod  M giri-kicad-lib/switches_lib.pretty/Gateron_Sw_1u.kicad_mod  M giri-kicad-lib/switches_lib.pretty/PGA2040_SMT_WITH_SLOT.kicad_mod  M giri-kicad-lib/switches_lib.pretty/SW_B3U-3000P.kicad_mod M  mx/rev3/border.py M  mx/rev3/pcb/fp-lib-table M  mx/rev3/pcb/pcb.kicad_pcb M  mx/rev3/pcb/pcb.kicad_prl M  mx/rev3/pcb/pcb.kicad_pro M  mx/rev3/pcb/pcb.kicad_sch M  mx/rev3/place.py M  mx/rev3/switch-plate/switch-plate.kicad_pcb M  mx/rev3/switch-plate/switch-plate.kicad_prl M  mx/rev3/switch-plate/switch-plate.kicad_pro M  mx/rev3/switch-plate/switch-plate.kicad_sch M  mx/rev3/wrist-washer/wrist-washer.kicad_pcb M  mx/rev3/wrist-washer/wrist-washer.kicad_prl M  mx/rev3/wrist-washer/wrist-washer.kicad_pro M  mx/rev3/wrist-washer/wrist-washer.kicad_sch ?? giri-kicad-lib/switches_lib.pretty/ALS-PT19.kicad_mod ?? giri-kicad-lib/switches_lib.pretty/Debug_PinHeader_1x06_P2.00mm_Vertical.kicad_mod ?? giri-kicad-lib/switches_lib.pretty/Debug_PinHeader_1x06_P2.54mm_Vertical.kicad_mod ?? giri-kicad-lib/switches_lib.pretty/Gateron_1.25.kicad_mod ?? giri-kicad-lib/switches_lib.pretty/Gateron_1.25u_v2.kicad_mod ?? giri-kicad-lib/switches_lib.pretty/Gateron_1u_v2.kicad_mod ?? giri-kicad-lib/switches_lib.pretty/Gateron_2.25u.kicad_mod ?? giri-kicad-lib/switches_lib.pretty/Gateron_2u.kicad_mod ?? giri-kicad-lib/switches_lib.pretty/Gateron_2u_v2.kicad_mod ?? giri-kicad-lib/switches_lib.pretty/MountingHole_2.2mm_M2_NoPad.kicad_mod ?? giri-kicad-lib/switches_lib.pretty/PGA2040_SMT_NO_SLOT.kicad_mod ?? giri-kicad-lib/switches_lib.pretty/PinHeader_1x02_P2.54mm_Vertical.kicad_mod ?? giri-kicad-lib/switches_lib.pretty/Switch_Cutout_MX_2.25u.kicad_mod ?? giri-kicad-lib/switches_lib.pretty/Switch_Cutout_MX_2u.kicad_mod ?? giri-kicad-lib/switches_lib.pretty/TEMT6000-sensor.kicad_mod ?? giri-kicad-lib/switches_lib.pretty/mouse-bite-2mm-slot.kicad_mod ?? "resources/1x2 stabilizer.png" ?? resources/Keymodule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
Parts:
- removed Hs1, Hs2, Hs3, Hs4: MountingHoleSMD, giri:SMTSO_M2_Hole_Only, symbol giri:MountingHoleSMD
- added H1, H2, H3, H4: MountingHole, giri:SMTSO_M2, symbol Mechanical:MountingHole
Changed lines of the file:
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@@
-(kicad_sch (version 20211123) (generator eeschema)
+(kicad_sch (version 20230121) (generator eeschema)
   (paper "A4")
-  (symbol (lib_id "giri:MountingHoleSMD") (at 128.27 63.5 0) (unit 1)
-    (in_bom yes) (on_board yes) (fields_autoplaced)
-    (property "Reference" "Hs3" (id 0) (at 130.81 62.6653 0)
+  (symbol (lib_id "Mechanical:MountingHole") (at 101.6 85.09 0) (unit 1)
+    (in_bom yes) (on_board yes) (dnp no) (fields_autoplaced)
+    (property "Reference" "H4" (at 104.14 83.82 0)
       (effects (font (size 1.27 1.27)) (justify left))
     )
-    (property "Value" "MountingHoleSMD" (id 1) (at 130.81 65.2022 0)
+    (property "Value" "MountingHole" (at 104.14 86.36 0)
+      (effects (font (size 1.27 1.27)) (justify left) hide)
+    )
+    (property "Footprint" "giri:SMTSO_M2" (at 101.6 85.09 0)
+      (effects (font (size 1.27 1.27)) hide)
+    )
+    (property "Datasheet" "~" (at 101.6 85.09 0)
+      (effects (font (size 1.27 1.27)) hide)
+    )
+    (instances
+      (project "wrist-washer"
+        (path "/241fa2b9-8a6e-48ae-b92e-75d72404d862"
+          (reference "H4") (unit 1)
+        )
+      )
+    )
+  )
+  (symbol (lib_id "Mechanical:MountingHole") (at 101.6 77.47 0) (unit 1)
+    (in_bom yes) (on_board yes) (dnp no) (fields_autoplaced)
+    (property "Reference" "H3" (at 104.14 76.2 0)
       (effects (font (size 1.27 1.27)) (justify left))
     )
-    (property "Footprint" "giri:SMTSO_M2_Hole_Only" (id 2) (at 128.27 63.5 0)
+    (property "Value" "MountingHole" (at 104.14 78.74 0)
+      (effects (font (size 1.27 1.27)) (justify left) hide)
+    )
+    (property "Footprint" "giri:SMTSO_M2" (at 101.6 77.47 0)
       (effects (font (size 1.27 1.27)) hide)
     )
-    (property "Datasheet" "~" (id 3) (at 128.27 63.5 0)
+    (property "Datasheet" "~" (at 101.6 77.47 0)
       (effects (font (size 1.27 1.27)) hide)
     )
+    (instances
+      (project "wrist-washer"
+        (path "/241fa2b9-8a6e-48ae-b92e-75d72404d862"
+          (reference "H3") (unit 1)
+        )
+      )
+    )
   )
-  (symbol (lib_id "giri:MountingHoleSMD") (at 157.48 63.5 0) (unit 1)
-    (in_bom yes) (on_board yes) (fields_autoplaced)
-    (property "Reference" "Hs4" (id 0) (at 160.02 62.6653 0)
+  (symbol (lib_id "Mechanical:MountingHole") (at 101.6 62.23 0) (unit 1)
+    (in_bom yes) (on_board yes) (dnp no) (fields_autoplaced)
+    (property "Reference" "H1" (at 104.14 60.96 0)
       (effects (font (size 1.27 1.27)) (justify left))
     )
-    (property "Value" "MountingHoleSMD" (id 1) (at 160.02 65.2022 0)
+    (property "Value" "MountingHole" (at 104.14 63.5 0)
+      (effects (font (size 1.27 1.27)) (justify left) hide)
+    )
+    (property "Footprint" "giri:SMTSO_M2" (at 101.6 62.23 0)
+      (effects (font (size 1.27 1.27)) hide)
+    )
+    (property "Datasheet" "~" (at 101.6 62.23 0)
+      (effects (font (size 1.27 1.27)) hide)
+    )
+    (instances
+      (project "wrist-washer"
+        (path "/241fa2b9-8a6e-48ae-b92e-75d72404d862"
+          (reference "H1") (unit 1)
+        )
+      )
+    )
+  )
+  (symbol (lib_id "Mechanical:MountingHole") (at 101.6 69.85 0) (unit 1)
+    (in_bom yes) (on_board yes) (dnp no) (fields_autoplaced)
+    (property "Reference" "H2" (at 104.14 68.58 0)
       (effects (font (size 1.27 1.27)) (justify left))
     )
-    (property "Footprint" "giri:SMTSO_M2_Hole_Only" (id 2) (at 157.48 63.5 0)
+    (property "Value" "MountingHole" (at 104.14 71.12 0)
+      (effects (font (size 1.27 1.27)) (justify left) hide)
+    )
+    (property "Footprint" "giri:SMTSO_M2" (at 101.6 69.85 0)
       (effects (font (size 1.27 1.27)) hide)
     )
-    (property "Datasheet" "~" (id 3) (at 157.48 63.5 0)
+    (property "Datasheet" "~" (at 101.6 69.85 0)
       (effects (font (size 1.27 1.27)) hide)
     )
-  )
-  (symbol (lib_id "giri:MountingHoleSMD") (at 68.58 63.5 0) (unit 1)
-    (in_bom yes) (on_board yes) (fields_autoplaced)
-    (property "Reference" "Hs1" (id 0) (at 71.12 62.6653 0)
-      (effects (font (size 1.27 1.27)) (justify left))
-    )
-    (property "Value" "MountingHoleSMD" (id 1) (at 71.12 65.2022 0)
-      (effects (font (size 1.27 1.27)) (justify left))
-    )
-    (property "Footprint" "giri:SMTSO_M2_Hole_Only" (id 2) (at 68.58 63.5 0)
-      (effects (font (size 1.27 1.27)) hide)
-    )
-    (property "Datasheet" "~" (id 3) (at 68.58 63.5 0)
-      (effects (font (size 1.27 1.27)) hide)
-    )
-  )
-  (symbol (lib_id "giri:MountingHoleSMD") (at 99.06 63.5 0) (unit 1)
-    (in_bom yes) (on_board yes) (fields_autoplaced)
-    (property "Reference" "Hs2" (id 0) (at 101.6 62.6653 0)
-      (effects (font (size 1.27 1.27)) (justify left))
-    )
-    (property "Value" "MountingHoleSMD" (id 1) (at 101.6 65.2022 0)
-      (effects (font (size 1.27 1.27)) (justify left))
-    )
-    (property "Footprint" "giri:SMTSO_M2_Hole_Only" (id 2) (at 99.06 63.5 0)
-      (effects (font (size 1.27 1.27)) hide)
-    )
-    (property "Datasheet" "~" (id 3) (at 99.06 63.5 0)
-      (effects (font (size 1.27 1.27)) hide)
+    (instances
+      (project "wrist-washer"
+        (path "/241fa2b9-8a6e-48ae-b92e-75d72404d862"
+          (reference "H2") (unit 1)
+        )
+      )
     )
   )
@@
     (path "/" (page "1"))
   )
-  (symbol_instances
-    (path "/bb465400-d056-48d8-8ba5-696842908e55"
-      (reference "Hs1") (unit 1) (value "MountingHoleSMD") (footprint "giri:SMTSO_M2_Hole_Only")
-    )
-    (path "/ce5edef7-4c7c-4b12-a180-5ffb7fa751ed"
-      (reference "Hs2") (unit 1) (value "MountingHoleSMD") (footprint "giri:SMTSO_M2_Hole_Only")
-    )
-    (path "/43e9b3ad-41a3-4e53-9d87-9c81955861ec"
-      (reference "Hs3") (unit 1) (value "MountingHoleSMD") (footprint "giri:SMTSO_M2_Hole_Only")
-    )
-    (path "/b7452ebf-8c1d-4909-a02b-50fbb747f63b"
-      (reference "Hs4") (unit 1) (value "MountingHoleSMD") (footprint "giri:SMTSO_M2_Hole_Only")
-    )
-  )
 )
