File: mx/rev3/wrist-washer/wrist-washer.kicad_pcb (KiCad board)
At the start: 2 copper layers, 88 x 65 mm, 4 parts

Commit message: M giri-kicad-lib/switches.kicad_sym  M giri-kicad-lib/switches_lib.pretty/Gateron_1u.kicad_mod  M giri-kicad-lib/switches_lib.pretty/Gateron_Sw_1u.kicad_mod  M giri-kicad-lib/switches_lib.pretty/PGA2040_SMT_WITH_SLOT.kicad_mod  M giri-kicad-lib/switches_lib.pretty/SW_B3U-3000P.kicad_mod M  mx/rev3/border.py M  mx/rev3/pcb/fp-lib-table M  mx/rev3/pcb/pcb.kicad_pcb M  mx/rev3/pcb/pcb.kicad_prl M  mx/rev3/pcb/pcb.kicad_pro M  mx/rev3/pcb/pcb.kicad_sch M  mx/rev3/place.py M  mx/rev3/switch-plate/switch-plate.kicad_pcb M  mx/rev3/switch-plate/switch-plate.kicad_prl M  mx/rev3/switch-plate/switch-plate.kicad_pro M  mx/rev3/switch-plate/switch-plate.kicad_sch M  mx/rev3/wrist-washer/wrist-washer.kicad_pcb M  mx/rev3/wrist-washer/wrist-washer.kicad_prl M  mx/rev3/wrist-washer/wrist-washer.kicad_pro M  mx/rev3/wrist-washer/wrist-washer.kicad_sch ?? giri-kicad-lib/switches_lib.pretty/ALS-PT19.kicad_mod ?? giri-kicad-lib/switches_lib.pretty/Debug_PinHeader_1x06_P2.00mm_Vertical.kicad_mod ?? giri-kicad-lib/switches_lib.pretty/Debug_PinHeader_1x06_P2.54mm_Vertical.kicad_mod ?? giri-kicad-lib/switches_lib.pretty/Gateron_1.25.kicad_mod ?? giri-kicad-lib/switches_lib.pretty/Gateron_1.25u_v2.kicad_mod ?? giri-kicad-lib/switches_lib.pretty/Gateron_1u_v2.kicad_mod ?? giri-kicad-lib/switches_lib.pretty/Gateron_2.25u.kicad_mod ?? giri-kicad-lib/switches_lib.pretty/Gateron_2u.kicad_mod ?? giri-kicad-lib/switches_lib.pretty/Gateron_2u_v2.kicad_mod ?? giri-kicad-lib/switches_lib.pretty/MountingHole_2.2mm_M2_NoPad.kicad_mod ?? giri-kicad-lib/switches_lib.pretty/PGA2040_SMT_NO_SLOT.kicad_mod ?? giri-kicad-lib/switches_lib.pretty/PinHeader_1x02_P2.54mm_Vertical.kicad_mod ?? giri-kicad-lib/switches_lib.pretty/Switch_Cutout_MX_2.25u.kicad_mod ?? giri-kicad-lib/switches_lib.pretty/Switch_Cutout_MX_2u.kicad_mod ?? giri-kicad-lib/switches_lib.pretty/TEMT6000-sensor.kicad_mod ?? giri-kicad-lib/switches_lib.pretty/mouse-bite-2mm-slot.kicad_mod ?? "resources/1x2 stabilizer.png" ?? resources/Keymodule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
Parts:
- removed Hs1, Hs2, Hs3, Hs4: MountingHoleSMD, giri:SMTSO_M2_Hole_Only
- added H1: MountingHole, giri:SMTSO_M2, F.Cu at (3.43, 3.43)
- added H2: MountingHole, giri:SMTSO_M2, F.Cu at (3.43, 10.9)
- added H3: MountingHole, giri:SMTSO_M2, F.Cu at (3.43, 18.3)
- added H4: MountingHole, giri:SMTSO_M2, F.Cu at (3.43, 25.8)
Other:
- board outline removed
Changed lines of the file:
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@@
-(kicad_pcb (version 20211014) (generator pcbnew)
+(kicad_pcb (version 20221018) (generator pcbnew)
   (general
     (thickness 1.6)
@@
     (pcbplotparams
       (layerselection 0x00010fc_ffffffff)
+      (plot_on_all_layers_selection 0x0000000_00000000)
       (disableapertmacros false)
       (usegerberextensions true)
@@
       (usegerberadvancedattributes false)
       (creategerberjobfile false)
-      (svguseinch false)
+      (dashed_line_dash_ratio 12.000000)
+      (dashed_line_gap_ratio 3.000000)
       (svgprecision 6)
-      (excludeedgelayer true)
       (plotframeref false)
       (viasonmask false)
@@
   )
   (net 0 "")
-  (footprint "giri:SMTSO_M2_Hole_Only" (layer "F.Cu")
-    (at 6.5 44.025)
+  (footprint "giri:SMTSO_M2" (layer "F.Cu")
+    (at 3.427924 25.777924)
     (descr "Mounting Hole 2.2mm, M2")
     (tags "mounting hole 2.2mm m2")
     (property "Sheetfile" "wrist-washer.kicad_sch")
     (property "Sheetname" "")
+    (property "ki_description" "Mounting Hole without connection")
+    (property "ki_keywords" "mounting hole")
     (attr exclude_from_pos_files)
-    (fp_text reference "Hs4" (at 0 -3.2) (layer "Dwgs.User")
-      (effects (font (size 1 1) (thickness 0.15)))
+    (fp_text reference "H4" (at 0 -3.2) (layer "Dwgs.User")
+        (effects (font (size 1 1) (thickness 0.15)))
     )
-    (fp_text value "MountingHoleSMD" (at 0 3.2) (layer "F.Fab")
-      (effects (font (size 1 1) (thickness 0.15)))
+    (fp_text value "MountingHole" (at 0 3.2) (layer "F.Fab")
+        (effects (font (size 1 1) (thickness 0.15)))
     )
-    (fp_text user "${REFERENCE}" (at -2.4 -3.7) (layer "F.Fab")
-      (effects (font (size 1 1) (thickness 0.15)))
+    (fp_text user "${REFERENCE}" (at 0 0) (layer "F.Fab")
+        (effects (font (size 1 1) (thickness 0.15)))
     )
-    (fp_circle (center 0 0) (end 3.2 0) (layer "F.CrtYd") (width 0.05) (fill none))
-    (fp_circle (center 0 0) (end 0 0) (layer "B.Fab") (width 0.1) (fill none))
-    (fp_circle (center 0 0) (end 2.78 0) (layer "B.Fab") (width 0.1) (fill none))
-    (pad "" np_thru_hole circle (at 0 0) (size 5.7 5.7) (drill 5.7) (layers F&B.Cu))
+    (fp_circle (center 0 0) (end 3.2 0)
+      (stroke (width 0.05) (type solid)) (fill none) (layer "F.CrtYd"))
+    (fp_circle (center 0 0) (end 0 0)
+      (stroke (width 0.1) (type solid)) (fill none) (layer "B.Fab"))
+    (fp_circle (center 0 0) (end 2.78 0)
+      (stroke (width 0.1) (type solid)) (fill none) (layer "B.Fab"))
+    (pad "" thru_hole circle (at 0 0) (size 6.2 6.2) (drill 3.73) (layers "*.Cu" "*.Mask"))
   )
-  (footprint "giri:SMTSO_M2_Hole_Only" (layer "F.Cu")
-    (at 81.5 44.025)
+  (footprint "giri:SMTSO_M2" (layer "F.Cu")
+    (at 3.427924 10.877924)
     (descr "Mounting Hole 2.2mm, M2")
     (tags "mounting hole 2.2mm m2")
     (property "Sheetfile" "wrist-washer.kicad_sch")
     (property "Sheetname" "")
+    (property "ki_description" "Mounting Hole without connection")
+    (property "ki_keywords" "mounting hole")
     (attr exclude_from_pos_files)
-    (fp_text reference "Hs1" (at 0 -3.2) (layer "Dwgs.User")
-      (effects (font (size 1 1) (thickness 0.15)))
+    (fp_text reference "H2" (at 0 -3.2) (layer "Dwgs.User")
+        (effects (font (size 1 1) (thickness 0.15)))
     )
-    (fp_text value "MountingHoleSMD" (at 0 3.2) (layer "F.Fab")
-      (effects (font (size 1 1) (thickness 0.15)))
+    (fp_text value "MountingHole" (at 0 3.2) (layer "F.Fab")
+        (effects (font (size 1 1) (thickness 0.15)))
     )
-    (fp_text user "${REFERENCE}" (at -2.4 -3.7) (layer "F.Fab")
-      (effects (font (size 1 1) (thickness 0.15)))
+    (fp_text user "${REFERENCE}" (at 0 0) (layer "F.Fab")
+        (effects (font (size 1 1) (thickness 0.15)))
     )
-    (fp_circle (center 0 0) (end 3.2 0) (layer "F.CrtYd") (width 0.05) (fill none))
-    (fp_circle (center 0 0) (end 0 0) (layer "B.Fab") (width 0.1) (fill none))
-    (fp_circle (center 0 0) (end 2.78 0) (layer "B.Fab") (width 0.1) (fill none))
-    (pad "" np_thru_hole circle (at 0 0) (size 5.7 5.7) (drill 5.7) (layers F&B.Cu))
+    (fp_circle (center 0 0) (end 3.2 0)
+      (stroke (width 0.05) (type solid)) (fill none) (layer "F.CrtYd"))
+    (fp_circle (center 0 0) (end 0 0)
+      (stroke (width 0.1) (type solid)) (fill none) (layer "B.Fab"))
+    (fp_circle (center 0 0) (end 2.78 0)
+      (stroke (width 0.1) (type solid)) (fill none) (layer "B.Fab"))
+    (pad "" thru_hole circle (at 0 0) (size 6.2 6.2) (drill 3.73) (layers "*.Cu" "*.Mask"))
   )
-  (footprint "giri:SMTSO_M2_Hole_Only" (layer "F.Cu")
-    (at 81.5 96.025)
+  (footprint "giri:SMTSO_M2" (layer "F.Cu")
+    (at 3.427924 18.327924)
     (descr "Mounting Hole 2.2mm, M2")
     (tags "mounting hole 2.2mm m2")
     (property "Sheetfile" "wrist-washer.kicad_sch")
     (property "Sheetname" "")
+    (property "ki_description" "Mounting Hole without connection")
+    (property "ki_keywords" "mounting hole")
     (attr exclude_from_pos_files)
-    (fp_text reference "Hs2" (at 0 -3.2) (layer "Dwgs.User")
-      (effects (font (size 1 1) (thickness 0.15)))
+    (fp_text reference "H3" (at 0 -3.2) (layer "Dwgs.User")
+        (effects (font (size 1 1) (thickness 0.15)))
     )
-    (fp_text value "MountingHoleSMD" (at 0 3.2) (layer "F.Fab")
-      (effects (font (size 1 1) (thickness 0.15)))
+    (fp_text value "MountingHole" (at 0 3.2) (layer "F.Fab")
+        (effects (font (size 1 1) (thickness 0.15)))
     )
-    (fp_text user "${REFERENCE}" (at -2.4 -3.7) (layer "F.Fab")
-      (effects (font (size 1 1) (thickness 0.15)))
+    (fp_text user "${REFERENCE}" (at 0 0) (layer "F.Fab")
+        (effects (font (size 1 1) (thickness 0.15)))
     )
-    (fp_circle (center 0 0) (end 3.2 0) (layer "F.CrtYd") (width 0.05) (fill none))
-    (fp_circle (center 0 0) (end 0 0) (layer "B.Fab") (width 0.1) (fill none))
-    (fp_circle (center 0 0) (end 2.78 0) (layer "B.Fab") (width 0.1) (fill none))
-    (pad "" np_thru_hole circle (at 0 0) (size 5.7 5.7) (drill 5.7) (layers F&B.Cu))
+    (fp_circle (center 0 0) (end 3.2 0)
+      (stroke (width 0.05) (type solid)) (fill none) (layer "F.CrtYd"))
+    (fp_circle (center 0 0) (end 0 0)
+      (stroke (width 0.1) (type solid)) (fill none) (layer "B.Fab"))
+    (fp_circle (center 0 0) (end 2.78 0)
+      (stroke (width 0.1) (type solid)) (fill none) (layer "B.Fab"))
+    (pad "" thru_hole circle (at 0 0) (size 6.2 6.2) (drill 3.73) (layers "*.Cu" "*.Mask"))
   )
-  (footprint "giri:SMTSO_M2_Hole_Only" (layer "F.Cu")
-    (at 6.5 96.025)
+  (footprint "giri:SMTSO_M2" (layer "F.Cu")
+    (at 3.427924 3.427924)
     (descr "Mounting Hole 2.2mm, M2")
     (tags "mounting hole 2.2mm m2")
     (property "Sheetfile" "wrist-washer.kicad_sch")
     (property "Sheetname" "")
+    (property "ki_description" "Mounting Hole without connection")
+    (property "ki_keywords" "mounting hole")
     (attr exclude_from_pos_files)
-    (fp_text reference "Hs3" (at 0 -3.2) (layer "Dwgs.User")
-      (effects (font (size 1 1) (thickness 0.15)))
+    (fp_text reference "H1" (at 0 -3.2) (layer "Dwgs.User")
+        (effects (font (size 1 1) (thickness 0.15)))
     )
-    (fp_text value "MountingHoleSMD" (at 0 3.2) (layer "F.Fab")
-      (effects (font (size 1 1) (thickness 0.15)))
+    (fp_text value "MountingHole" (at 0 3.2) (layer "F.Fab")
+        (effects (font (size 1 1) (thickness 0.15)))
     )
-    (fp_text user "${REFERENCE}" (at -2.4 -3.7) (layer "F.Fab")
-      (effects (font (size 1 1) (thickness 0.15)))
+    (fp_text user "${REFERENCE}" (at 0 0) (layer "F.Fab")
+        (effects (font (size 1 1) (thickness 0.15)))
     )
-    (fp_circle (center 0 0) (end 3.2 0) (layer "F.CrtYd") (width 0.05) (fill none))
-    (fp_circle (center 0 0) (end 2.78 0) (layer "B.Fab") (width 0.1) (fill none))
-    (fp_circle (center 0 0) (end 0 0) (layer "B.Fab") (width 0.1) (fill none))
-    (pad "" np_thru_hole circle (at 0 0) (size 5.7 5.7) (drill 5.7) (layers F&B.Cu))
+    (fp_circle (center 0 0) (end 3.2 0)
+      (stroke (width 0.05) (type solid)) (fill none) (layer "F.CrtYd"))
+    (fp_circle (center 0 0) (end 0 0)
+      (stroke (width 0.1) (type solid)) (fill none) (layer "B.Fab"))
+    (fp_circle (center 0 0) (end 2.78 0)
+      (stroke (width 0.1) (type solid)) (fill none) (layer "B.Fab"))
+    (pad "" thru_hole circle (at 0 0) (size 6.2 6.2) (drill 3.73) (layers "*.Cu" "*.Mask"))
   )
-  (gr_arc (start 69 48.525) (mid 74.656854 50.868146) (end 77 56.525) (layer "Edge.Cuts") (width 0.1))
-  (gr_arc (start 0 45.525) (mid 2.343146 39.868146) (end 8 37.525) (layer "Edge.Cuts") (width 0.1))
-  (gr_arc (start 80 37.525) (mid 85.656854 39.868146) (end 88 45.525) (layer "Edge.Cuts") (width 0.1))
-  (gr_line (start 0 94.525) (end 0 45.525) (layer "Edge.Cuts") (width 0.1))
-  (gr_line (start 69 48.525) (end 19 48.525) (layer "Edge.Cuts") (width 0.1))
-  (gr_line (start 80 37.525) (end 8 37.525) (layer "Edge.Cuts") (width 0.1))
-  (gr_arc (start 19 91.525) (mid 13.343146 89.181854) (end 11 83.525) (layer "Edge.Cuts") (width 0.1))
-  (gr_line (start 77 56.525) (end 77 83.525) (layer "Edge.Cuts") (width 0.1))
-  (gr_line (start 88 45.525) (end 88 94.525) (layer "Edge.Cuts") (width 0.1))
-  (gr_line (start 69 91.525) (end 19 91.525) (layer "Edge.Cuts") (width 0.1))
-  (gr_line (start 80 102.525) (end 8 102.525) (layer "Edge.Cuts") (width 0.1))
-  (gr_arc (start 88 94.525) (mid 85.656854 100.181854) (end 80 102.525) (layer "Edge.Cuts") (width 0.1))
-  (gr_line (start 11 83.525) (end 11 56.525) (layer "Edge.Cuts") (width 0.1))
-  (gr_arc (start 77 83.525) (mid 74.656854 89.181854) (end 69 91.525) (layer "Edge.Cuts") (width 0.1))
-  (gr_arc (start 11 56.525) (mid 13.343146 50.868146) (end 19 48.525) (layer "Edge.Cuts") (width 0.1))
-  (gr_arc (start 8 102.525) (mid 2.343146 100.181854) (end 0 94.525) (layer "Edge.Cuts") (width 0.1))
   (via (at 76.15 40.4) (size 0.8) (drill 0.4) (layers "F.Cu" "B.Cu") (net 0))
 )

Commit message: M giri-kicad-lib/switches.kicad_sym  M giri-kicad-lib/switches_lib.pretty/C_0603_1608Metric.kicad_mod  M giri-kicad-lib/switches_lib.pretty/Gateron_1u.kicad_mod  M giri-kicad-lib/switches_lib.pretty/Gateron_Sw_1u.kicad_mod  M giri-kicad-lib/switches_lib.pretty/PGA2040_SMT_WITH_SLOT.kicad_mod  M giri-kicad-lib/switches_lib.pretty/Pad_Only_SMTSO_M2.kicad_mod  M giri-kicad-lib/switches_lib.pretty/SW_B3U-3000P.kicad_mod  D giri-kicad-lib/switches_lib.pretty/WristExtension.kicad_mod A  mx/rev3/Wrist-Plate2/Wrist-Plate2.kicad_pcb A  mx/rev3/Wrist-Plate2/Wrist-Plate2.kicad_prl A  mx/rev3/Wrist-Plate2/Wrist-Plate2.kicad_pro A  mx/rev3/Wrist-Plate2/Wrist-Plate2.kicad_sch A  mx/rev3/Wrist-Plate2/fp-lib-table M  mx/rev3/border.py R  mx/rev3/pcb/LED-Driver.kicad_sch -> mx/rev3/pcb-rev1/pcb/LED-Driver.kicad_sch R  mx/rev3/pcb/fp-lib-table -> mx/rev3/pcb-rev1/pcb/fp-lib-table R  mx/rev3/pcb/pcb-b.jpg -> mx/rev3/pcb-rev1/pcb/pcb-b.jpg R  mx/rev3/pcb/pcb.jpg -> mx/rev3/pcb-rev1/pcb/pcb.jpg R  mx/rev3/pcb/pcb.kicad_pcb -> mx/rev3/pcb-rev1/pcb/pcb.kicad_pcb A  mx/rev3/pcb-rev1/pcb/pcb.kicad_prl R  mx/rev3/pcb/pcb.kicad_pro -> mx/rev3/pcb-rev1/pcb/pcb.kicad_pro R  mx/rev3/pcb/pcb.kicad_sch -> mx/rev3/pcb-rev1/pcb/pcb.kicad_sch R  mx/rev3/pcb/sym-lib-table -> mx/rev3/pcb-rev1/pcb/sym-lib-table A  mx/rev3/pcb-rev2/pcb/LED-Driver.kicad_sch A  mx/rev3/pcb-rev2/pcb/fp-lib-table A  mx/rev3/pcb-rev2/pcb/pcb-b.jpg A  mx/rev3/pcb-rev2/pcb/pcb.jpg A  mx/rev3/pcb-rev2/pcb/pcb.kicad_pcb R  mx/rev3/pcb/pcb.kicad_prl -> mx/rev3/pcb-rev2/pcb/pcb.kicad_prl A  mx/rev3/pcb-rev2/pcb/pcb.kicad_pro A  mx/rev3/pcb-rev2/pcb/pcb.kicad_sch A  mx/rev3/pcb-rev2/pcb/sym-lib-table D  mx/rev3/pcb/.gitignore M  mx/rev3/place.py A  mx/rev3/switch-plate-wide/fp-lib-table A  mx/rev3/switch-plate-wide/switch-plate-wide.kicad_pcb A  mx/rev3/switch-plate-wide/switch-plate-wide.kicad_prl A  mx/rev3/switch-plate-wide/switch-plate-wide.kicad_pro A  mx/rev3/switch-plate-wide/switch-plate-wide.kicad_sch A  mx/rev3/switch-plat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
Parts:
- moved H3 99.3 mm to (82.8, 78.0)
- moved H4 79.4 mm to (82.8, 27.0)
- moved H2 67.3 mm to (8.80, 78.0)
- moved H1 24.2 mm to (8.80, 27.0)
Routing:
- net (no net): vias 1 -> 0
Other:
- board outline added: 88 x 65 mm
Changed lines of the file:
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@@
   (net 0 "")
   (footprint "giri:SMTSO_M2" (layer "F.Cu")
-    (at 3.427924 25.777924)
+    (at 82.8 27)
     (descr "Mounting Hole 2.2mm, M2")
     (tags "mounting hole 2.2mm m2")
@@
   )
   (footprint "giri:SMTSO_M2" (layer "F.Cu")
-    (at 3.427924 10.877924)
+    (at 8.8 78)
     (descr "Mounting Hole 2.2mm, M2")
     (tags "mounting hole 2.2mm m2")
@@
   )
   (footprint "giri:SMTSO_M2" (layer "F.Cu")
-    (at 3.427924 18.327924)
+    (at 82.8 78)
     (descr "Mounting Hole 2.2mm, M2")
     (tags "mounting hole 2.2mm m2")
@@
   )
   (footprint "giri:SMTSO_M2" (layer "F.Cu")
-    (at 3.427924 3.427924)
+    (at 8.8 27)
     (descr "Mounting Hole 2.2mm, M2")
     (tags "mounting hole 2.2mm m2")
@@
     (pad "" thru_hole circle (at 0 0) (size 6.2 6.2) (drill 3.73) (layers "*.Cu" "*.Mask"))
   )
-  (via (at 76.15 40.4) (size 0.8) (drill 0.4) (layers "F.Cu" "B.Cu") (net 0))
+  (gr_line (start 45.7 31) (end 18.8 31)
+    (stroke (width 0.1) (type default)) (layer "Edge.Cuts"))
+  (gr_line (start 10.1 85) (end 81.8 85)
+    (stroke (width 0.1) (type default)) (layer "Edge.Cuts"))
+  (gr_line (start 1.8 76.9) (end 1.8 77)
+    (stroke (width 0.1) (type default)) (layer "Edge.Cuts"))
+  (gr_line (start 45.9 31) (end 72.8 31)
+    (stroke (width 0.1) (type default)) (layer "Edge.Cuts"))
+  (gr_line (start 89.8 76.8) (end 89.8 76.7)
+    (stroke (width 0.1) (type default)) (layer "Edge.Cuts"))
+  (gr_line (start 45.9 74) (end 72.8 74)
+    (stroke (width 0.1) (type default)) (layer "Edge.Cuts"))
+  (gr_line (start 89.8 76.8) (end 89.8 76.9)
+    (stroke (width 0.1) (type default)) (layer "Edge.Cuts"))
+  (gr_line (start 9.9 85) (end 9.8 85)
+    (stroke (width 0.1) (type default)) (layer "Edge.Cuts"))
+  (gr_line (start 78.8 52.6) (end 78.8 68)
+    (stroke (width 0.1) (type default)) (layer "Edge.Cuts"))
+  (gr_line (start 45.8 31) (end 45.9 31)
+    (stroke (width 0.1) (type default)) (layer "Edge.Cuts"))
+  (gr_line (start 1.8 76.8) (end 1.8 76.7)
+    (stroke (width 0.1) (type default)) (layer "Edge.Cuts"))
+  (gr_line (start 81.7 20) (end 81.8 20)
+    (stroke (width 0.1) (type default)) (layer "Edge.Cuts"))
+  (gr_line (start 89.8 76.7) (end 89.8 28)
+    (stroke (width 0.1) (type default)) (layer "Edge.Cuts"))
+  (gr_line (start 1.8 76.8) (end 1.8 76.9)
+    (stroke (width 0.1) (type default)) (layer "Edge.Cuts"))
+  (gr_line (start 45.7 74) (end 18.8 74)
+    (stroke (width 0.1) (type default)) (layer "Edge.Cuts"))
+  (gr_arc (start 81.8 20) (mid 87.456854 22.343146) (end 89.8 28)
+    (stroke (width 0.1) (type default)) (layer "Edge.Cuts"))
+  (gr_line (start 78.8 52.5) (end 78.8 52.4)
+    (stroke (width 0.1) (type default)) (layer "Edge.Cuts"))
+  (gr_line (start 12.8 52.4) (end 12.8 37)
+    (stroke (width 0.1) (type default)) (layer "Edge.Cuts"))
+  (gr_line (start 78.8 52.4) (end 78.8 37)
+    (stroke (width 0.1) (type default)) (layer "Edge.Cuts"))
+  (gr_line (start 45.8 74) (end 45.7 74)
+    (stroke (width 0.1) (type default)) (layer "Edge.Cuts"))
+  (gr_line (start 9.9 20) (end 9.8 20)
+    (stroke (width 0.1) (type default)) (layer "Edge.Cuts"))
+  (gr_line (start 81.6 20) (end 81.7 20)
+    (stroke (width 0.1) (type default)) (layer "Edge.Cuts"))
+  (gr_arc (start 78.8 68) (mid 77.042641 72.242641) (end 72.8 74)
+    (stroke (width 0.1) (type default)) (layer "Edge.Cuts"))
+  (gr_line (start 12.8 52.5) (end 12.8 52.6)
+    (stroke (width 0.1) (type default)) (layer "Edge.Cuts"))
+  (gr_line (start 10 85) (end 10.1 85)
+    (stroke (width 0.1) (type default)) (layer "Edge.Cuts"))
+  (gr_line (start 12.8 52.6) (end 12.8 68)
+    (stroke (width 0.1) (type default)) (layer "Edge.Cuts"))
+  (gr_line (start 89.8 76.9) (end 89.8 77)
+    (stroke (width 0.1) (type default)) (layer "Edge.Cuts"))
+  (gr_line (start 81.6 20) (end 10 20)
+    (stroke (width 0.1) (type default)) (layer "Edge.Cuts"))
+  (gr_line (start 10 20) (end 9.9 20)
+    (stroke (width 0.1) (type default)) (layer "Edge.Cuts"))
+  (gr_line (start 45.8 74) (end 45.9 74)
+    (stroke (width 0.1) (type default)) (layer "Edge.Cuts"))
+  (gr_arc (start 18.8 74) (mid 14.557359 72.242641) (end 12.8 68)
+    (stroke (width 0.1) (type default)) (layer "Edge.Cuts"))
+  (gr_line (start 45.8 31) (end 45.7 31)
+    (stroke (width 0.1) (type default)) (layer "Edge.Cuts"))
+  (gr_line (start 78.8 52.5) (end 78.8 52.6)
+    (stroke (width 0.1) (type default)) (layer "Edge.Cuts"))
+  (gr_arc (start 12.8 37) (mid 14.557359 32.757359) (end 18.8 31)
+    (stroke (width 0.1) (type default)) (layer "Edge.Cuts"))
+  (gr_arc (start 89.8 77) (mid 87.456854 82.656854) (end 81.8 85)
+    (stroke (width 0.1) (type default)) (layer "Edge.Cuts"))
+  (gr_line (start 10 85) (end 9.9 85)
+    (stroke (width 0.1) (type default)) (layer "Edge.Cuts"))
+  (gr_arc (start 1.8 28) (mid 4.143146 22.343146) (end 9.8 20)
+    (stroke (width 0.1) (type default)) (layer "Edge.Cuts"))
+  (gr_arc (start 72.8 31) (mid 77.042641 32.757359) (end 78.8 37)
+    (stroke (width 0.1) (type default)) (layer "Edge.Cuts"))
+  (gr_line (start 12.8 52.5) (end 12.8 52.4)
+    (stroke (width 0.1) (type default)) (layer "Edge.Cuts"))
+  (gr_arc (start 9.8 85) (mid 4.143145 82.656855) (end 1.8 77)
+    (stroke (width 0.1) (type default)) (layer "Edge.Cuts"))
+  (gr_line (start 1.8 76.7) (end 1.8 28)
+    (stroke (width 0.1) (type default)) (layer "Edge.Cuts"))
 )
