File: mx/rev3/Wrist-Plate2/Wrist-Plate2.kicad_sch (KiCad schematic)
At the start: 4 parts

Commit message: M giri-kicad-lib/switches.kicad_sym  M giri-kicad-lib/switches_lib.pretty/C_0603_1608Metric.kicad_mod  M giri-kicad-lib/switches_lib.pretty/Gateron_1u.kicad_mod  M giri-kicad-lib/switches_lib.pretty/Gateron_Sw_1u.kicad_mod  M giri-kicad-lib/switches_lib.pretty/PGA2040_SMT_WITH_SLOT.kicad_mod  M giri-kicad-lib/switches_lib.pretty/Pad_Only_SMTSO_M2.kicad_mod  M giri-kicad-lib/switches_lib.pretty/SW_B3U-3000P.kicad_mod  D giri-kicad-lib/switches_lib.pretty/WristExtension.kicad_mod A  mx/rev3/Wrist-Plate2/Wrist-Plate2.kicad_pcb A  mx/rev3/Wrist-Plate2/Wrist-Plate2.kicad_prl A  mx/rev3/Wrist-Plate2/Wrist-Plate2.kicad_pro A  mx/rev3/Wrist-Plate2/Wrist-Plate2.kicad_sch A  mx/rev3/Wrist-Plate2/fp-lib-table M  mx/rev3/border.py R  mx/rev3/pcb/LED-Driver.kicad_sch -> mx/rev3/pcb-rev1/pcb/LED-Driver.kicad_sch R  mx/rev3/pcb/fp-lib-table -> mx/rev3/pcb-rev1/pcb/fp-lib-table R  mx/rev3/pcb/pcb-b.jpg -> mx/rev3/pcb-rev1/pcb/pcb-b.jpg R  mx/rev3/pcb/pcb.jpg -> mx/rev3/pcb-rev1/pcb/pcb.jpg R  mx/rev3/pcb/pcb.kicad_pcb -> mx/rev3/pcb-rev1/pcb/pcb.kicad_pcb A  mx/rev3/pcb-rev1/pcb/pcb.kicad_prl R  mx/rev3/pcb/pcb.kicad_pro -> mx/rev3/pcb-rev1/pcb/pcb.kicad_pro R  mx/rev3/pcb/pcb.kicad_sch -> mx/rev3/pcb-rev1/pcb/pcb.kicad_sch R  mx/rev3/pcb/sym-lib-table -> mx/rev3/pcb-rev1/pcb/sym-lib-table A  mx/rev3/pcb-rev2/pcb/LED-Driver.kicad_sch A  mx/rev3/pcb-rev2/pcb/fp-lib-table A  mx/rev3/pcb-rev2/pcb/pcb-b.jpg A  mx/rev3/pcb-rev2/pcb/pcb.jpg A  mx/rev3/pcb-rev2/pcb/pcb.kicad_pcb R  mx/rev3/pcb/pcb.kicad_prl -> mx/rev3/pcb-rev2/pcb/pcb.kicad_prl A  mx/rev3/pcb-rev2/pcb/pcb.kicad_pro A  mx/rev3/pcb-rev2/pcb/pcb.kicad_sch A  mx/rev3/pcb-rev2/pcb/sym-lib-table D  mx/rev3/pcb/.gitignore M  mx/rev3/place.py A  mx/rev3/switch-plate-wide/fp-lib-table A  mx/rev3/switch-plate-wide/switch-plate-wide.kicad_pcb A  mx/rev3/switch-plate-wide/switch-plate-wide.kicad_prl A  mx/rev3/switch-plate-wide/switch-plate-wide.kicad_pro A  mx/rev3/switch-plate-wide/switch-plate-wide.kicad_sch A  mx/rev3/switch-plat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
Parts:
- H1, H2, H3, H4: footprint giri:Pad_Only_SMTSO_M2 -> giri:SMTSO_M2_Pad_M2_hole
Connections:
- no-connect marks 1 -> 0
Other:
- title: Wrist Support -> (none)
Changed lines of the file:
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@@
 (kicad_sch (version 20230121) (generator eeschema)
   (paper "A4")
-  (title_block
-    (title "Wrist Support")
-    (date "2022-10-28")
+  (junction (at 52.07 49.53) (diameter 0) (color 0 0 0 0)
   )
-  (junction (at 87.63 44.45) (diameter 0) (color 0 0 0 0)
+  (junction (at 64.77 49.53) (diameter 0) (color 0 0 0 0)
   )
-  (junction (at 115.57 44.45) (diameter 0) (color 0 0 0 0)
+  (junction (at 76.2 49.53) (diameter 0) (color 0 0 0 0)
   )
-  (junction (at 101.6 44.45) (diameter 0) (color 0 0 0 0)
-  )
-  (no_connect (at 121.92 87.63))
-  (wire (pts (xy 72.39 44.45) (xy 87.63 44.45))
+  (wire (pts (xy 52.07 49.53) (xy 64.77 49.53))
     (stroke (width 0) (type default))
   )
-  (wire (pts (xy 115.57 44.45) (xy 115.57 48.26))
+  (wire (pts (xy 46.99 49.53) (xy 52.07 49.53))
     (stroke (width 0) (type default))
   )
-  (wire (pts (xy 115.57 48.26) (xy 64.77 48.26))
+  (wire (pts (xy 46.99 53.34) (xy 46.99 49.53))
     (stroke (width 0) (type default))
   )
-  (wire (pts (xy 64.77 48.26) (xy 64.77 60.96))
+  (wire (pts (xy 76.2 49.53) (xy 87.63 49.53))
     (stroke (width 0) (type default))
   )
-  (wire (pts (xy 87.63 44.45) (xy 101.6 44.45))
+  (wire (pts (xy 64.77 49.53) (xy 76.2 49.53))
     (stroke (width 0) (type default))
   )
-  (wire (pts (xy 101.6 44.45) (xy 115.57 44.45))
-    (stroke (width 0) (type default))
-  )
-  (symbol (lib_id "Mechanical:MountingHole_Pad") (at 72.39 41.91 0) (unit 1)
+  (symbol (lib_id "Mechanical:MountingHole_Pad") (at 64.77 46.99 0) (unit 1)
     (in_bom yes) (on_board yes) (dnp no) (fields_autoplaced)
-    (property "Reference" "H1" (at 74.93 39.37 0)
+    (property "Reference" "H2" (at 67.31 44.45 0)
       (effects (font (size 1.27 1.27)) (justify left))
     )
-    (property "Value" "MountingHole_Pad" (at 74.93 41.91 0)
+    (property "Value" "MountingHole_Pad" (at 67.31 46.99 0)
       (effects (font (size 1.27 1.27)) (justify left))
     )
-    (property "Footprint" "giri:Pad_Only_SMTSO_M2" (at 72.39 41.91 0)
+    (property "Footprint" "giri:SMTSO_M2_Pad_M2_hole" (at 64.77 46.99 0)
       (effects (font (size 1.27 1.27)) hide)
     )
-    (property "Datasheet" "~" (at 72.39 41.91 0)
+    (property "Datasheet" "~" (at 64.77 46.99 0)
       (effects (font (size 1.27 1.27)) hide)
     )
     (pin "1")
     (instances
-      (project "wrist-support"
-        (path "/4d3f447a-24fb-41a6-b3d4-979062f8252f"
+      (project "Wrist-Plate2"
+        (path "/6b65d7b3-c212-451c-a973-07a4b1081395"
+          (reference "H2") (unit 1)
+        )
+      )
+    )
+  )
+  (symbol (lib_id "Mechanical:MountingHole_Pad") (at 52.07 46.99 0) (unit 1)
+    (in_bom yes) (on_board yes) (dnp no) (fields_autoplaced)
+    (property "Reference" "H1" (at 54.61 44.45 0)
+      (effects (font (size 1.27 1.27)) (justify left))
+    )
+    (property "Value" "MountingHole_Pad" (at 54.61 46.99 0)
+      (effects (font (size 1.27 1.27)) (justify left))
+    )
+    (property "Footprint" "giri:SMTSO_M2_Pad_M2_hole" (at 52.07 46.99 0)
+      (effects (font (size 1.27 1.27)) hide)
+    )
+    (property "Datasheet" "~" (at 52.07 46.99 0)
+      (effects (font (size 1.27 1.27)) hide)
+    )
+    (pin "1")
+    (instances
+      (project "Wrist-Plate2"
+        (path "/6b65d7b3-c212-451c-a973-07a4b1081395"
           (reference "H1") (unit 1)
         )
@@
     )
   )
-  (symbol (lib_id "Mechanical:MountingHole_Pad") (at 115.57 41.91 0) (unit 1)
+  (symbol (lib_id "Mechanical:MountingHole_Pad") (at 76.2 46.99 0) (unit 1)
     (in_bom yes) (on_board yes) (dnp no) (fields_autoplaced)
-    (property "Reference" "H4" (at 118.11 39.37 0)
+    (property "Reference" "H3" (at 78.74 44.45 0)
       (effects (font (size 1.27 1.27)) (justify left))
     )
-    (property "Value" "MountingHole_Pad" (at 118.11 41.91 0)
+    (property "Value" "MountingHole_Pad" (at 78.74 46.99 0)
       (effects (font (size 1.27 1.27)) (justify left))
     )
-    (property "Footprint" "giri:Pad_Only_SMTSO_M2" (at 115.57 41.91 0)
+    (property "Footprint" "giri:SMTSO_M2_Pad_M2_hole" (at 76.2 46.99 0)
       (effects (font (size 1.27 1.27)) hide)
     )
-    (property "Datasheet" "~" (at 115.57 41.91 0)
+    (property "Datasheet" "~" (at 76.2 46.99 0)
       (effects (font (size 1.27 1.27)) hide)
     )
     (pin "1")
     (instances
-      (project "wrist-support"
-        (path "/4d3f447a-24fb-41a6-b3d4-979062f8252f"
-          (reference "H4") (unit 1)
+      (project "Wrist-Plate2"
+        (path "/6b65d7b3-c212-451c-a973-07a4b1081395"
+          (reference "H3") (unit 1)
         )
       )
     )
   )
-  (symbol (lib_id "Mechanical:MountingHole_Pad") (at 87.63 41.91 0) (unit 1)
+  (symbol (lib_id "power:GND") (at 46.99 53.34 0) (unit 1)
     (in_bom yes) (on_board yes) (dnp no) (fields_autoplaced)
-    (property "Reference" "H2" (at 90.17 39.37 0)
-      (effects (font (size 1.27 1.27)) (justify left))
-    )
-    (property "Value" "MountingHole_Pad" (at 90.17 41.91 0)
-      (effects (font (size 1.27 1.27)) (justify left))
-    )
-    (property "Footprint" "giri:Pad_Only_SMTSO_M2" (at 87.63 41.91 0)
+    (property "Reference" "#PWR01" (at 46.99 59.69 0)
       (effects (font (size 1.27 1.27)) hide)
     )
-    (property "Datasheet" "~" (at 87.63 41.91 0)
+    (property "Value" "GND" (at 46.99 57.7834 0)
+      (effects (font (size 1.27 1.27)))
+    )
+    (property "Footprint" "" (at 46.99 53.34 0)
       (effects (font (size 1.27 1.27)) hide)
     )
-    (pin "1")
-    (instances
-      (project "wrist-support"
-        (path "/4d3f447a-24fb-41a6-b3d4-979062f8252f"
-          (reference "H2") (unit 1)
-        )
-      )
-    )
-  )
-  (symbol (lib_id "power:GND") (at 64.77 60.96 0) (unit 1)
-    (in_bom yes) (on_board yes) (dnp no) (fields_autoplaced)
-    (property "Reference" "#PWR01" (at 64.77 67.31 0)
-      (effects (font (size 1.27 1.27)) hide)
-    )
-    (property "Value" "GND" (at 64.77 65.4034 0)
-      (effects (font (size 1.27 1.27)))
-    )
-    (property "Footprint" "" (at 64.77 60.96 0)
-      (effects (font (size 1.27 1.27)) hide)
-    )
-    (property "Datasheet" "" (at 64.77 60.96 0)
+    (property "Datasheet" "" (at 46.99 53.34 0)
       (effects (font (size 1.27 1.27)) hide)
     )
@@
         )
       )
+      (project "Wrist-Plate2"
+        (path "/6b65d7b3-c212-451c-a973-07a4b1081395"
+          (reference "#PWR01") (unit 1)
+        )
+      )
     )
   )
-  (symbol (lib_id "Mechanical:MountingHole_Pad") (at 101.6 41.91 0) (unit 1)
+  (symbol (lib_id "Mechanical:MountingHole_Pad") (at 87.63 46.99 0) (unit 1)
     (in_bom yes) (on_board yes) (dnp no) (fields_autoplaced)
-    (property "Reference" "H3" (at 104.14 39.37 0)
+    (property "Reference" "H4" (at 90.17 44.45 0)
       (effects (font (size 1.27 1.27)) (justify left))
     )
-    (property "Value" "MountingHole_Pad" (at 104.14 41.91 0)
+    (property "Value" "MountingHole_Pad" (at 90.17 46.99 0)
       (effects (font (size 1.27 1.27)) (justify left))
     )
-    (property "Footprint" "giri:Pad_Only_SMTSO_M2" (at 101.6 41.91 0)
+    (property "Footprint" "giri:SMTSO_M2_Pad_M2_hole" (at 87.63 46.99 0)
       (effects (font (size 1.27 1.27)) hide)
     )
-    (property "Datasheet" "~" (at 101.6 41.91 0)
+    (property "Datasheet" "~" (at 87.63 46.99 0)
       (effects (font (size 1.27 1.27)) hide)
     )
     (pin "1")
     (instances
-      (project "wrist-support"
-        (path "/4d3f447a-24fb-41a6-b3d4-979062f8252f"
-          (reference "H3") (unit 1)
+      (project "Wrist-Plate2"
+        (path "/6b65d7b3-c212-451c-a973-07a4b1081395"
+          (reference "H4") (unit 1)
         )
       )
