File: mx/rev3/pcb-rev1/pcb/pcb.kicad_pcb (KiCad board)
At the start: 2 copper layers, 309.8 x 191 mm, 279 parts, among them J1 Conn_01x06_Socket, Q1 MMBT3904, Q10 MMBT3904, Q11 MMBT3904, Q12 MMBT3904, Q13 MMBT3904, Q14 MMBT3904, Q15 MMBT3904, Q2 MMBT3904, Q3 MMBT3904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

Commit message: M giri-kicad-lib/switches.kicad_sym  M giri-kicad-lib/switches_lib.pretty/C_0603_1608Metric.kicad_mod  M giri-kicad-lib/switches_lib.pretty/Gateron_1u.kicad_mod  M giri-kicad-lib/switches_lib.pretty/Gateron_Sw_1u.kicad_mod  M giri-kicad-lib/switches_lib.pretty/PGA2040_SMT_WITH_SLOT.kicad_mod  M giri-kicad-lib/switches_lib.pretty/Pad_Only_SMTSO_M2.kicad_mod  M giri-kicad-lib/switches_lib.pretty/SW_B3U-3000P.kicad_mod  D giri-kicad-lib/switches_lib.pretty/WristExtension.kicad_mod A  mx/rev3/Wrist-Plate2/Wrist-Plate2.kicad_pcb A  mx/rev3/Wrist-Plate2/Wrist-Plate2.kicad_prl A  mx/rev3/Wrist-Plate2/Wrist-Plate2.kicad_pro A  mx/rev3/Wrist-Plate2/Wrist-Plate2.kicad_sch A  mx/rev3/Wrist-Plate2/fp-lib-table M  mx/rev3/border.py R  mx/rev3/pcb/LED-Driver.kicad_sch -> mx/rev3/pcb-rev1/pcb/LED-Driver.kicad_sch R  mx/rev3/pcb/fp-lib-table -> mx/rev3/pcb-rev1/pcb/fp-lib-table R  mx/rev3/pcb/pcb-b.jpg -> mx/rev3/pcb-rev1/pcb/pcb-b.jpg R  mx/rev3/pcb/pcb.jpg -> mx/rev3/pcb-rev1/pcb/pcb.jpg R  mx/rev3/pcb/pcb.kicad_pcb -> mx/rev3/pcb-rev1/pcb/pcb.kicad_pcb A  mx/rev3/pcb-rev1/pcb/pcb.kicad_prl R  mx/rev3/pcb/pcb.kicad_pro -> mx/rev3/pcb-rev1/pcb/pcb.kicad_pro R  mx/rev3/pcb/pcb.kicad_sch -> mx/rev3/pcb-rev1/pcb/pcb.kicad_sch R  mx/rev3/pcb/sym-lib-table -> mx/rev3/pcb-rev1/pcb/sym-lib-table A  mx/rev3/pcb-rev2/pcb/LED-Driver.kicad_sch A  mx/rev3/pcb-rev2/pcb/fp-lib-table A  mx/rev3/pcb-rev2/pcb/pcb-b.jpg A  mx/rev3/pcb-rev2/pcb/pcb.jpg A  mx/rev3/pcb-rev2/pcb/pcb.kicad_pcb R  mx/rev3/pcb/pcb.kicad_prl -> mx/rev3/pcb-rev2/pcb/pcb.kicad_prl A  mx/rev3/pcb-rev2/pcb/pcb.kicad_pro A  mx/rev3/pcb-rev2/pcb/pcb.kicad_sch A  mx/rev3/pcb-rev2/pcb/sym-lib-table D  mx/rev3/pcb/.gitignore M  mx/rev3/place.py A  mx/rev3/switch-plate-wide/fp-lib-table A  mx/rev3/switch-plate-wide/switch-plate-wide.kicad_pcb A  mx/rev3/switch-plate-wide/switch-plate-wide.kicad_prl A  mx/rev3/switch-plate-wide/switch-plate-wide.kicad_pro A  mx/rev3/switch-plate-wide/switch-plate-wide.kicad_sch A  mx/rev3/switch-plat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
Parts:
- Ba1: footprint giri:PinHeader_1x02_P2.54mm_Vertical -> giri:Battery_Pads_2x2.0x2.0mm
- J1: footprint giri:Debug_PinHeader_1x06_P2.54mm_Vertical -> Connector_JST:JST_SH_SM06B-SRSS-TB_1x06-1MP_P1.00mm_Horizontal
- moved Hs18 21.1 mm to (166.2, 104.5)
- moved Hs17 18.0 mm to (109.2, 104.5)
- moved J1 6.54 mm to (-10.5, 65.6), turned to -90 degrees
- moved Ba1 3.73 mm to (-8.98, 132.6), turned to 0 degrees
- moved C1 2.48 mm to (151.9, 77.0)
- moved C2 2.48 mm to (153.9, 76.4)
- moved C3 2.48 mm to (155.5, 76.4)
- moved R3 2.48 mm to (158.7, 76.4)
- moved R4 2.48 mm to (157.1, 76.4)
- moved R5 2.48 mm to (160.3, 76.4)
- moved Hs3 1.90 mm to (-7.60, 79.2)
- moved H1 1.41 mm to (-8.25, 119.5)
- moved H2 1.41 mm to (-8.25, 172.5)
- moved H3 1.41 mm to (67.8, 172.5)
- moved H4 1.41 mm to (67.8, 119.5)
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Connections:
- J1 pad 1: GND -> +3V3
- J1 pad 2: SWCLK -> SWDIO
- J1 pad 3: SWDIO -> SWCLK
- J1 pad 4: +3V3 -> /RUN
- J1 pad 5: /RUN -> GND
Routing:
- net /R5_SINK: track 226.4 -> 242.7 mm
- net CB1: track 456.4 -> 465.6 mm, vias 10 -> 9
- net Net-(S63-IR_K): track 22.2 -> 30.4 mm
- net +3V3: track 1654.8 -> 1647.3 mm, vias 28 -> 29
- net /RUN: track 84.3 -> 77.0 mm
- net BATT: track 87.3 -> 94.0 mm
- net GND: track 360.9 -> 367.4 mm, vias 37 -> 35
- net CB2: track 412.5 -> 406.2 mm
- net /~{SDB}: track 226.7 -> 220.5 mm
- net CB6: track 342.8 -> 347.3 mm
- net Net-(S62-IR_K): track 25.9 -> 29.9 mm
- net SWDIO: track 67.4 -> 64.1 mm
- net Net-(S66-IR_K): track 42.2 -> 45.2 mm
- net +5V: track 784.1 -> 781.1 mm
- net /R_EXT: track 7.43 -> 4.99 mm
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Other:
- outline, holes or cut-outs redrawn
