File: mx/rev3/bottom-cover/pcb/pcb.kicad_sch (KiCad schematic)
At the start: 99 parts

Commit message: M  giri-kicad-lib/switches_lib.pretty/Gateron_1.25u_v2.kicad_mod M  giri-kicad-lib/switches_lib.pretty/Gateron_1u_v2.kicad_mod M  giri-kicad-lib/switches_lib.pretty/Gateron_2u_v2.kicad_mod A  giri-kicad-lib/switches_lib.pretty/SMTSO_M2_FrontPad_M2_hole.kicad_mod A  giri-kicad-lib/switches_lib.pretty/Switch_Cutout2_MX.kicad_mod A  giri-kicad-lib/switches_lib.pretty/Switch_Cutout2_MX_1.25u.kicad_mod A  giri-kicad-lib/switches_lib.pretty/Switch_Cutout2_MX_2u.kicad_mod M  mx/rev3/bottom-cover/pcb/pcb.kicad_pcb M  mx/rev3/bottom-cover/pcb/pcb.kicad_prl M  mx/rev3/bottom-cover/pcb/pcb.kicad_sch M  mx/rev3/pcb-rev2/pcb/pcb.kicad_pcb M  mx/rev3/pcb-rev2/pcb/pcb.kicad_prl M  mx/rev3/pcb-rev2/pcb/pcb.kicad_sch M  mx/rev3/switch-plate-wide/fp-lib-table M  mx/rev3/switch-plate-wide/switch-plate-wide.kicad_pcb M  mx/rev3/switch-plate-wide/switch-plate-wide.kicad_sch A  mx/rev4/notes D  nrfStamp/rev1/pcb/~pcb.kicad_sch.lck D  rp2040stamp/rev2/pcb/~pcb.kicad_sch.lck M  rp2040stamp/rev3/pcb/fp-lib-table M  rp2040stamp/rev3/pcb/pcb.kicad_pcb M  rp2040stamp/rev3/pcb/pcb.kicad_prl M  rp2040stamp/rev3/pcb/pcb.kicad_sch M  rp2040stamp/rev3/pcb/sym-lib-table
Parts:
- H1, H2, H3, H4, H5, H6, H7, H8, Hs1, Hs10, Hs11, Hs12, Hs13, Hs14, Hs15, Hs16, Hs17, Hs18, Hs2, Hs3, Hs4, Hs5, Hs6, Hs7, Hs8, Hs9: footprint giri:SMTSO_M2_Front_Pad -> giri:SMTSO_M2_FrontPad_M2_hole
Changed lines of the file:
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@@
       (effects (font (size 1.27 1.27)) (justify left))
     )
-    (property "Footprint" "giri:SMTSO_M2_Front_Pad" (at 142.875 109.22 0)
+    (property "Footprint" "giri:SMTSO_M2_FrontPad_M2_hole" (at 142.875 109.22 0)
       (effects (font (size 1.27 1.27)) hide)
     )
@@
       (effects (font (size 1.27 1.27)) (justify left))
     )
-    (property "Footprint" "giri:SMTSO_M2_Front_Pad" (at 177.165 116.84 0)
+    (property "Footprint" "giri:SMTSO_M2_FrontPad_M2_hole" (at 177.165 116.84 0)
       (effects (font (size 1.27 1.27)) hide)
     )
@@
       (effects (font (size 1.27 1.27)) (justify left))
     )
-    (property "Footprint" "giri:SMTSO_M2_Front_Pad" (at 165.735 109.22 0)
+    (property "Footprint" "giri:SMTSO_M2_FrontPad_M2_hole" (at 165.735 109.22 0)
       (effects (font (size 1.27 1.27)) hide)
     )
@@
       (effects (font (size 1.27 1.27)) (justify left) hide)
     )
-    (property "Footprint" "giri:SMTSO_M2_Front_Pad" (at 69.215 139.7 0)
+    (property "Footprint" "giri:SMTSO_M2_FrontPad_M2_hole" (at 69.215 139.7 0)
       (effects (font (size 1.27 1.27)) hide)
     )
@@
       (effects (font (size 1.27 1.27)) (justify left) hide)
     )
-    (property "Footprint" "giri:SMTSO_M2_Front_Pad" (at 69.215 120.65 0)
+    (property "Footprint" "giri:SMTSO_M2_FrontPad_M2_hole" (at 69.215 120.65 0)
       (effects (font (size 1.27 1.27)) hide)
     )
@@
       (effects (font (size 1.27 1.27)) (justify left) hide)
     )
-    (property "Footprint" "giri:SMTSO_M2_Front_Pad" (at 80.645 139.7 0)
+    (property "Footprint" "giri:SMTSO_M2_FrontPad_M2_hole" (at 80.645 139.7 0)
       (effects (font (size 1.27 1.27)) hide)
     )
@@
       (effects (font (size 1.27 1.27)) (justify left) hide)
     )
-    (property "Footprint" "giri:SMTSO_M2_Front_Pad" (at 69.215 111.76 0)
+    (property "Footprint" "giri:SMTSO_M2_FrontPad_M2_hole" (at 69.215 111.76 0)
       (effects (font (size 1.27 1.27)) hide)
     )
@@
       (effects (font (size 1.27 1.27)) (justify left) hide)
     )
-    (property "Footprint" "giri:SMTSO_M2_Front_Pad" (at 103.505 120.65 0)
+    (property "Footprint" "giri:SMTSO_M2_FrontPad_M2_hole" (at 103.505 120.65 0)
       (effects (font (size 1.27 1.27)) hide)
     )
@@
       (effects (font (size 1.27 1.27)) (justify left))
     )
-    (property "Footprint" "giri:SMTSO_M2_Front_Pad" (at 165.735 116.84 0)
+    (property "Footprint" "giri:SMTSO_M2_FrontPad_M2_hole" (at 165.735 116.84 0)
       (effects (font (size 1.27 1.27)) hide)
     )
@@
       (effects (font (size 1.27 1.27)) (justify left) hide)
     )
-    (property "Footprint" "giri:SMTSO_M2_Front_Pad" (at 114.935 120.65 0)
+    (property "Footprint" "giri:SMTSO_M2_FrontPad_M2_hole" (at 114.935 120.65 0)
       (effects (font (size 1.27 1.27)) hide)
     )
@@
       (effects (font (size 1.27 1.27)) (justify left) hide)
     )
-    (property "Footprint" "giri:SMTSO_M2_Front_Pad" (at 92.075 120.65 0)
+    (property "Footprint" "giri:SMTSO_M2_FrontPad_M2_hole" (at 92.075 120.65 0)
       (effects (font (size 1.27 1.27)) hide)
     )
@@
       (effects (font (size 1.27 1.27)) (justify left) hide)
     )
-    (property "Footprint" "giri:SMTSO_M2_Front_Pad" (at 114.935 111.76 0)
+    (property "Footprint" "giri:SMTSO_M2_FrontPad_M2_hole" (at 114.935 111.76 0)
       (effects (font (size 1.27 1.27)) hide)
     )
@@
       (effects (font (size 1.27 1.27)) (justify left) hide)
     )
-    (property "Footprint" "giri:SMTSO_M2_Front_Pad" (at 103.505 111.76 0)
+    (property "Footprint" "giri:SMTSO_M2_FrontPad_M2_hole" (at 103.505 111.76 0)
       (effects (font (size 1.27 1.27)) hide)
     )
@@
       (effects (font (size 1.27 1.27)) (justify left))
     )
-    (property "Footprint" "giri:SMTSO_M2_Front_Pad" (at 142.875 116.84 0)
+    (property "Footprint" "giri:SMTSO_M2_FrontPad_M2_hole" (at 142.875 116.84 0)
       (effects (font (size 1.27 1.27)) hide)
     )
@@
       (effects (font (size 1.27 1.27)) (justify left) hide)
     )
-    (property "Footprint" "giri:SMTSO_M2_Front_Pad" (at 80.645 129.54 0)
+    (property "Footprint" "giri:SMTSO_M2_FrontPad_M2_hole" (at 80.645 129.54 0)
       (effects (font (size 1.27 1.27)) hide)
     )
@@
       (effects (font (size 1.27 1.27)) (justify left) hide)
     )
-    (property "Footprint" "giri:SMTSO_M2_Front_Pad" (at 69.215 129.54 0)
+    (property "Footprint" "giri:SMTSO_M2_FrontPad_M2_hole" (at 69.215 129.54 0)
       (effects (font (size 1.27 1.27)) hide)
     )
@@
       (effects (font (size 1.27 1.27)) (justify left))
     )
-    (property "Footprint" "giri:SMTSO_M2_Front_Pad" (at 154.305 109.22 0)
+    (property "Footprint" "giri:SMTSO_M2_FrontPad_M2_hole" (at 154.305 109.22 0)
       (effects (font (size 1.27 1.27)) hide)
     )
@@
       (effects (font (size 1.27 1.27)) (justify left) hide)
     )
-    (property "Footprint" "giri:SMTSO_M2_Front_Pad" (at 114.935 129.54 0)
+    (property "Footprint" "giri:SMTSO_M2_FrontPad_M2_hole" (at 114.935 129.54 0)
       (effects (font (size 1.27 1.27)) hide)
     )
@@
       (effects (font (size 1.27 1.27)) (justify left))
     )
-    (property "Footprint" "giri:SMTSO_M2_Front_Pad" (at 154.305 116.84 0)
+    (property "Footprint" "giri:SMTSO_M2_FrontPad_M2_hole" (at 154.305 116.84 0)
       (effects (font (size 1.27 1.27)) hide)
     )
@@
       (effects (font (size 1.27 1.27)) (justify left) hide)
     )
-    (property "Footprint" "giri:SMTSO_M2_Front_Pad" (at 80.645 120.65 0)
+    (property "Footprint" "giri:SMTSO_M2_FrontPad_M2_hole" (at 80.645 120.65 0)
       (effects (font (size 1.27 1.27)) hide)
     )
@@
       (effects (font (size 1.27 1.27)) (justify left) hide)
     )
-    (property "Footprint" "giri:SMTSO_M2_Front_Pad" (at 92.075 111.76 0)
+    (property "Footprint" "giri:SMTSO_M2_FrontPad_M2_hole" (at 92.075 111.76 0)
       (effects (font (size 1.27 1.27)) hide)
     )
@@
       (effects (font (size 1.27 1.27)) (justify left))
     )
-    (property "Footprint" "giri:SMTSO_M2_Front_Pad" (at 177.165 109.22 0)
+    (property "Footprint" "giri:SMTSO_M2_FrontPad_M2_hole" (at 177.165 109.22 0)
       (effects (font (size 1.27 1.27)) hide)
     )
@@
       (effects (font (size 1.27 1.27)) (justify left) hide)
     )
-    (property "Footprint" "giri:SMTSO_M2_Front_Pad" (at 92.075 129.54 0)
+    (property "Footprint" "giri:SMTSO_M2_FrontPad_M2_hole" (at 92.075 129.54 0)
       (effects (font (size 1.27 1.27)) hide)
     )
@@
       (effects (font (size 1.27 1.27)) (justify left) hide)
     )
-    (property "Footprint" "giri:SMTSO_M2_Front_Pad" (at 92.075 139.7 0)
+    (property "Footprint" "giri:SMTSO_M2_FrontPad_M2_hole" (at 92.075 139.7 0)
       (effects (font (size 1.27 1.27)) hide)
     )
@@
       (effects (font (size 1.27 1.27)) (justify left) hide)
     )
-    (property "Footprint" "giri:SMTSO_M2_Front_Pad" (at 80.645 111.76 0)
+    (property "Footprint" "giri:SMTSO_M2_FrontPad_M2_hole" (at 80.645 111.76 0)
       (effects (font (size 1.27 1.27)) hide)
     )
@@
       (effects (font (size 1.27 1.27)) (justify left) hide)
     )
-    (property "Footprint" "giri:SMTSO_M2_Front_Pad" (at 103.505 129.54 0)
-      (effects (font (size 1.27 1.27)) hide)
-    )
+    (property "Footprint" "giri:SMTSO_M2_FrontPad_M2_hole" (at 103.505 129.54 0)
+      (effects (font (size 1.27 1.27)) hide)
+    )
