File: mx/rev3/pcb-rev2/pcb/pcb.kicad_pcb (KiCad board)
At the start: 2 copper layers, 309.8 x 191 mm, 280 parts, among them J1 Conn_01x06_Socket, Q1 MMBT3904, Q10 MMBT3904, Q11 MMBT3904, Q12 MMBT3904, Q13 MMBT3904, Q14 MMBT3904, Q15 MMBT3904, Q2 MMBT3904, Q3 MMBT3904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

Commit message: A  NuvotonStamp/rev1/fp-lib-table A  NuvotonStamp/rev1/rev1.kicad_pcb A  NuvotonStamp/rev1/rev1.kicad_prl R  mx/rev3/wrist-washer/wrist-washer.kicad_pro -> NuvotonStamp/rev1/rev1.kicad_pro A  NuvotonStamp/rev1/rev1.kicad_sch A  NuvotonStamp/rev1/sym-lib-table M  giri-kicad-lib/switches.kicad_sym A  giri-kicad-lib/switches_lib.pretty/ALS-PT19.kicad_mod A  giri-kicad-lib/switches_lib.pretty/Battery_Pads_2x2.0x2.0mm.kicad_mod M  giri-kicad-lib/switches_lib.pretty/C_0603_1608Metric.kicad_mod A  giri-kicad-lib/switches_lib.pretty/Debug_PinHeader_1x06_P2.00mm_Vertical.kicad_mod A  giri-kicad-lib/switches_lib.pretty/Debug_PinHeader_1x06_P2.54mm_Vertical.kicad_mod A  giri-kicad-lib/switches_lib.pretty/Gateron_1.25.kicad_mod A  giri-kicad-lib/switches_lib.pretty/Gateron_1.25u_v2.kicad_mod M  giri-kicad-lib/switches_lib.pretty/Gateron_1u.kicad_mod A  giri-kicad-lib/switches_lib.pretty/Gateron_1u_v2.kicad_mod A  giri-kicad-lib/switches_lib.pretty/Gateron_2.25u.kicad_mod A  giri-kicad-lib/switches_lib.pretty/Gateron_2u.kicad_mod A  giri-kicad-lib/switches_lib.pretty/Gateron_2u_v2.kicad_mod M  giri-kicad-lib/switches_lib.pretty/Gateron_Sw_1u.kicad_mod A  giri-kicad-lib/switches_lib.pretty/MINEW-MS88SF3-AllPads.kicad_mod M  giri-kicad-lib/switches_lib.pretty/MINEW-MS88SF3.kicad_mod A  giri-kicad-lib/switches_lib.pretty/MountingHole_2.1mm_M2_NoPad.kicad_mod A  giri-kicad-lib/switches_lib.pretty/MountingHole_2.2mm_M2_NoPad.kicad_mod A  giri-kicad-lib/switches_lib.pretty/MountingHole_2.2mm_M2_SmallPad.kicad_mod A  giri-kicad-lib/switches_lib.pretty/PGA2040_SMT_NO_SLOT.kicad_mod M  giri-kicad-lib/switches_lib.pretty/PGA2040_SMT_WITH_SLOT.kicad_mod M  giri-kicad-lib/switches_lib.pretty/Pad_Only_SMTSO_M2.kicad_mod A  giri-kicad-lib/switches_lib.pretty/PinHeader_1x02_P2.54mm_Vertical.kicad_mod A  giri-kicad-lib/switches_lib.pretty/SMTSO_M2_Front_Pad.kicad_mod A  giri-kicad-lib/switches_lib.pretty/SMTSO_M2_Pad_M2_hole.kicad_mod M  giri-kicad-lib/switches_lib.pretty/SW_B3U-3000P.kicad_mod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
Parts:
- moved ST1 0.90 mm to (-12.7, 9.57)
Routing:
- net Net-(JP7-B): track 60.2 -> 64.8 mm
- net Net-(JP5-B): track 58.5 -> 60.1 mm
- net GND: track 322.8 -> 321.2 mm
- net /USB_D+: track 16.7 -> 15.3 mm
- net /RUN: track 81.0 -> 82.3 mm
- net /ROW2: track 82.2 -> 81.1 mm
- net SENSOR: track 33.5 -> 34.4 mm
- net /USB_D-: track 16.3 -> 15.4 mm
- net SWDIO: track 63.2 -> 64.0 mm
- net VBUS: track 29.9 -> 29.1 mm
- net Net-(JP6-B): track 20.2 -> 19.6 mm
- net SCL: track 201.2 -> 200.6 mm
- net /~{SDB}: track 208.9 -> 208.4 mm
- net /ROW4: track 105.7 -> 105.1 mm
- net /ROW3: track 91.2 -> 90.7 mm
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
Commit message: M  giri-kicad-lib/switches_lib.pretty/Gateron_1.25u_v2.kicad_mod M  giri-kicad-lib/switches_lib.pretty/Gateron_1u_v2.kicad_mod M  giri-kicad-lib/switches_lib.pretty/Gateron_2u_v2.kicad_mod A  giri-kicad-lib/switches_lib.pretty/SMTSO_M2_FrontPad_M2_hole.kicad_mod A  giri-kicad-lib/switches_lib.pretty/Switch_Cutout2_MX.kicad_mod A  giri-kicad-lib/switches_lib.pretty/Switch_Cutout2_MX_1.25u.kicad_mod A  giri-kicad-lib/switches_lib.pretty/Switch_Cutout2_MX_2u.kicad_mod M  mx/rev3/bottom-cover/pcb/pcb.kicad_pcb M  mx/rev3/bottom-cover/pcb/pcb.kicad_prl M  mx/rev3/bottom-cover/pcb/pcb.kicad_sch M  mx/rev3/pcb-rev2/pcb/pcb.kicad_pcb M  mx/rev3/pcb-rev2/pcb/pcb.kicad_prl M  mx/rev3/pcb-rev2/pcb/pcb.kicad_sch M  mx/rev3/switch-plate-wide/fp-lib-table M  mx/rev3/switch-plate-wide/switch-plate-wide.kicad_pcb M  mx/rev3/switch-plate-wide/switch-plate-wide.kicad_sch A  mx/rev4/notes D  nrfStamp/rev1/pcb/~pcb.kicad_sch.lck D  rp2040stamp/rev2/pcb/~pcb.kicad_sch.lck M  rp2040stamp/rev3/pcb/fp-lib-table M  rp2040stamp/rev3/pcb/pcb.kicad_pcb M  rp2040stamp/rev3/pcb/pcb.kicad_prl M  rp2040stamp/rev3/pcb/pcb.kicad_sch M  rp2040stamp/rev3/pcb/sym-lib-table
Parts:
- removed J1: Conn_01x06_Socket, Connector_JST:JST_SH_SM06B-SRSS-TB_1x06-1MP_P1.00mm_Horizontal
- removed JP7: SolderJumper_2_Open, Jumper:SolderJumper-2_P1.3mm_Open_TrianglePad1.0x1.5mm
- added J2: Conn_02x05_Odd_Even, Connector_PinHeader_1.27mm:PinHeader_2x05_P1.27mm_Horizontal, F.Cu at (-6.80, 64.0)
- R4: value 20k -> 100k
Connections:
- net /RUN renamed /RESET
- net /~{SDB} renamed /SDB
- R4 pad 1: +3V3 -> GND
- ST1 pad 2: unconnected-(ST1-P2-Pad2) -> /SWO
- ST1 pad 3: Net-(JP7-B) -> /TDI
Routing:
- net /TDI: track 0.00 -> 71.2 mm, vias 0 -> 2
- net Net-(JP7-B): track 64.8 -> 0.00 mm, vias 2 -> 0
- net /SWO: track 0.00 -> 55.8 mm, vias 0 -> 1
- net +3V3: track 1658.3 -> 1684.8 mm
- net /RESET: track 82.3 -> 58.2 mm, vias 4 -> 0
- net VDDH: track 3.38 -> 0.00 mm
- net SWCLK: track 68.4 -> 71.4 mm
- net GND: track 321.2 -> 323.9 mm, vias 29 -> 30
- net Net-(JP5-B): track 60.1 -> 62.3 mm
- net SWDIO: track 64.0 -> 66.0 mm
- net SENSOR: track 34.4 -> 33.2 mm
- net /ROW3: track 90.7 -> 90.1 mm
