File: mx/rev3/pcb-rev2/pcb/pcb.kicad_sch (KiCad schematic)
At the start: 280 parts, among them J1 Conn_01x06_Socket, Q1 MMBT3904, Q2 MMBT3904, Q3 MMBT3904, SW1 SW_DIP_x01_XKB_TS_2030, SW2 SW_DIP_x01_XKB_TS_2030, U1 IS31FL3731-QF

Commit message: M  giri-kicad-lib/switches_lib.pretty/Gateron_1.25u_v2.kicad_mod M  giri-kicad-lib/switches_lib.pretty/Gateron_1u_v2.kicad_mod M  giri-kicad-lib/switches_lib.pretty/Gateron_2u_v2.kicad_mod A  giri-kicad-lib/switches_lib.pretty/SMTSO_M2_FrontPad_M2_hole.kicad_mod A  giri-kicad-lib/switches_lib.pretty/Switch_Cutout2_MX.kicad_mod A  giri-kicad-lib/switches_lib.pretty/Switch_Cutout2_MX_1.25u.kicad_mod A  giri-kicad-lib/switches_lib.pretty/Switch_Cutout2_MX_2u.kicad_mod M  mx/rev3/bottom-cover/pcb/pcb.kicad_pcb M  mx/rev3/bottom-cover/pcb/pcb.kicad_prl M  mx/rev3/bottom-cover/pcb/pcb.kicad_sch M  mx/rev3/pcb-rev2/pcb/pcb.kicad_pcb M  mx/rev3/pcb-rev2/pcb/pcb.kicad_prl M  mx/rev3/pcb-rev2/pcb/pcb.kicad_sch M  mx/rev3/switch-plate-wide/fp-lib-table M  mx/rev3/switch-plate-wide/switch-plate-wide.kicad_pcb M  mx/rev3/switch-plate-wide/switch-plate-wide.kicad_sch A  mx/rev4/notes D  nrfStamp/rev1/pcb/~pcb.kicad_sch.lck D  rp2040stamp/rev2/pcb/~pcb.kicad_sch.lck M  rp2040stamp/rev3/pcb/fp-lib-table M  rp2040stamp/rev3/pcb/pcb.kicad_pcb M  rp2040stamp/rev3/pcb/pcb.kicad_prl M  rp2040stamp/rev3/pcb/pcb.kicad_sch M  rp2040stamp/rev3/pcb/sym-lib-table
Parts:
- removed J1: Conn_01x06_Socket, Connector_JST:JST_SH_SM06B-SRSS-TB_1x06-1MP_P1.00mm_Horizontal, symbol giri:JST_Conn_01x07_Pin
- removed JP7: SolderJumper_2_Open, Jumper:SolderJumper-2_P1.3mm_Open_TrianglePad1.0x1.5mm, symbol Jumper:SolderJumper_2_Open
- added J2: Conn_02x05_Odd_Even, Connector_PinHeader_1.27mm:PinHeader_2x05_P1.27mm_Horizontal, symbol Connector_Generic:Conn_02x05_Odd_Even
- R4: value 20k -> 100k
Connections:
- net +3V3: now also J2.1 (Pin_1); no longer R4.1
- net GND: now also R4.1, J2.3 (Pin_3), J2.5 (Pin_5), J2.7 (Pin_7), J2.9 (Pin_9)
- net SWCLK: now also J2.4 (Pin_4)
- net SWDIO: now also J2.2 (Pin_2)
- net SWO: now reaches ST1.2 (P2)
- net SWO: now also J2.6 (Pin_6)
- net TDI: now reaches ST1.3 (P3)
- net TDI: now also J2.8 (Pin_8)
- net RUN renamed RESET
- net RESET: now also J2.10 (Pin_10)
- net ~{SDB} renamed SDB
- no-connect marks 7 -> 6
Other:
- note added: "JTAG Connector"
- note removed: "Debug"

Commit message: A  giri-kicad-lib/RP2040_Minimal.kicad_sym A  giri-kicad-lib/RP2040_minimal.pretty/8-USON-Handsolder.kicad_mod A  giri-kicad-lib/RP2040_minimal.pretty/8-USON.kicad_mod A  giri-kicad-lib/RP2040_minimal.pretty/C_0402_1005Metric.kicad_mod A  giri-kicad-lib/RP2040_minimal.pretty/C_0603_1608Metric.kicad_mod A  giri-kicad-lib/RP2040_minimal.pretty/C_0603_1608Metric_Pad1.08x0.95mm_HandSolder.kicad_mod A  giri-kicad-lib/RP2040_minimal.pretty/C_1206_3216Metric.kicad_mod A  giri-kicad-lib/RP2040_minimal.pretty/Crystal_SMD_2520-4Pin_2.5x2.0mm-Handsolder.kicad_mod A  giri-kicad-lib/RP2040_minimal.pretty/Crystal_SMD_HC49-US.kicad_mod A  giri-kicad-lib/RP2040_minimal.pretty/D_0402_1005Metric.kicad_mod A  giri-kicad-lib/RP2040_minimal.pretty/D_SOD-523.kicad_mod A  giri-kicad-lib/RP2040_minimal.pretty/Diodes_U_DFN1212_3.kicad_mod A  giri-kicad-lib/RP2040_minimal.pretty/Diodes_U_DFN1212_3_Handsolder.kicad_mod A  giri-kicad-lib/RP2040_minimal.pretty/LED_0402_1005Metric.kicad_mod A  giri-kicad-lib/RP2040_minimal.pretty/LED_Driver_Mod_Conn.kicad_mod A  giri-kicad-lib/RP2040_minimal.pretty/LED_Driver_Mod_Conn_1.27.kicad_mod A  giri-kicad-lib/RP2040_minimal.pretty/Module_Conn_Regular.kicad_mod A  giri-kicad-lib/RP2040_minimal.pretty/Module_Conn_Regular2.kicad_mod A  giri-kicad-lib/RP2040_minimal.pretty/Module_Conn_Regular_Outline.kicad_mod A  giri-kicad-lib/RP2040_minimal.pretty/QFN-28-1EP_4x4mm_P0.4mm_EP2.3x2.3mm-Handsolder.kicad_mod A  giri-kicad-lib/RP2040_minimal.pretty/QFN-28-1EP_4x4mm_P0.4mm_EP2.3x2.3mm.kicad_mod A  giri-kicad-lib/RP2040_minimal.pretty/RP2040-QFN-56-Handsolder.kicad_mod A  giri-kicad-lib/RP2040_minimal.pretty/RP2040-QFN-56.kicad_mod A  giri-kicad-lib/RP2040_minimal.pretty/R_0402_1005Metric.kicad_mod A  giri-kicad-lib/RP2040_minimal.pretty/R_0603_1608Metric_Pad0.98x0.95mm_HandSolder.kicad_mod A  giri-kicad-lib/RP2040_minimal.pretty/SW_CK_KXT3.kicad_mod A  giri-kicad-lib/RP2040_minimal.pretty/SW_SPST_Panasonic_EVPAF.kicad_mod A  giri-kicad-lib/RP2040_minimal.pretty/S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
Parts:
- renumbered N4 to N5, Q1 to Q10, Q2 to Q11, Q3 to Q12, Q1 to Q13, Q2 to Q14, Q3 to Q15, Q1 to Q4, Q2 to Q5, Q3 to Q6, Q1 to Q7, Q2 to Q8, Q3 to Q9, R1_r1 to R1_r10, R1_r2 to R1_r11, R1_r3 to R1_r12, R1_r1 to R1_r13, R1_r2 to R1_r14, R1_r3 to R1_r15, R1_r1 to R1_r4, R1_r2 to R1_r5, R1_r3 to R1_r6, R1_r1 to R1_r7, R1_r2 to R1_r8, R1_r3 to R1_r9, R2_r1 to R2_r10, R2_r2 to R2_r11, R2_r3 to R2_r12, R2_r1 to R2_r13, R2_r2 to R2_r14, R2_r3 to R2_r15, R2_r1 to R2_r4, R2_r2 to R2_r5, R2_r3 to R2_r6, R2_r1 to R2_r7, R2_r2 to R2_r8, R2_r3 to R2_r9, Rgr4 to Rgr5, Ri2 to Ri10, Ri3 to Ri11, Ri3 to Ri12, Ri3 to Ri13, Ri3 to Ri14, Ri3 to Ri15, Ri4 to Ri16, Ri4 to Ri17, Ri4 to Ri18, Ri4 to Ri19, Ri1 to Ri2, Ri4 to Ri20, Ri5 to Ri21, Ri5 to Ri22, Ri5 to Ri23, Ri5 to Ri24, Ri1 to Ri3, Ri1 to Ri4, Ri1 to Ri5, Ri2 to Ri6, Ri2 to Ri7, Ri2 to Ri8, Ri2 to Ri9, S1 to S10, S6 to S11, S11 to S12, S1 to S13, S6 to S14, S11 to S15, S2 to S16, S7 to S17, S12 to S18, S2 to S19, S6 to S2, S7 to S20, S12 to S21, S2 to S22, S7 to S23, S12 to S24, S2 to S25, S7 to S26, S12 to S27, S7 to S28, S12 to S29, S11 to S3, S3 to S30, S8 to S31, S13 to S32, S3 to S33, S8 to S34, S13 to S35, S3 to S36, S8 to S37, S13 to S38, S3 to S39, S1 to S4, S8 to S40, S13 to S41, S3 to S42, S8 to S43, S13 to S44, S4 to S45, S9 to S46, S14 to S47, S4 to S48, S9 to S49, S6 to S5, S14 to S50, S4 to S51, S9 to S52, S14 to S53, S4 to S54, S9 to S55, S14 to S56, S4 to S57, S14 to S58, S5 to S59, S11 to S6, S10 to S60, S15 to S61, S5 to S62, S10 to S63, S15 to S64, S5 to S65, S10 to S66, S15 to S67, S5 to S68, S10 to S69, S1 to S7, S15 to S70, S2 to S71, S9 to S72, S6 to S8, S11 to S9
