File: mx/rev3/switch-plate-wide/switch-plate-wide.kicad_pcb (KiCad board)
At the start: 2 copper layers, 309.8 x 191 mm, 101 parts

Commit message: M  giri-kicad-lib/switches_lib.pretty/Gateron_1.25u_v2.kicad_mod M  giri-kicad-lib/switches_lib.pretty/Gateron_1u_v2.kicad_mod M  giri-kicad-lib/switches_lib.pretty/Gateron_2u_v2.kicad_mod A  giri-kicad-lib/switches_lib.pretty/SMTSO_M2_FrontPad_M2_hole.kicad_mod A  giri-kicad-lib/switches_lib.pretty/Switch_Cutout2_MX.kicad_mod A  giri-kicad-lib/switches_lib.pretty/Switch_Cutout2_MX_1.25u.kicad_mod A  giri-kicad-lib/switches_lib.pretty/Switch_Cutout2_MX_2u.kicad_mod M  mx/rev3/bottom-cover/pcb/pcb.kicad_pcb M  mx/rev3/bottom-cover/pcb/pcb.kicad_prl M  mx/rev3/bottom-cover/pcb/pcb.kicad_sch M  mx/rev3/pcb-rev2/pcb/pcb.kicad_pcb M  mx/rev3/pcb-rev2/pcb/pcb.kicad_prl M  mx/rev3/pcb-rev2/pcb/pcb.kicad_sch M  mx/rev3/switch-plate-wide/fp-lib-table M  mx/rev3/switch-plate-wide/switch-plate-wide.kicad_pcb M  mx/rev3/switch-plate-wide/switch-plate-wide.kicad_sch A  mx/rev4/notes D  nrfStamp/rev1/pcb/~pcb.kicad_sch.lck D  rp2040stamp/rev2/pcb/~pcb.kicad_sch.lck M  rp2040stamp/rev3/pcb/fp-lib-table M  rp2040stamp/rev3/pcb/pcb.kicad_pcb M  rp2040stamp/rev3/pcb/pcb.kicad_prl M  rp2040stamp/rev3/pcb/pcb.kicad_sch M  rp2040stamp/rev3/pcb/sym-lib-table
Parts:
- S1, S10, S11, S12, S13, S14, S15, S16, S17, S18, S19, S2, S20, S21, S22, S23, S24, S25, S26, S27, S28, S29, S3, S31, S32, S33, S34, S35, S36, S37, S38, S39, S4, S40, S41, S42, S43, S44, S45, S46, S47, S48, S49, S5, S50, S51, S52, S53, S54, S55, S56, S58, S59, S6, S61, S65, S67, S68, S69, S7, S70, S71, S72, S8, S9: footprint Giri_Library:Switch_Cutout_MX -> Giri_Library:Switch_Cutout2_MX
- S30, S57, S60, S62, S63: footprint Giri_Library:Switch_Cutout_MX_1.25u -> Giri_Library:Switch_Cutout2_MX_1.25u
- S64, S66: footprint Giri_Library:Switch_Cutout_MX_2u -> Giri_Library:Switch_Cutout2_MX_2u
