File: mx/rev3/switch-plate-wide/switch-plate-wide.kicad_sch (KiCad schematic)
At the start: 91 parts

Commit message: M giri-kicad-lib/switches.kicad_sym  M giri-kicad-lib/switches_lib.pretty/C_0603_1608Metric.kicad_mod  M giri-kicad-lib/switches_lib.pretty/Gateron_1u.kicad_mod  M giri-kicad-lib/switches_lib.pretty/Gateron_Sw_1u.kicad_mod  M giri-kicad-lib/switches_lib.pretty/PGA2040_SMT_WITH_SLOT.kicad_mod  M giri-kicad-lib/switches_lib.pretty/Pad_Only_SMTSO_M2.kicad_mod  M giri-kicad-lib/switches_lib.pretty/SW_B3U-3000P.kicad_mod  D giri-kicad-lib/switches_lib.pretty/WristExtension.kicad_mod A  mx/rev3/Wrist-Plate2/Wrist-Plate2.kicad_pcb A  mx/rev3/Wrist-Plate2/Wrist-Plate2.kicad_prl A  mx/rev3/Wrist-Plate2/Wrist-Plate2.kicad_pro A  mx/rev3/Wrist-Plate2/Wrist-Plate2.kicad_sch A  mx/rev3/Wrist-Plate2/fp-lib-table M  mx/rev3/border.py R  mx/rev3/pcb/LED-Driver.kicad_sch -> mx/rev3/pcb-rev1/pcb/LED-Driver.kicad_sch R  mx/rev3/pcb/fp-lib-table -> mx/rev3/pcb-rev1/pcb/fp-lib-table R  mx/rev3/pcb/pcb-b.jpg -> mx/rev3/pcb-rev1/pcb/pcb-b.jpg R  mx/rev3/pcb/pcb.jpg -> mx/rev3/pcb-rev1/pcb/pcb.jpg R  mx/rev3/pcb/pcb.kicad_pcb -> mx/rev3/pcb-rev1/pcb/pcb.kicad_pcb A  mx/rev3/pcb-rev1/pcb/pcb.kicad_prl R  mx/rev3/pcb/pcb.kicad_pro -> mx/rev3/pcb-rev1/pcb/pcb.kicad_pro R  mx/rev3/pcb/pcb.kicad_sch -> mx/rev3/pcb-rev1/pcb/pcb.kicad_sch R  mx/rev3/pcb/sym-lib-table -> mx/rev3/pcb-rev1/pcb/sym-lib-table A  mx/rev3/pcb-rev2/pcb/LED-Driver.kicad_sch A  mx/rev3/pcb-rev2/pcb/fp-lib-table A  mx/rev3/pcb-rev2/pcb/pcb-b.jpg A  mx/rev3/pcb-rev2/pcb/pcb.jpg A  mx/rev3/pcb-rev2/pcb/pcb.kicad_pcb R  mx/rev3/pcb/pcb.kicad_prl -> mx/rev3/pcb-rev2/pcb/pcb.kicad_prl A  mx/rev3/pcb-rev2/pcb/pcb.kicad_pro A  mx/rev3/pcb-rev2/pcb/pcb.kicad_sch A  mx/rev3/pcb-rev2/pcb/sym-lib-table D  mx/rev3/pcb/.gitignore M  mx/rev3/place.py A  mx/rev3/switch-plate-wide/fp-lib-table A  mx/rev3/switch-plate-wide/switch-plate-wide.kicad_pcb A  mx/rev3/switch-plate-wide/switch-plate-wide.kicad_prl A  mx/rev3/switch-plate-wide/switch-plate-wide.kicad_pro A  mx/rev3/switch-plate-wide/switch-plate-wide.kicad_sch A  mx/rev3/switch-plat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
Parts:
- added H1, H2, H3, H4, H5, H6, H7, H8: MountingHole, Giri_Library:MountingHole_2.2mm_M2_SmallPad, symbol Mechanical:MountingHole
- added TP1, TP2: TestPoint, TestPoint:TestPoint_Pad_1.0x1.0mm, symbol Connector:TestPoint
- Hs1, Hs10, Hs11, Hs12, Hs13, Hs14, Hs15, Hs16, Hs17, Hs18, Hs2, Hs3, Hs4, Hs5, Hs6, Hs7, Hs8, Hs9: footprint Giri_Library:MountingHole_2.2mm_M2_NoPad -> Giri_Library:MountingHole_2.2mm_M2_SmallPad
- S30, S57, S60, S62, S63: footprint Giri_Library:Switch_Cutout_MX -> Giri_Library:Switch_Cutout_MX_1.25u
Connections:
- new net GND: TP1.1, TP2.1
Other:
- title: Switch Plate - Keychron Switch -> Switch Plate

Commit message: M  giri-kicad-lib/switches_lib.pretty/Gateron_1.25u_v2.kicad_mod M  giri-kicad-lib/switches_lib.pretty/Gateron_1u_v2.kicad_mod M  giri-kicad-lib/switches_lib.pretty/Gateron_2u_v2.kicad_mod A  giri-kicad-lib/switches_lib.pretty/SMTSO_M2_FrontPad_M2_hole.kicad_mod A  giri-kicad-lib/switches_lib.pretty/Switch_Cutout2_MX.kicad_mod A  giri-kicad-lib/switches_lib.pretty/Switch_Cutout2_MX_1.25u.kicad_mod A  giri-kicad-lib/switches_lib.pretty/Switch_Cutout2_MX_2u.kicad_mod M  mx/rev3/bottom-cover/pcb/pcb.kicad_pcb M  mx/rev3/bottom-cover/pcb/pcb.kicad_prl M  mx/rev3/bottom-cover/pcb/pcb.kicad_sch M  mx/rev3/pcb-rev2/pcb/pcb.kicad_pcb M  mx/rev3/pcb-rev2/pcb/pcb.kicad_prl M  mx/rev3/pcb-rev2/pcb/pcb.kicad_sch M  mx/rev3/switch-plate-wide/fp-lib-table M  mx/rev3/switch-plate-wide/switch-plate-wide.kicad_pcb M  mx/rev3/switch-plate-wide/switch-plate-wide.kicad_sch A  mx/rev4/notes D  nrfStamp/rev1/pcb/~pcb.kicad_sch.lck D  rp2040stamp/rev2/pcb/~pcb.kicad_sch.lck M  rp2040stamp/rev3/pcb/fp-lib-table M  rp2040stamp/rev3/pcb/pcb.kicad_pcb M  rp2040stamp/rev3/pcb/pcb.kicad_prl M  rp2040stamp/rev3/pcb/pcb.kicad_sch M  rp2040stamp/rev3/pcb/sym-lib-table
Parts:
- S1, S10, S11, S12, S13, S14, S15, S16, S17, S18, S19, S2, S20, S21, S22, S23, S24, S25, S26, S27, S28, S29, S3, S31, S32, S33, S34, S35, S36, S37, S38, S39, S4, S40, S41, S42, S43, S44, S45, S46, S47, S48, S49, S5, S50, S51, S52, S53, S54, S55, S56, S58, S59, S6, S61, S65, S67, S68, S69, S7, S70, S71, S72, S8, S9: footprint Giri_Library:Switch_Cutout_MX -> Giri_Library:Switch_Cutout2_MX
- S30, S57, S60, S62, S63: footprint Giri_Library:Switch_Cutout_MX_1.25u -> Giri_Library:Switch_Cutout2_MX_1.25u
- S64, S66: footprint Giri_Library:Switch_Cutout_MX_2u -> Giri_Library:Switch_Cutout2_MX_2u
